File: hardware/sheets/b4_switching.kicad_sch (KiCad schematic)
At the start: 54 parts, among them J401 KF301-5.0-3P, J402 KF301-5.0-3P, J403 KF301-5.0-3P, J404 KF301-5.0-3P, J411 KF301-5.0-2P, J412 KF301-5.0-2P, K401 HK4100F-DC5V-SHG, K402 HK4100F-DC5V-SHG, K403 HK4100F-DC5V-SHG, K404 HK4100F-DC5V-SHG, Q401 AO3400A, Q402 AO3400A, Q403 AO3400A, Q404 AO3400A, Q411 MMBT5551, Q412 MMBT5551, Q421 MMBT5551, Q422 MMBT5551, U401 6N137S-TA1-L, U402 6N137S-TA1-L

Commit message: hardware: chip resistors and ceramic capacitors on KiCad standard footprints (Decision #47); schematic, library and gapped copies regenerated, ERC 0 errors
Co-Authored-By: Claude Fable 5.1 <noreply@anthropic.com>
Parts:
- C401, C402: footprint class_board:C0603 -> Capacitor_SMD:C_0603_1608Metric
- R401, R402, R403, R404, R411, R412, R413, R414, R421, R422, R423, R424, R431, R432, R441, R442, R451, R452, R461, R462, R471, R472: footprint class_board:R0603 -> Resistor_SMD:R_0603_1608Metric

Commit message: hardware: panel stacked on the back (180 x 100, three 2x20 headers, 17 SMA, TTL strip, TX terminal, Qwiic); TTL/fast/TX-coil/Qwiic connectors leave the main board; mains-safe relay channels (JQC-3FF 10 A, MAINS net class + DRC rules); library, sheets, gapped copies, docs regenerated; ERC 0 errors
Decisions #45-#50 in the course repo. The main-board PCB is unchanged: Update PCB from Schematic, header placement, relay re-spacing and connector rotation are the instructor's GUI steps on the master.

Co-Authored-By: Claude Fable 5.1 <noreply@anthropic.com>
Parts:
- K401, K402, K403, K404: value HK4100F-DC5V-SHG -> JQC-3FF/005-1ZS; footprint class_board:RELAY-TH_HK4100F-DC5V-SHG -> Relay_THT:Relay_SPDT_Hongfa_JQC-3FF_0XX-1Z; symbol class_board:HK4100F-DC5V-SHG -> class_board:JQC-3FF-005-1ZS; LCSC C12072 -> C9221; MPN HK4100F-DC5V-SHG -> JQC-3FF/005-1ZS(551); Manufacturer Ningbo Huike -> Hongfa
Connections:
- net +5V_RAW: now also K401.A1 (COIL+), K402.A1 (COIL+), K403.A1 (COIL+), K404.A1 (COIL+); no longer K401.3 (COIL+), K402.3 (COIL+), K403.3 (COIL+), K404.3 (COIL+)
- net RLY_COM1: now also K401.11 (COM); no longer K401.5 (COM), K401.6 (COM)
- net RLY_COM2: now also K402.11 (COM); no longer K402.5 (COM), K402.6 (COM)
- net RLY_COM3: now also K403.11 (COM); no longer K403.5 (COM), K403.6 (COM)
- net RLY_COM4: now also K404.11 (COM); no longer K404.5 (COM), K404.6 (COM)
- net RLY_NC1: now also K401.12 (NC); no longer K401.2 (NC)
- net RLY_NC2: now also K402.12 (NC); no longer K402.2 (NC)
- net RLY_NC3: now also K403.12 (NC); no longer K403.2 (NC)
- net RLY_NC4: now also K404.12 (NC); no longer K404.2 (NC)
- net RLY_NO1: now also K401.14 (NO); no longer K401.1 (NO)
- net RLY_NO2: now also K402.14 (NO); no longer K402.1 (NO)
- net RLY_NO3: now also K403.14 (NO); no longer K403.1 (NO)
- net RLY_NO4: now also K404.14 (NO); no longer K404.1 (NO)
- net at D401.2 (A), D411.1 (K), Q401.3 (D): now also K401.A2 (COIL-); no longer K401.4 (COIL-)
- net at D404.2 (A), D414.1 (K), Q404.3 (D): now also K404.A2 (COIL-); no longer K404.4 (COIL-)
- net at D403.2 (A), D413.1 (K), Q403.3 (D): now also K403.A2 (COIL-); no longer K403.4 (COIL-)
- net at D402.2 (A), D412.1 (K), Q402.3 (D): now also K402.A2 (COIL-); no longer K402.4 (COIL-)
Other:
- note added: "B4 — MAINS-CAPABLE SWITCHING: 4 x SPDT relay (10 A @ 277 V AC) on AO3400A MOSFETs; 2 x 6N137 isolated inputs, 5-24 V"
- note added: "Coil current: 4 x 71 mA = 285 mA from +5V_RAW (the 125 ohm HK4100F coils drew 160 mA) — see the rails table on the root sheet."
- note added: "Contacts: COM/NO/NC to the 3P terminal, NO = pad 1, COM = pad 2, NC = pad 3. Relay pins are the footprint pad names (EN 50005): A1/A2 = coil, 11 = COM, 12 = NC, 14 = NO. The coil-to-contact distance inside the relay is the manufacturer's isolation (1.5 kV test) and is excluded from the 5 mm rule; mains is switched only with the instructor present, the load fused <= 5 A and the lid on."
- note added: "J401: 1 = NO, 2 = COM, 3 = NC MAINS: 250 V AC 5 A MAX, load fused <= 5 A"
- note added: "J402: 1 = NO, 2 = COM, 3 = NC MAINS: 250 V AC 5 A MAX, load fused <= 5 A"
- note added: "J403: 1 = NO, 2 = COM, 3 = NC MAINS: 250 V AC 5 A MAX, load fused <= 5 A"
- note added: "J404: 1 = NO, 2 = COM, 3 = NC MAINS: 250 V AC 5 A MAX, load fused <= 5 A"
- note added: "K401: SPDT 10 A @ 277 V AC / 28 V DC, coil 5 V 70 ohm (71 mA); terminal directly behind the relay"
- note added: "K402: SPDT 10 A @ 277 V AC / 28 V DC, coil 5 V 70 ohm (71 mA); terminal directly behind the relay"
- note added: "K403: SPDT 10 A @ 277 V AC / 28 V DC, coil 5 V 70 ohm (71 mA); terminal directly behind the relay"
- note added: "K404: SPDT 10 A @ 277 V AC / 28 V DC, coil 5 V 70 ohm (71 mA); terminal directly behind the relay"
- note added: "MAINS design rules (class-board.kicad_dru): MAINS copper keeps 5 mm to every other net on every layer and 5 mm channel-to-channel, 2 mm between the nets of one channel, 2 mm to the board edge; F.Cu only, no vias, tracks >= 3 mm."
- note added: "MAINS-capable channel: relay 10 A @ 277 V AC; board rating 250 V AC 5 A MAX per channel, load fused <= 5 A; MAINS net class: 5 mm to all other copper on every layer, F.Cu only, no vias, >= 3 mm tracks; terminal directly behind its relay on the rear edge; coil 70 ohm = 71 mA per relay (4 x 71 = 285 mA from +5V_RAW)."
- note added: "Relay drive: AO3400A (48 mOhm) instead of a Darlington: the 5 V coil gets the full +5V_RAW (JQC-3FF/005-1ZS pull-in <= 3.75 V, coil 70 ohm = 71 mA per relay, 4 x 71 = 285 mA from +5V_RAW). 1 k gate series, 1N4148W flyback across the coil. Yellow LED shows coil on."
- note removed: "B4 — ISOLATED SWITCHING: 4 x SPDT relay (3 A / 30 VDC) on AO3400A MOSFETs; 2 x 6N137 isolated inputs, 5-24 V"
- note removed: "Contacts: COM/NO/NC to a 3P terminal. Rated 3 A at 30 VDC / 250 VAC by the relay, but this board is limited to <= 30 V DC, 1 A (silkscreen). NO = pad 1, NC = pad 2, COM = pads 5/6 (HK4100F drawing, bottom view mirrored)."
- note removed: "J401: 1 = NO, 2 = COM, 3 = NC (<= 30 V DC, 1 A)"
- note removed: "J402: 1 = NO, 2 = COM, 3 = NC (<= 30 V DC, 1 A)"
- note removed: "J403: 1 = NO, 2 = COM, 3 = NC (<= 30 V DC, 1 A)"
- note removed: "J404: 1 = NO, 2 = COM, 3 = NC (<= 30 V DC, 1 A)"
- note removed: "Relay drive: AO3400A (48 mOhm) instead of a Darlington: the 5 V coil gets the full +5V_RAW (HK4100F pull-in <= 3.75 V guaranteed, coil 125 R = 40 mA). 1 k gate series, 1N4148W flyback across the coil. Yellow LED shows coil on."
- title: B4: 4 relays (MOSFET drive) + 2 isolated 5-24 V inputs -> B4: 4 mains-capable relays (MOSFET drive) + 2 isolated 5-24 V inputs
- moved on the sheet: J401, J402, J403, J404
