File: hardware/sheets/front_panel_link.kicad_sch (KiCad schematic)
At the start: 1 part, among them J6 Panel link 2x20 R/A

Commit message: hardware: panel stacked on the back (180 x 100, three 2x20 headers, 17 SMA, TTL strip, TX terminal, Qwiic); TTL/fast/TX-coil/Qwiic connectors leave the main board; mains-safe relay channels (JQC-3FF 10 A, MAINS net class + DRC rules); library, sheets, gapped copies, docs regenerated; ERC 0 errors
Decisions #45-#50 in the course repo. The main-board PCB is unchanged: Update PCB from Schematic, header placement, relay re-spacing and connector rotation are the instructor's GUI steps on the master.

Co-Authored-By: Claude Fable 5.1 <noreply@anthropic.com>
Parts:
- added J7, J8: Panel link 2x20 male, Connector_PinHeader_2.54mm:PinHeader_2x20_P2.54mm_Vertical, symbol class_board:HDR_2x20_MALE
- J6: value Panel link 2x20 R/A -> Panel link 2x20 male; footprint class_board:HDR-TH_40P-P2.54-H-R2-C20-S2.54-W10.0 -> Connector_PinHeader_2.54mm:PinHeader_2x20_P2.54mm_Vertical; symbol class_board:HDR_2x20_RA_MALE -> class_board:HDR_2x20_MALE; Assembly (none) -> hand; JLC_CLASS Extended -> (none); LCSC C124369 -> (none); MPN B-2100R40P-B110 -> 2x20 straight pin header 2.54 mm; Manufacturer Ckmtw -> any; Purchase (none) -> C5224014; now left out of the parts list
Connections:
- net +3V3: now also J7.27, J7.29, J8.5; no longer J6.29, J6.31
- net AGND: now also J6.26, J6.28, J6.30, J6.32, J6.34, J6.36, J6.6
- net AI1: now also J6.1; no longer J6.9
- net AI2: now also J6.3; no longer J6.11
- net AI3: now also J6.5; no longer J6.13
- net AI4: now also J6.7; no longer J6.15
- net AI5: now also J6.9; no longer J6.17
- net AI6: now also J6.11; no longer J6.19
- net AI7: now also J6.13; no longer J6.21
- net AI8: now also J6.15; no longer J6.23
- net AO1: now also J6.25; no longer J6.1
- net AO2: now also J6.27; no longer J6.3
- net AUX: now also J6.23; no longer J6.7
- net GND: now also J7.10, J7.12, J7.14, J7.16, J7.18, J7.2, J7.20, J7.22, J7.24, J7.26, J7.28, J7.30, J7.32, J7.34, J7.36, J7.38, J7.4, J7.40, J7.6, J7.8, J8.10, J8.12, J8.14, J8.16, J8.18, J8.2, J8.20, J8.22, J8.24, J8.26, J8.28, J8.30, J8.32, J8.34, J8.36, J8.38, J8.4, J8.40, J8.6, J8.8; no longer J6.26, J6.28, J6.30, J6.32, J6.34, J6.36, J6.6
- net I2C_SCL: now also J7.25; no longer J6.27
- net I2C_SDA: now also J7.23; no longer J6.25
- net LED_ACT: now also J7.33; no longer J6.35
- net LED_WIFI: now also J7.31; no longer J6.33
- net RX: now also J6.17; no longer J6.37
- net TRIG_5V: now also J7.21; no longer J6.5
- net TX: now also J6.19, J6.21; no longer J6.39
- new net +5V_RAW: J8.1, J8.3
- new net FASTTTL1: J7.17
- new net FASTTTL2: J7.19
- new net GPIO15: J8.13
- new net GPIO4: J8.7
- new net GPIO43: J8.15
- new net GPIO44: J8.17
- new net GPIO6: J8.9
- new net GPIO7: J8.11
- new net TTL1: J7.1
- new net TTL2: J7.3
- new net TTL3: J7.5
- new net TTL4: J7.7
- new net TTL5: J7.9
- new net TTL6: J7.11
- new net TTL7: J7.13
- new net TTL8: J7.15
- no-connect marks 0 -> 20
Other:
- note added: "+5V_RAW GND +5V_RAW GND +3V3 GND"
- note added: "1-6"
- note added: "13-18"
- note added: "19-24"
- note added: "7-12"
- note added: "AI1 AGND AI2 AGND AI3 AGND"
- note added: "AI4 AGND AI5 AGND AI6 AGND"
- note added: "AI7 AGND AI8 AGND RX AGND"
- note added: "AO1 AGND AO2 AGND spare AGND"
- note added: "FASTTTL2 GND TRIG_5V GND I2C_SDA GND"
- note added: "FRONT-PANEL LINK - three 2x20 straight male headers on the BOTTOM side of the main board (v0.8)"
- note added: "GPIO15 GND GPIO43 GND GPIO44 GND"
- note added: "GPIO4 GND GPIO6 GND GPIO7 GND"
- note added: "I2C_SCL GND +3V3 GND LED_PWR GND"
- note added: "J6 - analog, at x = 12 mm on the bottom side"
- note added: "J6 pin table"
- note added: "J7 - digital, at x = 90 mm on the bottom side"
- note added: "J7 pin table"
- note added: "J8 - power + spares, at x = 168 mm on the bottom side"
- note added: "J8 pin table"
- note added: "LED_PWR is +3V3 (always on; the LED series resistor sits on the panel). LED_WIFI / LED_ACT come from GPIO43 / GPIO44 through JP1 / JP2 (base sheet). GPIO4/6/7/15/43/44 on J8 are the same nets as on the expansion header J5. TX is on two pins (19 and 21) so the coil current has two paths."
- note added: "LED_WIFI GND LED_ACT GND spare GND"
- note added: "Odd pins = row 1 (signal), even pins = row 2 (return): every signal pin has its return, AGND or GND, on the adjacent even pin. J6 carries the analog signals (nearest the panel SMAs), J7 the digital ones, J8 the rails and the spare GPIO."
- note added: "Pin 29 of J7 (LED_PWR) is +3V3 directly; the panel LED series resistor sits on the panel PCB."
- note added: "Pins marked spare are not connected on the main board; on the panel they reach labelled test pads, so a later panel part needs no new main-board revision. Panel copper is AGND and meets GND only at the star point NT1 on the main board."
- note added: "Signals (odd = signal, even = its return)"
- note added: "Spare pins: J6 has 6 (29-39 odd, AGND partners), J7 has 3 (35-39 odd), J8 has 11 (19-39 odd) - 20 spare signal pins with their returns."
- note added: "TTL1 GND TTL2 GND TTL3 GND"
- note added: "TTL4 GND TTL5 GND TTL6 GND"
- note added: "TTL7 GND TTL8 GND FASTTTL1 GND"
- note added: "TX AGND TX AGND AUX AGND"
- note added: "The panel stacks flat on the BACK of the main board (Decision #45). J6/J7/J8 are mounted on the BOTTOM side of the main board and hand-soldered from the top; they mate the panel's three female headers. Positions along the 180 mm edge: x ~ 12 (J6), x ~ 90 (J7), x ~ 168 (J8) mm."
- note added: "The three headers (and the panel's three female headers) are bought separately and soldered by the instructor: they carry the field Assembly = hand and are excluded from the JLC BOM and CPL."
- note added: "spare AGND spare AGND"
- note added: "spare AGND spare AGND spare AGND"
- note added: "spare GND spare GND"
- note added: "spare GND spare GND spare GND"
- note removed: "1-8"
- note removed: "17-24"
- note removed: "9-16"
- note removed: "AI1 AGND AI2 AGND AI3 AGND AI4 AGND"
- note removed: "AI5 AGND AI6 AGND AI7 AGND AI8 AGND"
- note removed: "AO1 AGND AO2 AGND TRIG_5V GND AUX AGND"
- note removed: "FRONT-PANEL LINK — J6 2x20 right-angle male (front edge), pinout per design brief 7.8"
- note removed: "I2C_SDA GND I2C_SCL GND +3V3 GND"
- note removed: "LED_PWR GND LED_WIFI GND LED_ACT GND"
- note removed: "LED_PWR is +3V3 (always on, resistor on the panel). LED_WIFI/LED_ACT come from GPIO43/GPIO44 through JP1/JP2 (base sheet). Pins 37/39 = RX/TX (the NMR receive/transmit coil ports, analog) to the panel SMAs with AGND on 38/40 (v0.7); +5V_RAW no longer reaches the panel."
- note removed: "Odd pins = row A, even pins = row B. Analog signals AO1/AO2/AUX/AI1-8 are each paired with AGND; TRIG_5V, I2C, LEDs and rails with GND. Panel copper is AGND and reaches GND only through the main-board star point NT1."
- note removed: "Pin 31 (LED_PWR) = +3V3 directly; the panel LED series resistor sits on the panel PCB"
- note removed: "RX AGND TX AGND"
- note removed: "Signals"
- title: Front-panel link J6 (2x20, brief 7.8) -> Front-panel link J6/J7/J8 (3 x 2x20, bottom side)
- moved on the sheet: J6

Commit message: v0.7d: relays and mains removed, MODULE OUT 1-7 (5 V TTL) on a shrouded 2x6 header on the front panel, isolated inputs moved to the panel, section C = the front-panel board (4-layer, 18 mm SMA grid, OLED clear of headers, unrouted student copy), main board re-placed; workbook, tutor guide, firmware docs, hardware docs updated (Decision #58)
Co-Authored-By: Claude Fable 5.1 <noreply@anthropic.com>
Parts:
- J6, J7, J8: LCSC (none) -> C5224014; MPN 2x20 straight pin header 2.54 mm -> PZ2.54-2*20; Manufacturer any -> ZHOURI
Connections:
- net MOD1: now reaches J8.19
- net MOD2: now reaches J8.21
- net MOD3: now reaches J8.23
- net MOD4: now reaches J8.25
- net MOD5: now reaches J8.27
- net MOD6: now reaches J8.29
- net MOD7: now reaches J8.31
- net OPTO_IN1: now reaches J8.35
- net OPTO_IN2: now reaches J8.37
- no-connect marks 20 -> 11
Other:
- note added: "J8 - rails, GPIO, module outputs, at x = 168 mm on the bottom side"
- note added: "MOD1 GND MOD2 GND MOD3 GND"
- note added: "MOD4 GND MOD5 GND MOD6 GND"
- note added: "MOD7 GND spare GND OPTO_IN1 GND"
- note added: "MODULE OUT 1..7 (J8 pins 19-31 odd) are 3.3 V logic from the TCA9535 expander: the panel buffers them to 5 V TTL to drive commercial"
- note added: "OPTO_IN2 GND spare GND"
- note added: "Odd pins = row 1 (signal), even pins = row 2 (return): every signal pin has its return, AGND or GND, on the adjacent even pin. J6 carries the analog signals (nearest the panel SMAs), J7 the digital ones, J8 the rails, the free GPIO, the seven module outputs MODULE OUT 1..7 and the two isolated-input returns OPTO_IN1/2."
- note added: "and their open-collector outputs reach GPIO16/17 here. Spare pins: J6 has 6 (29-39 odd), J7 has 3 (35-39 odd), J8 has 2 (33, 39)."
- note added: "on the main board and the panel pulls it down. OPTO_IN1/2 (pins 35, 37) come the other way: the two 6N137 isolated inputs live on the panel"
- note added: "opto-isolated relay modules (5 mA per input). MODULE OUT 8 (pin 33) is RESERVED: no expander port is free for it, so it is not connected"
- note removed: "J8 - power + spares, at x = 168 mm on the bottom side"
- note removed: "Odd pins = row 1 (signal), even pins = row 2 (return): every signal pin has its return, AGND or GND, on the adjacent even pin. J6 carries the analog signals (nearest the panel SMAs), J7 the digital ones, J8 the rails and the spare GPIO."
- note removed: "Spare pins: J6 has 6 (29-39 odd, AGND partners), J7 has 3 (35-39 odd), J8 has 11 (19-39 odd) - 20 spare signal pins with their returns."
- note removed: "spare GND spare GND spare GND"

Commit message: main board: link sockets J6/J7/J8 are female (PinSocket_2x20) on the bottom side, panel headers male (Decision #62); placement regenerated after the density pass, DRC 0 errors, unrouted; schematic + netlist + scripts
Co-Authored-By: Claude Fable 5.1 <noreply@anthropic.com>
Parts:
- J6, J7, J8: value Panel link 2x20 male -> Panel link 2x20 female; footprint Connector_PinHeader_2.54mm:PinHeader_2x20_P2.54mm_Vertical -> Connector_PinSocket_2.54mm:PinSocket_2x20_P2.54mm_Vertical; symbol class_board:HDR_2x20_MALE -> class_board:HDR_2x20_FEMALE; LCSC C5224014 -> C5124634; MPN PZ2.54-2*20 -> 2.54-2*20P (8.5 mm); Manufacturer ZHOURI -> BOOMELE; Purchase C5224014 -> C5124634
Changed lines of the file:
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@@
   (global_label "OPTO_IN1" (shape bidirectional) (at 306.07 168.91 180) (fields_autoplaced yes) (effects (font (size 1.27 1.27)) (justify right)))
   (global_label "OPTO_IN2" (shape bidirectional) (at 306.07 171.45 180) (fields_autoplaced yes) (effects (font (size 1.27 1.27)) (justify right)))
-  (symbol (lib_id "class_board:HDR_2x20_MALE") (at 59.69 149.86 0) (unit 1)
+  (symbol (lib_id "class_board:HDR_2x20_FEMALE") (at 59.69 149.86 0) (unit 1)
     (exclude_from_sim no) (in_bom no) (on_board yes) (dnp no) (fields_autoplaced yes)
     (property "Reference" "J6" (at 55.88 122.428 0) (show_name no) (effects (font (size 1.27 1.27)) (justify left bottom)))
-    (property "Value" "Panel link 2x20 male" (at 55.88 177.292 0) (show_name no) (effects (font (size 1.27 1.27)) (justify left top)))
-    (property "Footprint" "Connector_PinHeader_2.54mm:PinHeader_2x20_P2.54mm_Vertical" (at 59.69 149.86 0) (show_name no) (effects (font (size 1.27 1.27)) (hide yes)))
-    (property "Datasheet" "https://www.lcsc.com/product-detail/C5224014.html" (at 59.69 149.86 0) (show_name no) (effects (font (size 1.27 1.27)) (hide yes)))
-    (property "Description" "2x20 straight male pin header, 2.54 mm, KiCad standard footprint. Bottom side of the main board, hand-soldered from the top; mates the panel's female headers." (at 59.69 149.86 0) (show_name no) (effects (font (size 1.27 1.27)) (hide yes)))
+    (property "Value" "Panel link 2x20 female" (at 55.88 177.292 0) (show_name no) (effects (font (size 1.27 1.27)) (justify left top)))
+    (property "Footprint" "Connector_PinSocket_2.54mm:PinSocket_2x20_P2.54mm_Vertical" (at 59.69 149.86 0) (show_name no) (effects (font (size 1.27 1.27)) (hide yes)))
+    (property "Datasheet" "https://www.lcsc.com/product-detail/C5124634.html" (at 59.69 149.86 0) (show_name no) (effects (font (size 1.27 1.27)) (hide yes)))
+    (property "Description" "2x20 straight female header 8.5 mm, 2.54 mm, KiCad standard footprint. Panel inner face, hand-soldered; mates the main board's male headers." (at 59.69 149.86 0) (show_name no) (effects (font (size 1.27 1.27)) (hide yes)))
     (property "Assembly" "hand" (at 59.69 149.86 0) (show_name no) (effects (font (size 1.27 1.27)) (hide yes)))
-    (property "MPN" "PZ2.54-2*20" (at 59.69 149.86 0) (show_name no) (effects (font (size 1.27 1.27)) (hide yes)))
-    (property "Manufacturer" "ZHOURI" (at 59.69 149.86 0) (show_name no) (effects (font (size 1.27 1.27)) (hide yes)))
-    (property "Purchase" "C5224014" (at 59.69 149.86 0) (show_name no) (effects (font (size 1.27 1.27)) (hide yes)))
-    (property "LCSC" "C5224014" (at 59.69 149.86 0) (show_name no) (effects (font (size 1.27 1.27)) (hide yes)))
+    (property "MPN" "2.54-2*20P (8.5 mm)" (at 59.69 149.86 0) (show_name no) (effects (font (size 1.27 1.27)) (hide yes)))
+    (property "Manufacturer" "BOOMELE" (at 59.69 149.86 0) (show_name no) (effects (font (size 1.27 1.27)) (hide yes)))
+    (property "Purchase" "C5124634" (at 59.69 149.86 0) (show_name no) (effects (font (size 1.27 1.27)) (hide yes)))
+    (property "LCSC" "C5124634" (at 59.69 149.86 0) (show_name no) (effects (font (size 1.27 1.27)) (hide yes)))
     (property "Block" "BASE" (at 59.69 149.86 0) (show_name no) (effects (font (size 1.27 1.27)) (hide yes)))
     (pin "1")
@@
     (instances (project "class-board" (path "/21416d14-3056-576f-bbf8-3b43eaeb7e71/4198837a-1c2a-56d0-94fc-14c5f2abeec5" (reference "#PWR6020") (unit 1))))
   )
-  (symbol (lib_id "class_board:HDR_2x20_MALE") (at 190.5 149.86 0) (unit 1)
+  (symbol (lib_id "class_board:HDR_2x20_FEMALE") (at 190.5 149.86 0) (unit 1)
     (exclude_from_sim no) (in_bom no) (on_board yes) (dnp no) (fields_autoplaced yes)
     (property "Reference" "J7" (at 186.69 122.428 0) (show_name no) (effects (font (size 1.27 1.27)) (justify left bottom)))
-    (property "Value" "Panel link 2x20 male" (at 186.69 177.292 0) (show_name no) (effects (font (size 1.27 1.27)) (justify left top)))
-    (property "Footprint" "Connector_PinHeader_2.54mm:PinHeader_2x20_P2.54mm_Vertical" (at 190.5 149.86 0) (show_name no) (effects (font (size 1.27 1.27)) (hide yes)))
-    (property "Datasheet" "https://www.lcsc.com/product-detail/C5224014.html" (at 190.5 149.86 0) (show_name no) (effects (font (size 1.27 1.27)) (hide yes)))
-    (property "Description" "2x20 straight male pin header, 2.54 mm, KiCad standard footprint. Bottom side of the main board, hand-soldered from the top; mates the panel's female headers." (at 190.5 149.86 0) (show_name no) (effects (font (size 1.27 1.27)) (hide yes)))
+    (property "Value" "Panel link 2x20 female" (at 186.69 177.292 0) (show_name no) (effects (font (size 1.27 1.27)) (justify left top)))
+    (property "Footprint" "Connector_PinSocket_2.54mm:PinSocket_2x20_P2.54mm_Vertical" (at 190.5 149.86 0) (show_name no) (effects (font (size 1.27 1.27)) (hide yes)))
+    (property "Datasheet" "https://www.lcsc.com/product-detail/C5124634.html" (at 190.5 149.86 0) (show_name no) (effects (font (size 1.27 1.27)) (hide yes)))
+    (property "Description" "2x20 straight female header 8.5 mm, 2.54 mm, KiCad standard footprint. Panel inner face, hand-soldered; mates the main board's male headers." (at 190.5 149.86 0) (show_name no) (effects (font (size 1.27 1.27)) (hide yes)))
     (property "Assembly" "hand" (at 190.5 149.86 0) (show_name no) (effects (font (size 1.27 1.27)) (hide yes)))
-    (property "MPN" "PZ2.54-2*20" (at 190.5 149.86 0) (show_name no) (effects (font (size 1.27 1.27)) (hide yes)))
-    (property "Manufacturer" "ZHOURI" (at 190.5 149.86 0) (show_name no) (effects (font (size 1.27 1.27)) (hide yes)))
-    (property "Purchase" "C5224014" (at 190.5 149.86 0) (show_name no) (effects (font (size 1.27 1.27)) (hide yes)))
-    (property "LCSC" "C5224014" (at 190.5 149.86 0) (show_name no) (effects (font (size 1.27 1.27)) (hide yes)))
+    (property "MPN" "2.54-2*20P (8.5 mm)" (at 190.5 149.86 0) (show_name no) (effects (font (size 1.27 1.27)) (hide yes)))
+    (property "Manufacturer" "BOOMELE" (at 190.5 149.86 0) (show_name no) (effects (font (size 1.27 1.27)) (hide yes)))
+    (property "Purchase" "C5124634" (at 190.5 149.86 0) (show_name no) (effects (font (size 1.27 1.27)) (hide yes)))
+    (property "LCSC" "C5124634" (at 190.5 149.86 0) (show_name no) (effects (font (size 1.27 1.27)) (hide yes)))
     (property "Block" "BASE" (at 190.5 149.86 0) (show_name no) (effects (font (size 1.27 1.27)) (hide yes)))
     (pin "1")
@@
     (instances (project "class-board" (path "/21416d14-3056-576f-bbf8-3b43eaeb7e71/4198837a-1c2a-56d0-94fc-14c5f2abeec5" (reference "#PWR6042") (unit 1))))
   )
-  (symbol (lib_id "class_board:HDR_2x20_MALE") (at 320.04 149.86 0) (unit 1)
+  (symbol (lib_id "class_board:HDR_2x20_FEMALE") (at 320.04 149.86 0) (unit 1)
     (exclude_from_sim no) (in_bom no) (on_board yes) (dnp no) (fields_autoplaced yes)
     (property "Reference" "J8" (at 316.23 122.428 0) (show_name no) (effects (font (size 1.27 1.27)) (justify left bottom)))
-    (property "Value" "Panel link 2x20 male" (at 316.23 177.292 0) (show_name no) (effects (font (size 1.27 1.27)) (justify left top)))
-    (property "Footprint" "Connector_PinHeader_2.54mm:PinHeader_2x20_P2.54mm_Vertical" (at 320.04 149.86 0) (show_name no) (effects (font (size 1.27 1.27)) (hide yes)))
-    (property "Datasheet" "https://www.lcsc.com/product-detail/C5224014.html" (at 320.04 149.86 0) (show_name no) (effects (font (size 1.27 1.27)) (hide yes)))
-    (property "Description" "2x20 straight male pin header, 2.54 mm, KiCad standard footprint. Bottom side of the main board, hand-soldered from the top; mates the panel's female headers." (at 320.04 149.86 0) (show_name no) (effects (font (size 1.27 1.27)) (hide yes)))
+    (property "Value" "Panel link 2x20 female" (at 316.23 177.292 0) (show_name no) (effects (font (size 1.27 1.27)) (justify left top)))
+    (property "Footprint" "Connector_PinSocket_2.54mm:PinSocket_2x20_P2.54mm_Vertical" (at 320.04 149.86 0) (show_name no) (effects (font (size 1.27 1.27)) (hide yes)))
+    (property "Datasheet" "https://www.lcsc.com/product-detail/C5124634.html" (at 320.04 149.86 0) (show_name no) (effects (font (size 1.27 1.27)) (hide yes)))
+    (property "Description" "2x20 straight female header 8.5 mm, 2.54 mm, KiCad standard footprint. Panel inner face, hand-soldered; mates the main board's male headers." (at 320.04 149.86 0) (show_name no) (effects (font (size 1.27 1.27)) (hide yes)))
     (property "Assembly" "hand" (at 320.04 149.86 0) (show_name no) (effects (font (size 1.27 1.27)) (hide yes)))
-    (property "MPN" "PZ2.54-2*20" (at 320.04 149.86 0) (show_name no) (effects (font (size 1.27 1.27)) (hide yes)))
-    (property "Manufacturer" "ZHOURI" (at 320.04 149.86 0) (show_name no) (effects (font (size 1.27 1.27)) (hide yes)))
-    (property "Purchase" "C5224014" (at 320.04 149.86 0) (show_name no) (effects (font (size 1.27 1.27)) (hide yes)))
-    (property "LCSC" "C5224014" (at 320.04 149.86 0) (show_name no) (effects (font (size 1.27 1.27)) (hide yes)))
+    (property "MPN" "2.54-2*20P (8.5 mm)" (at 320.04 149.86 0) (show_name no) (effects (font (size 1.27 1.27)) (hide yes)))
+    (property "Manufacturer" "BOOMELE" (at 320.04 149.86 0) (show_name no) (effects (font (size 1.27 1.27)) (hide yes)))
+    (property "Purchase" "C5124634" (at 320.04 149.86 0) (show_name no) (effects (font (size 1.27 1.27)) (hide yes)))
+    (property "LCSC" "C5124634" (at 320.04 149.86 0) (show_name no) (effects (font (size 1.27 1.27)) (hide yes)))
     (property "Block" "BASE" (at 320.04 149.86 0) (show_name no) (effects (font (size 1.27 1.27)) (hide yes)))
     (pin "1")

Commit message: Schematic spacing rework: all nine sheets checker-clean, netlist fixes (LM66100 inputs off GND, TCXO divider joined), arrow rails, A2 for b5/c_switch/nmr_tx/nmr_rx; sch_check.py + net_diff.py; renders in docs/sch
Co-Authored-By: Claude Fable 5.1 <noreply@anthropic.com>
Other:
- note added: "LED_PWR is +3V3 (always on; the LED series resistor sits on the panel). LED_WIFI / LED_ACT come from GPIO43 / GPIO44 through JP1 / JP2 (base sheet). GPIO4/6/7/15/43/44 on J8 are the same nets as on the expansion header J5. TX is on two pins (19 and 21) so the"
- note added: "Odd pins = row 1 (signal), even pins = row 2 (return): every signal pin has its return, AGND or GND, on the adjacent even pin. The whole even row of a header is one net, so it is drawn as one comb with a single symbol. J6 carries the analog signals (nearest"
- note added: "The panel stacks flat on the BACK of the main board (Decision #45). J6/J7/J8 are mounted on the BOTTOM side of the main board and hand-soldered from the top; they mate the panel's three female headers. Positions along the 180 mm edge: x ~ 12 (J6), x ~ 90 (J7),"
- note added: "coil current has two paths."
- note added: "the panel SMAs), J7 the digital ones, J8 the rails, the free GPIO, the seven module outputs MODULE OUT 1..7 and the two isolated-input returns OPTO_IN1/2."
- note added: "x ~ 168 (J8) mm."
- note removed: "LED_PWR is +3V3 (always on; the LED series resistor sits on the panel). LED_WIFI / LED_ACT come from GPIO43 / GPIO44 through JP1 / JP2 (base sheet). GPIO4/6/7/15/43/44 on J8 are the same nets as on the expansion header J5. TX is on two pins (19 and 21) so the coil current has two paths."
- note removed: "Odd pins = row 1 (signal), even pins = row 2 (return): every signal pin has its return, AGND or GND, on the adjacent even pin. J6 carries the analog signals (nearest the panel SMAs), J7 the digital ones, J8 the rails, the free GPIO, the seven module outputs MODULE OUT 1..7 and the two isolated-input returns OPTO_IN1/2."
- note removed: "The panel stacks flat on the BACK of the main board (Decision #45). J6/J7/J8 are mounted on the BOTTOM side of the main board and hand-soldered from the top; they mate the panel's three female headers. Positions along the 180 mm edge: x ~ 12 (J6), x ~ 90 (J7), x ~ 168 (J8) mm."
