File: hardware/sheets/front_panel_link.kicad_sch (KiCad schematic)
At the start: 3 parts, among them J6 Panel link 2x20 female, J7 Panel link 2x20 female, J8 Panel link 2x20 female

Commit message: Boards as hand-reworked by the instructor 2026-09-18 (Decision #66): three 2x20 links re-placed, jumpers -> headers, TCXO removed, 16 SMA; layout and routing in progress; review in the course repo notes
Co-Authored-By: Claude Fable 5.1 <noreply@anthropic.com>
Parts:
- removed J6, J7, J8: Panel link 2x20 female, Connector_PinSocket_2.54mm:PinSocket_2x20_P2.54mm_Vertical, symbol class_board:HDR_2x20_FEMALE
Connections:
- no-connect marks 11 -> 0
Other:
- note removed: "+5V_RAW GND +5V_RAW GND +3V3 GND"
- note removed: "1-6"
- note removed: "13-18"
- note removed: "19-24"
- note removed: "25-30"
- note removed: "31-36"
- note removed: "37-40"
- note removed: "7-12"
- note removed: "AI1 AGND AI2 AGND AI3 AGND"
- note removed: "AI4 AGND AI5 AGND AI6 AGND"
- note removed: "AI7 AGND AI8 AGND RX AGND"
- note removed: "AO1 AGND AO2 AGND spare AGND"
- note removed: "FASTTTL2 GND TRIG_5V GND I2C_SDA GND"
- note removed: "GPIO15 GND GPIO43 GND GPIO44 GND"
- note removed: "GPIO4 GND GPIO6 GND GPIO7 GND"
- note removed: "I2C_SCL GND +3V3 GND LED_PWR GND"
- note removed: "J6 - analog, at x = 12 mm on the bottom side"
- note removed: "J6 pin table"
- note removed: "J7 - digital, at x = 90 mm on the bottom side"
- note removed: "J7 pin table"
- note removed: "J8 - rails, GPIO, module outputs, at x = 168 mm on the bottom side"
- note removed: "J8 pin table"
- note removed: "LED_WIFI GND LED_ACT GND spare GND"
- note removed: "MOD1 GND MOD2 GND MOD3 GND"
- note removed: "MOD4 GND MOD5 GND MOD6 GND"
- note removed: "MOD7 GND spare GND OPTO_IN1 GND"
- note removed: "OPTO_IN2 GND spare GND"
- note removed: "Pins"
- note removed: "Signals (odd = signal, even = its return)"
- note removed: "TTL1 GND TTL2 GND TTL3 GND"
- note removed: "TTL4 GND TTL5 GND TTL6 GND"
- note removed: "TTL7 GND TTL8 GND FASTTTL1 GND"
- note removed: "TX AGND TX AGND AUX AGND"
- note removed: "spare AGND spare AGND"
- note removed: "spare AGND spare AGND spare AGND"
- note removed: "spare GND spare GND"
