File: hardware/sheets/nmr_rx.kicad_sch (KiCad schematic)
At the start: 93 parts, among them U701 SI5351A-B-GT, U702 74HC74D,653, U703 OPA1656IDR, U704 DG419DY-T1-E3, U705 OPA1612AIDR, U706 OPA1612AIDR, U901 TS5A23157DGSR, U902 TS5A23157DGSR, Y701 25 MHz

Commit message: hardware: three LCSC numbers corrected (C701/C702 3.9 pF -> C519107, R722 9.1 k -> C23260, 100 uF 35 V -> C37309); library, sheets and gapped copies regenerated, ERC 0 errors; PROTOCOL: hbridge/polarizer commands, presence flags in info
Found by bom/verification/jlc_check.py in the course repo (full-BOM JLC check).

Co-Authored-By: Claude Fable 5.1 <noreply@anthropic.com>
Parts:
- C701, C702: symbol class_board:C0603_100nF -> class_board:C0603_4pF; JLC_CLASS Basic -> Extended; LCSC C14663 -> C519107; MPN CC0603KRX7R9BB104 -> CC0603BRNPO9BN3R9; Manufacturer Yageo -> YAGEO
- R722: symbol class_board:R0603_10k -> class_board:R0603_9R09k; LCSC C25804 -> C23260; MPN 0603WAF1002T5E -> 0603WAF9101T5E
Changed lines of the file:
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@@
     (instances (project "class-board" (path "/21416d14-3056-576f-bbf8-3b43eaeb7e71/27fece37-25e5-55f8-9b4c-3407e1c1ba01" (reference "TP701") (unit 1))))
   )
-  (symbol (lib_id "class_board:C0603_100nF") (at 350.52 59.69 90) (unit 1)
+  (symbol (lib_id "class_board:C0603_4pF") (at 350.52 59.69 90) (unit 1)
     (exclude_from_sim no) (in_bom yes) (on_board yes) (dnp no) (fields_autoplaced yes)
     (property "Reference" "C701" (at 346.71 56.388 0) (show_name no) (effects (font (size 1.27 1.27)) (justify left bottom)))
     (property "Value" "3.9pF" (at 346.71 62.992 0) (show_name no) (effects (font (size 1.27 1.27)) (justify left top)))
     (property "Footprint" "class_board:C0603" (at 350.52 59.69 0) (show_name no) (effects (font (size 1.27 1.27)) (hide yes)))
-    (property "Datasheet" "https://www.lcsc.com/product-detail/C14663.html" (at 350.52 59.69 0) (show_name no) (effects (font (size 1.27 1.27)) (hide yes)))
-    (property "Description" "Capacitor 100 nF 50 V X7R 0603 (Yageo CC0603KRX7R9BB104)" (at 350.52 59.69 0) (show_name no) (effects (font (size 1.27 1.27)) (hide yes)))
-    (property "LCSC" "C14663" (at 350.52 59.69 0) (show_name no) (effects (font (size 1.27 1.27)) (hide yes)))
-    (property "JLC_CLASS" "Basic" (at 350.52 59.69 0) (show_name no) (effects (font (size 1.27 1.27)) (hide yes)))
-    (property "MPN" "CC0603KRX7R9BB104" (at 350.52 59.69 0) (show_name no) (effects (font (size 1.27 1.27)) (hide yes)))
-    (property "Manufacturer" "Yageo" (at 350.52 59.69 0) (show_name no) (effects (font (size 1.27 1.27)) (hide yes)))
+    (property "Datasheet" "https://www.lcsc.com/product-detail/C519107.html" (at 350.52 59.69 0) (show_name no) (effects (font (size 1.27 1.27)) (hide yes)))
+    (property "Description" "Capacitor 3.9 pF 50 V NP0 0603 (Si5351 crystal load; circuits note 1.2 asks for 4 pF - 3.9 pF is the stocked NP0 value, XTAL_CL = 10 pF unchanged) (YAGEO CC0603BRNPO9BN3R9)" (at 350.52 59.69 0) (show_name no) (effects (font (size 1.27 1.27)) (hide yes)))
+    (property "LCSC" "C519107" (at 350.52 59.69 0) (show_name no) (effects (font (size 1.27 1.27)) (hide yes)))
+    (property "JLC_CLASS" "Extended" (at 350.52 59.69 0) (show_name no) (effects (font (size 1.27 1.27)) (hide yes)))
+    (property "MPN" "CC0603BRNPO9BN3R9" (at 350.52 59.69 0) (show_name no) (effects (font (size 1.27 1.27)) (hide yes)))
+    (property "Manufacturer" "YAGEO" (at 350.52 59.69 0) (show_name no) (effects (font (size 1.27 1.27)) (hide yes)))
     (property "Block" "NMR_RX" (at 350.52 59.69 0) (show_name no) (effects (font (size 1.27 1.27)) (hide yes)))
     (pin "1")
@@
     (instances (project "class-board" (path "/21416d14-3056-576f-bbf8-3b43eaeb7e71/27fece37-25e5-55f8-9b4c-3407e1c1ba01" (reference "#PWR7013") (unit 1))))
   )
-  (symbol (lib_id "class_board:C0603_100nF") (at 350.52 68.58 90) (unit 1)
+  (symbol (lib_id "class_board:C0603_4pF") (at 350.52 68.58 90) (unit 1)
     (exclude_from_sim no) (in_bom yes) (on_board yes) (dnp no) (fields_autoplaced yes)
     (property "Reference" "C702" (at 346.71 65.278 0) (show_name no) (effects (font (size 1.27 1.27)) (justify left bottom)))
     (property "Value" "3.9pF" (at 346.71 71.882 0) (show_name no) (effects (font (size 1.27 1.27)) (justify left top)))
     (property "Footprint" "class_board:C0603" (at 350.52 68.58 0) (show_name no) (effects (font (size 1.27 1.27)) (hide yes)))
-    (property "Datasheet" "https://www.lcsc.com/product-detail/C14663.html" (at 350.52 68.58 0) (show_name no) (effects (font (size 1.27 1.27)) (hide yes)))
-    (property "Description" "Capacitor 100 nF 50 V X7R 0603 (Yageo CC0603KRX7R9BB104)" (at 350.52 68.58 0) (show_name no) (effects (font (size 1.27 1.27)) (hide yes)))
-    (property "LCSC" "C14663" (at 350.52 68.58 0) (show_name no) (effects (font (size 1.27 1.27)) (hide yes)))
-    (property "JLC_CLASS" "Basic" (at 350.52 68.58 0) (show_name no) (effects (font (size 1.27 1.27)) (hide yes)))
-    (property "MPN" "CC0603KRX7R9BB104" (at 350.52 68.58 0) (show_name no) (effects (font (size 1.27 1.27)) (hide yes)))
-    (property "Manufacturer" "Yageo" (at 350.52 68.58 0) (show_name no) (effects (font (size 1.27 1.27)) (hide yes)))
+    (property "Datasheet" "https://www.lcsc.com/product-detail/C519107.html" (at 350.52 68.58 0) (show_name no) (effects (font (size 1.27 1.27)) (hide yes)))
+    (property "Description" "Capacitor 3.9 pF 50 V NP0 0603 (Si5351 crystal load; circuits note 1.2 asks for 4 pF - 3.9 pF is the stocked NP0 value, XTAL_CL = 10 pF unchanged) (YAGEO CC0603BRNPO9BN3R9)" (at 350.52 68.58 0) (show_name no) (effects (font (size 1.27 1.27)) (hide yes)))
+    (property "LCSC" "C519107" (at 350.52 68.58 0) (show_name no) (effects (font (size 1.27 1.27)) (hide yes)))
+    (property "JLC_CLASS" "Extended" (at 350.52 68.58 0) (show_name no) (effects (font (size 1.27 1.27)) (hide yes)))
+    (property "MPN" "CC0603BRNPO9BN3R9" (at 350.52 68.58 0) (show_name no) (effects (font (size 1.27 1.27)) (hide yes)))
+    (property "Manufacturer" "YAGEO" (at 350.52 68.58 0) (show_name no) (effects (font (size 1.27 1.27)) (hide yes)))
     (property "Block" "NMR_RX" (at 350.52 68.58 0) (show_name no) (effects (font (size 1.27 1.27)) (hide yes)))
     (pin "1")
@@
     (instances (project "class-board" (path "/21416d14-3056-576f-bbf8-3b43eaeb7e71/27fece37-25e5-55f8-9b4c-3407e1c1ba01" (reference "#PWR7071") (unit 1))))
   )
-  (symbol (lib_id "class_board:R0603_10k") (at 406.4 215.9 90) (unit 1)
+  (symbol (lib_id "class_board:R0603_9R09k") (at 406.4 215.9 90) (unit 1)
     (exclude_from_sim no) (in_bom yes) (on_board yes) (dnp no) (fields_autoplaced yes)
     (property "Reference" "R722" (at 402.59 212.598 0) (show_name no) (effects (font (size 1.27 1.27)) (justify left bottom)))
     (property "Value" "9.1k" (at 402.59 219.202 0) (show_name no) (effects (font (size 1.27 1.27)) (justify left top)))
     (property "Footprint" "class_board:R0603" (at 406.4 215.9 0) (show_name no) (effects (font (size 1.27 1.27)) (hide yes)))
-    (property "Datasheet" "https://www.lcsc.com/product-detail/C25804.html" (at 406.4 215.9 0) (show_name no) (effects (font (size 1.27 1.27)) (hide yes)))
-    (property "Description" "Resistor 10k 1% 0603 100 mW (Uniroyal 0603WAF1002T5E)" (at 406.4 215.9 0) (show_name no) (effects (font (size 1.27 1.27)) (hide yes)))
-    (property "LCSC" "C25804" (at 406.4 215.9 0) (show_name no) (effects (font (size 1.27 1.27)) (hide yes)))
+    (property "Datasheet" "https://www.lcsc.com/product-detail/C23260.html" (at 406.4 215.9 0) (show_name no) (effects (font (size 1.27 1.27)) (hide yes)))
+    (property "Description" "Resistor 9.1 kOhm 1% 0603 fitted where the design says 9.09 kOhm (stage-2 gain 10.01 instead of 10.00). The exact E96 9.09 kOhm is C23125 (Extended, 93 k stock) if the ratio must be exact (UNI-ROYAL 0603WAF9101T5E)" (at 406.4 215.9 0) (show_name no) (effects (font (size 1.27 1.27)) (hide yes)))
+    (property "LCSC" "C23260" (at 406.4 215.9 0) (show_name no) (effects (font (size 1.27 1.27)) (hide yes)))
     (property "JLC_CLASS" "Basic" (at 406.4 215.9 0) (show_name no) (effects (font (size 1.27 1.27)) (hide yes)))
-    (property "MPN" "0603WAF1002T5E" (at 406.4 215.9 0) (show_name no) (effects (font (size 1.27 1.27)) (hide yes)))
+    (property "MPN" "0603WAF9101T5E" (at 406.4 215.9 0) (show_name no) (effects (font (size 1.27 1.27)) (hide yes)))
     (property "Manufacturer" "UNI-ROYAL" (at 406.4 215.9 0) (show_name no) (effects (font (size 1.27 1.27)) (hide yes)))
     (property "Block" "NMR_RX" (at 406.4 215.9 0) (show_name no) (effects (font (size 1.27 1.27)) (hide yes)))

Commit message: hardware: chip resistors and ceramic capacitors on KiCad standard footprints (Decision #47); schematic, library and gapped copies regenerated, ERC 0 errors
Co-Authored-By: Claude Fable 5.1 <noreply@anthropic.com>
Parts:
- C701, C702, C703, C704, C705, C706, C707, C710, C711, C712, C720, C721, C722, C723, C724, C725, C901, C902, C903, C904, C906, C907, C908, C910, C911, C912, C913, C914, C915, C916, C917, C918, C919: footprint class_board:C0603 -> Capacitor_SMD:C_0603_1608Metric
- C726, C727, C905: footprint class_board:C0805 -> Capacitor_SMD:C_0805_2012Metric
- R701, R702, R703, R704, R705, R706, R710, R711, R712, R713, R714, R721, R722, R723, R724, R901, R902, R903, R904, R905, R906, R907, R908, R909, R910, R911, R912, R913, R914, R915, R916, R917, R918, R919, R923, R924: footprint class_board:R0603 -> Resistor_SMD:R_0603_1608Metric

Commit message: Schematic spacing rework: all nine sheets checker-clean, netlist fixes (LM66100 inputs off GND, TCXO divider joined), arrow rails, A2 for b5/c_switch/nmr_tx/nmr_rx; sch_check.py + net_diff.py; renders in docs/sch
Co-Authored-By: Claude Fable 5.1 <noreply@anthropic.com>
Other:
- note added: "D905-D908: BAV99 clamps to AGND / +3V3A — the LNA runs on +-12 V"
- note added: "and must not push the switch inputs outside 0..3.3 V."
- note removed: "D905-D908: BAV99 clamps to AGND / +3V3A — the LNA runs on +-12 V and must not push the switch inputs outside 0..3.3 V."
- moved on the sheet: C701, C702, C703, C704, C705, C706, C707, C710, C711, C712, C720, C721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

Commit message: Boards as hand-reworked by the instructor 2026-09-18 (Decision #66): three 2x20 links re-placed, jumpers -> headers, TCXO removed, 16 SMA; layout and routing in progress; review in the course repo notes
Co-Authored-By: Claude Fable 5.1 <noreply@anthropic.com>
Parts:
- removed JP701: AUX -> LNA (open), class_board:SolderJumper-3_P1.3mm_Open_RoundedPad1.0x1.5mm, symbol class_board:SolderJumper_3_Open
- removed JP702: G=101 / G=11, class_board:SolderJumper-3_P1.3mm_Bridged12_RoundedPad1.0x1.5mm, symbol class_board:SolderJumper_3_Bridged12
- removed JP703: open = G 1, class_board:SolderJumper-2_P1.3mm_Bridged_RoundedPad1.0x1.5mm, symbol class_board:SolderJumper_2_Bridged
- added J3, J9: C2937625_-_Conn_01x03, DDS_Library:C2937625-HDR-TH_3P-P2.54-V-M, symbol DDS_Library:C2937625_-_Conn_01x03
- added R715, R716: 0, Resistor_SMD:R_0805_2012Metric_Pad1.20x1.40mm_HandSolder, symbol class_board:R0603_100
Connections:
- net AGND: now also C710.1, C711.1, C712.1, R711.1, J9.1 (Pin_1), R716.1; no longer C710.2, C711.2, C712.2, R711.2
- net AUX: now also R715.2
- net DIF_Q_P: now also R923.1; no longer R923.2
- net IF_IPF: now also C910.2; no longer C910.1
- net IF_QPF: now also C911.2, R923.2; no longer C911.1, R923.1
- net LNA_FB1: now also J3.2 (Pin_2)
- net RX: now also C710.2, C711.2, C712.2, R710.2, R711.2; no longer C710.1, C711.1, C712.1, R710.1, R711.1
- net RX_IN: now also R710.1, R715.1, R716.2; no longer R710.2
- net ST2_GAIN: now also J9.2 (Pin_2)
- net V_MID: now also C910.1, C911.1; no longer C910.2, C911.2
- net CLK2_TP: no longer names the net of R705.2, TP701.1
- net JP702A: no longer names the net of R712.2
- net JP702A: now also J3.1 (Pin_1)
- net JP702B: no longer names the net of R714.2
- net JP702B: now also J3.3 (Pin_3)
- net SI_CLK0: no longer names the net of R703.1, U701.10 (CLK0)
- net SI_CLK1: no longer names the net of R704.1, U701.9 (CLK1)
- net SI_CLK2: no longer names the net of R705.1, U701.6 (CLK2)
- no-connect marks 1 -> 2
Other:
- note added: "G=101"
- note added: "G=11"
- moved on the sheet: C701, C702, C703, C704, C705, C706, C720, C721, C911, C912, C913, C914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

Commit message: WIP main board routing + schematic (instructor), 2026-09-21 05:04
Co-Authored-By: Claude Fable 5.1 <noreply@anthropic.com>
Parts:
- R715, R716: value 0 -> 0R
Changed lines of the file:
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@@
 			)
 		)
-		(property "Value" "0"
+		(property "Value" "0R"
 			(at 153.162 199.644 0)
 			(show_name no)
@@
 			)
 		)
-		(property "Value" "0"
+		(property "Value" "0R"
 			(at 153.162 216.154 0)
 			(show_name no)

Commit message: hardware: board, sheets and DC jack footprint as on disk 2026-09-27 (snapshot committed by the projector-developer session, Shayne 2026-09-27)
Co-Authored-By: Claude Fable 5.1 <noreply@anthropic.com>
Parts:
- removed R701, R702: 4.7k, Resistor_SMD:R_0603_1608Metric, symbol class_board:R0603_4R7k
