File: hardware/sheets/c_switch.kicad_sch (KiCad schematic)
At the start: 30 parts, among them J901 KF301-5.0-2P, J903 KF301-5.0-2P, J905 KF301-5.0-3P, Q901 AOD4185, Q904 AOD4184A, U903 DRV8871DDAR, U904 UCC27517DBVR

Commit message: hardware: three LCSC numbers corrected (C701/C702 3.9 pF -> C519107, R722 9.1 k -> C23260, 100 uF 35 V -> C37309); library, sheets and gapped copies regenerated, ERC 0 errors; PROTOCOL: hbridge/polarizer commands, presence flags in info
Found by bom/verification/jlc_check.py in the course repo (full-BOM JLC check).

Co-Authored-By: Claude Fable 5.1 <noreply@anthropic.com>
Parts:
- C921, C940: LCSC C72479 -> C37309
Changed lines of the file:
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@@
     (property "Value" "100uF 35V" (at 130.81 99.822 0) (show_name no) (effects (font (size 1.27 1.27)) (justify left top)))
     (property "Footprint" "class_board:CAP-SMD_BD8.0-L8.3-W8.3-LS9.3-FD" (at 133.35 95.25 0) (show_name no) (effects (font (size 1.27 1.27)) (hide yes)))
-    (property "Datasheet" "https://www.lcsc.com/product-detail/C72479.html" (at 133.35 95.25 0) (show_name no) (effects (font (size 1.27 1.27)) (hide yes)))
+    (property "Datasheet" "https://www.lcsc.com/product-detail/C37309.html" (at 133.35 95.25 0) (show_name no) (effects (font (size 1.27 1.27)) (hide yes)))
     (property "Description" "Aluminium electrolytic 100 uF 35 V, SMD can 8x10 mm (ROQANG RVT1V101M0810) - +VEXT bulk; PIN 1 = +" (at 133.35 95.25 0) (show_name no) (effects (font (size 1.27 1.27)) (hide yes)))
-    (property "LCSC" "C72479" (at 133.35 95.25 0) (show_name no) (effects (font (size 1.27 1.27)) (hide yes)))
+    (property "LCSC" "C37309" (at 133.35 95.25 0) (show_name no) (effects (font (size 1.27 1.27)) (hide yes)))
     (property "JLC_CLASS" "Extended" (at 133.35 95.25 0) (show_name no) (effects (font (size 1.27 1.27)) (hide yes)))
     (property "MPN" "RVT1V101M0810" (at 133.35 95.25 0) (show_name no) (effects (font (size 1.27 1.27)) (hide yes)))
@@
     (property "Value" "100uF 35V" (at 246.38 87.122 0) (show_name no) (effects (font (size 1.27 1.27)) (justify left top)))
     (property "Footprint" "class_board:CAP-SMD_BD8.0-L8.3-W8.3-LS9.3-FD" (at 248.92 82.55 0) (show_name no) (effects (font (size 1.27 1.27)) (hide yes)))
-    (property "Datasheet" "https://www.lcsc.com/product-detail/C72479.html" (at 248.92 82.55 0) (show_name no) (effects (font (size 1.27 1.27)) (hide yes)))
+    (property "Datasheet" "https://www.lcsc.com/product-detail/C37309.html" (at 248.92 82.55 0) (show_name no) (effects (font (size 1.27 1.27)) (hide yes)))
     (property "Description" "Aluminium electrolytic 100 uF 35 V, SMD can 8x10 mm (ROQANG RVT1V101M0810) - +VEXT bulk; PIN 1 = +" (at 248.92 82.55 0) (show_name no) (effects (font (size 1.27 1.27)) (hide yes)))
-    (property "LCSC" "C72479" (at 248.92 82.55 0) (show_name no) (effects (font (size 1.27 1.27)) (hide yes)))
+    (property "LCSC" "C37309" (at 248.92 82.55 0) (show_name no) (effects (font (size 1.27 1.27)) (hide yes)))
     (property "JLC_CLASS" "Extended" (at 248.92 82.55 0) (show_name no) (effects (font (size 1.27 1.27)) (hide yes)))
     (property "MPN" "RVT1V101M0810" (at 248.92 82.55 0) (show_name no) (effects (font (size 1.27 1.27)) (hide yes)))

Commit message: hardware: chip resistors and ceramic capacitors on KiCad standard footprints (Decision #47); schematic, library and gapped copies regenerated, ERC 0 errors
Co-Authored-By: Claude Fable 5.1 <noreply@anthropic.com>
Parts:
- C920, C930, C931, C941: footprint class_board:C0603 -> Capacitor_SMD:C_0603_1608Metric
- R920, R921, R922, R930, R931, R932, R940, R941: footprint class_board:R0603 -> Resistor_SMD:R_0603_1608Metric
- R933: footprint class_board:R2512 -> Resistor_SMD:R_2512_6332Metric

Commit message: Schematic spacing rework: all nine sheets checker-clean, netlist fixes (LM66100 inputs off GND, TCXO divider joined), arrow rails, A2 for b5/c_switch/nmr_tx/nmr_rx; sch_check.py + net_diff.py; renders in docs/sch
Co-Authored-By: Claude Fable 5.1 <noreply@anthropic.com>
Other:
- note added: "Flyback (6.1), one footprint set, three stuffing options: (a) D930 SS54 freewheel, tau = L/R = 2.6 ms — fitted by default; (b) the RC snubber (the Michal route, 2.2 R 5 W + 4700 uF 50 V) over-damped at ~10 ms, +VCOIL <= 24 V — wired EXTERNALLY across J905 pins 1-2, the parts are too big for the board; (c) D934 SMBJ20A fast dump, 591 us, +VCOIL <= 12 V."
- note removed: "Flyback (6.1), one footprint set, three stuffing options: (a) D930 SS54 freewheel, tau = L/R = 2.6 ms — fitted by default; (b) the RC snubber (the Michal route, 2.2 R 5 W + 4700 uF 50 V) over-damped at ~10 ms, +VCOIL <= 24 V — wired EXTERNALLY across J905 pins 1-2, the parts are too big for the board; (c) D934 SMBJ20A fast dump, 591 us, +VCOIL <= 12 V. This board does the ADIABATIC transfer, not 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"
- moved on the sheet: C920, C921, C930, C931, C940, C941, D920, D930, D931, D932, D933, D934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

Commit message: Boards as hand-reworked by the instructor 2026-09-18 (Decision #66): three 2x20 links re-placed, jumpers -> headers, TCXO removed, 16 SMA; layout and routing in progress; review in the course repo notes
Co-Authored-By: Claude Fable 5.1 <noreply@anthropic.com>
Parts:
- removed JP904: SolderJumper_3_Bridged12, class_board:SolderJumper-3_P1.3mm_Bridged12_RoundedPad1.0x1.5mm, symbol class_board:SolderJumper_3_Bridged12
- added J12: C2937625_-_Conn_01x03, DDS_Library:C2937625-HDR-TH_3P-P2.54-V-M, symbol DDS_Library:C2937625_-_Conn_01x03
- added J13: C492401-PZ254V-11-02P, mike_JLCPCB:C492401-HDR-TH_2P-P2.54-V-M, symbol mike_JLCPCB:C492401-PZ254V-11-02P
Connections:
- net +5V_RAW: now also J12.3 (Pin_3)
- net +VEXT: now also J12.1 (Pin_1)
- net GND: now also J13.2
- net ISENSE_COIL: now also J13.1
- net VDD904: now also J12.2 (Pin_2)

Commit message: WIP main board routing + schematic (instructor), 2026-09-21 05:04
Co-Authored-By: Claude Fable 5.1 <noreply@anthropic.com>
Parts:
- R933: value 0 -> 0R
Changed lines of the file:
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@@
 			)
 		)
-		(property "Value" "0"
+		(property "Value" "0R"
 			(at 223.774 275.082 0)
 			(show_name no)

Commit message: Schematic review fixes, part 2 (Konnect): panel RX/AUX labels + SMA labels swapped to match the main board (copper unchanged); TX_VMID -> R820 47k -> TX_IN (C810 couples into TX_IN); Q901 D/S corrected + D932 to +VEXT; R950 10k Q904 gate-source; R712 permanent (J3 pin 1 tied to pin 2); U302/C308 on +5VA; panel 6N137 VCC/VE + C401/C402 on +5V_RAW; R521-R528 DIO pull-downs; front_panel_link sheet removed from the root; change notes on six sheets; panel silk: pairing labels corrected, stale J3 texts deleted, TX/RX/AUX labels fixed, OUT1..7. ERC unchanged (2 cosmetic), panel DRC 0/0; netlist diff = intended changes only
Co-Authored-By: Claude Fable 5.1 <noreply@anthropic.com>
Parts:
- added R950: 10k, Resistor_SMD:R_0603_1608Metric, symbol class_board:R0603_10k
Connections:
- net +VEXT: now also D932.3 (K), Q901.3 (S); no longer Q901.2 (D)
- net ISENSE_COIL: now also R950.2
- net VIN_F: now also Q901.2 (D); no longer D932.3 (K), Q901.3 (S)
- net at Q904.1 (G), R932.2: now also R950.1
Other:
- note added: "2026-10-01: Q901 turned so that D = VIN_F (input side) and S = +VEXT (load side); the body diode now blocks a reversed input. D932 clamps gate-to-source (+VEXT). R950 10k gate-source pull-down added to Q904. D934: mark Do Not Populate (fit ONE of D930/D934). Older notes naming NT1, JP904 and "D934 (DNP)" are stale."
- moved on the sheet: Q901
