File: hardware/sheets/c_switch.kicad_sch (KiCad schematic)
At the start: 32 parts, among them J12 C2937625_-_Conn_01x03, J13 C492401-PZ254V-11-02P, J901 KF301-5.0-2P, J903 KF301-5.0-2P, J905 KF301-5.0-3P, Q901 AOD4185, Q904 AOD4184A, U903 DRV8871DDAR, U904 UCC27517DBVR

Commit message: hardware: instructor 2026-10-01 saves synced (one GND net on both boards, PCB updated, R951-R958, headers DNP per Decision #73) + nmr_tx R808 -> TX_VMID, C813 removed, R805/R806 10 k (review B2)
Co-Authored-By: Claude Fable 5.1 <noreply@anthropic.com>
Parts:
- D934, J12: now not fitted; now left out of the parts list

Commit message: Instructor 2026-10-01 afternoon saves (after the review: Update PCB for the nmr_tx change and further sheet edits); ignore the board STEP export
Co-Authored-By: Claude Fable 5.1 <noreply@anthropic.com>
Parts:
- J12: now fitted; now in the parts list
- J13: now fitted
Changed lines of the file:
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@@
 		(body_style 1)
 		(exclude_from_sim no)
-		(in_bom no)
+		(in_bom yes)
 		(on_board yes)
 		(in_pos_files yes)
-		(dnp yes)
+		(dnp no)
 		(property "Reference" "J12"
 			(at 165.1 236.2201 90)
@@
 		(on_board yes)
 		(in_pos_files yes)
-		(dnp yes)
+		(dnp no)
 		(property "Reference" "J13"
 			(at 247.65 264.922 0)

Commit message: Boards as ordered: instructor saves 2026-10-05 04:34 (J1/R1/R2/TP1/FID3 nudged, DNP flags on D934 R715 R716 R811 R812), JLC production files 04:03/04:04
Co-Authored-By: Claude Fable 5.1 <noreply@anthropic.com>
Parts:
- D934: value SMBJ20A -> DNP-SMBJ20A
Changed lines of the file:
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@@
 			)
 		)
-		(property "Value" "SMBJ20A"
+		(property "Value" "DNP-SMBJ20A"
 			(at 247.65 242.57 90)
 			(show_name no)

Commit message: LED polarity fixed in the design (synced from the class repo main aaaec0f)
Co-Authored-By: Claude Fable 5.1 <noreply@anthropic.com>
Connections:
- net GND: now also D933.2 (K); no longer D933.1 (K)
- net at R941.2: now also D933.1 (A); no longer D933.2 (A)
