File: hardware/sheets/b3_outputs.kicad_sch (KiCad schematic)
At the start: 25 parts, among them U301 DAC8563SDGSR, U302 74HCT125PW, U303 OPA2192IDR

Commit message: hardware: chip resistors and ceramic capacitors on KiCad standard footprints (Decision #47); schematic, library and gapped copies regenerated, ERC 0 errors
Co-Authored-By: Claude Fable 5.1 <noreply@anthropic.com>
Parts:
- C301, C302, C304, C305, C308: footprint class_board:C0603 -> Capacitor_SMD:C_0603_1608Metric
- C303, C306, C307: footprint class_board:C0805 -> Capacitor_SMD:C_0805_2012Metric
- R301, R302, R303, R304, R305, R306, R307, R308, R309, R310, R311: footprint class_board:R0603 -> Resistor_SMD:R_0603_1608Metric

Commit message: Schematic spacing rework: all nine sheets checker-clean, netlist fixes (LM66100 inputs off GND, TCXO divider joined), arrow rails, A2 for b5/c_switch/nmr_tx/nmr_rx; sch_check.py + net_diff.py; renders in docs/sch
Co-Authored-By: Claude Fable 5.1 <noreply@anthropic.com>
Other:
- note added: "OPA2192 supplies +-12 V: 100 nF + 10 uF per rail to AGND"
- note removed: "OPA2192 supplies +-12 V, 100 nF + 10 uF each to AGND"
- moved on the sheet: C301, C302, C303, C304, C305, C306, C307, C308, D301, D302, R304, R305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

Commit message: WIP main board routing + schematic (instructor), 2026-09-21 05:04
Co-Authored-By: Claude Fable 5.1 <noreply@anthropic.com>
Parts:
- TP301: value TP -> VREF
Changed lines of the file:
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@@
 			)
 		)
-		(property "Value" "TP"
+		(property "Value" "VREF"
 			(at 203.2 112.776 0)
 			(show_name no)

Commit message: Schematic review fixes, part 2 (Konnect): panel RX/AUX labels + SMA labels swapped to match the main board (copper unchanged); TX_VMID -> R820 47k -> TX_IN (C810 couples into TX_IN); Q901 D/S corrected + D932 to +VEXT; R950 10k Q904 gate-source; R712 permanent (J3 pin 1 tied to pin 2); U302/C308 on +5VA; panel 6N137 VCC/VE + C401/C402 on +5V_RAW; R521-R528 DIO pull-downs; front_panel_link sheet removed from the root; change notes on six sheets; panel silk: pairing labels corrected, stale J3 texts deleted, TX/RX/AUX labels fixed, OUT1..7. ERC unchanged (2 cosmetic), panel DRC 0/0; netlist diff = intended changes only
Co-Authored-By: Claude Fable 5.1 <noreply@anthropic.com>
Connections:
- net +5V_RAW is gone; now on net +5VA: C308.1, U302.14 (VCC)
Other:
- note added: "2026-10-01: U302 (74HCT125) and C308 now run from +5VA, the DAC8563 supply, so the DAC logic inputs are never driven above AVDD or before AVDD is present."
Changed lines of the file:
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@@
 		)
 	)
+  (text "2026-10-01: U302 (74HCT125) and C308 now run from +5VA, the DAC8563 supply, so the DAC logic inputs are never driven above AVDD or before AVDD is present."
+    (at 44.45 80.01 0)
+    (effects (font (size 1.27 1.27)) (justify left bottom))
+  )
 	(symbol
 		(lib_id "class_board:C0603_1uF")
@@
 	)
 	(symbol
-		(lib_id "class_board:PWR_p5V_RAW")
+		(lib_id "class_board:PWR_p5VA")
 		(at 101.6 69.85 0)
 		(unit 1)
@@
 			)
 		)
-		(property "Value" "+5V_RAW"
+		(property "Value" "+5VA"
 			(at 101.6 66.548 0)
 			(show_name no)
@@
 	)
 	(symbol
-		(lib_id "class_board:PWR_p5V_RAW")
+		(lib_id "class_board:PWR_p5VA")
 		(at 78.74 82.55 0)
 		(unit 1)
@@
 			)
 		)
-		(property "Value" "+5V_RAW"
+		(property "Value" "+5VA"
 			(at 78.74 79.248 0)
 			(show_name no)

Commit message: hardware: instructor 2026-10-01 saves synced (one GND net on both boards, PCB updated, R951-R958, headers DNP per Decision #73) + nmr_tx R808 -> TX_VMID, C813 removed, R805/R806 10 k (review B2)
Co-Authored-By: Claude Fable 5.1 <noreply@anthropic.com>
Connections:
- net AGND is gone; now on net GND: C301.2, C302.2, C303.2, C304.2, C305.2, C306.2, C307.2, R302.1, R306.1, U301.3 (GND), U301.4 (~{LDAC})
Changed lines of the file:
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@@
 		)
 	)
+	(text "2026-10-01: U302 (74HCT125) and C308 now run from +5VA, the DAC8563 supply, so the DAC logic inputs are never driven above AVDD or before AVDD is present."
+		(exclude_from_sim no)
+		(at 44.45 80.01 0)
+		(effects
+			(font
+				(size 1.27 1.27)
+			)
+			(justify left bottom)
+		)
+	)
 	(text "Gain = 2 is the DAC default once the internal reference is enabled by firmware (reset default: reference off, gain 1). /LDAC = AGND (synchronous), /CLR pulled up to +5VA."
 		(exclude_from_sim no)
@@
 		)
 	)
-  (text "2026-10-01: U302 (74HCT125) and C308 now run from +5VA, the DAC8563 supply, so the DAC logic inputs are never driven above AVDD or before AVDD is present."
-    (at 44.45 80.01 0)
-    (effects (font (size 1.27 1.27)) (justify left bottom))
-  )
 	(symbol
 		(lib_id "class_board:C0603_1uF")
@@
 	)
 	(symbol
-		(lib_id "class_board:PWR_AGND")
+		(lib_id "class_board:PWR_GND")
 		(at 152.4 86.36 0)
 		(unit 1)
@@
 		(fields_autoplaced yes)
 		(property "Reference" "#PWR3013"
-			(at 149.86 83.058 0)
+			(at 152.4 86.36 0)
 			(hide yes)
 			(show_name no)
@@
 					(size 1.27 1.27)
 				)
-				(justify left bottom)
 			)
 		)
-		(property "Value" "AGND"
-			(at 152.4 90.17 0)
+		(property "Value" "GND"
+			(at 152.4 91.44 0)
 			(show_name no)
 			(do_not_autoplace no)
@@
 			)
 		)
-		(property "Description" "Power symbol: AGND"
+		(property "Description" "Power symbol: GND"
 			(at 152.4 86.36 0)
 			(hide yes)
@@
 	)
 	(symbol
-		(lib_id "class_board:PWR_AGND")
+		(lib_id "class_board:PWR_GND")
 		(at 165.1 125.73 0)
 		(unit 1)
@@
 		(fields_autoplaced yes)
 		(property "Reference" "#PWR3009"
-			(at 162.56 122.428 0)
+			(at 165.1 125.73 0)
 			(hide yes)
 			(show_name no)
@@
 					(size 1.27 1.27)
 				)
-				(justify left bottom)
 			)
 		)
-		(property "Value" "AGND"
-			(at 165.1 129.54 0)
+		(property "Value" "GND"
+			(at 165.1 130.81 0)
 			(show_name no)
 			(do_not_autoplace no)
@@
 			)
 		)
-		(property "Description" "Power symbol: AGND"
+		(property "Description" "Power symbol: GND"
 			(at 165.1 125.73 0)
 			(hide yes)
@@
 	)
 	(symbol
-		(lib_id "class_board:PWR_AGND")
+		(lib_id "class_board:PWR_GND")
 		(at 287.02 73.66 180)
 		(unit 1)
@@
 		(fields_autoplaced yes)
 		(property "Reference" "#PWR3015"
-			(at 284.48 70.358 0)
+			(at 287.02 73.66 0)
 			(hide yes)
 			(show_name no)
@@
 					(size 1.27 1.27)
 				)
-				(justify left bottom)
 			)
 		)
-		(property "Value" "AGND"
-			(at 287.02 68.83 0)
+		(property "Value" "GND"
+			(at 287.02 68.58 0)
 			(show_name no)
 			(do_not_autoplace no)
@@
 			)
 		)
-		(property "Description" "Power symbol: AGND"
+		(property "Description" "Power symbol: GND"
 			(at 287.02 73.66 0)
 			(hide yes)
@@
 	)
 	(symbol
-		(lib_id "class_board:PWR_AGND")
+		(lib_id "class_board:PWR_GND")
 		(at 187.96 121.92 0)
 		(unit 1)
@@
 		(fields_autoplaced yes)
 		(property "Reference" "#PWR3014"
-			(at 185.42 118.618 0)
+			(at 187.96 121.92 0)
 			(hide yes)
 			(show_name no)
@@
 					(size 1.27 1.27)
 				)
-				(justify left bottom)
 			)
 		)
-		(property "Value" "AGND"
-			(at 187.96 125.73 0)
+		(property "Value" "GND"
+			(at 187.96 127 0)
 			(show_name no)
 			(do_not_autoplace no)
@@
 			)
 		)
-		(property "Description" "Power symbol: AGND"
+		(property "Description" "Power symbol: GND"
 			(at 187.96 121.92 0)
 			(hide yes)
@@
 	)
 	(symbol
-		(lib_id "class_board:PWR_AGND")
+		(lib_id "class_board:PWR_GND")
 		(at 133.35 115.57 0)
 		(unit 1)
@@
 		(fields_autoplaced yes)
 		(property "Reference" "#PWR3006"
-			(at 130.81 112.268 0)
+			(at 133.35 115.57 0)
 			(hide yes)
 			(show_name no)
@@
 					(size 1.27 1.27)
 				)
-				(justify left bottom)
 			)
 		)
-		(property "Value" "AGND"
-			(at 133.35 119.38 0)
+		(property "Value" "GND"
+			(at 133.35 120.65 0)
 			(show_name no)
 			(do_not_autoplace no)
@@
 			)
 		)
-		(property "Description" "Power symbol: AGND"
+		(property "Description" "Power symbol: GND"
 			(at 133.35 115.57 0)
 			(hide yes)
@@
 	)
 	(symbol
-		(lib_id "class_board:PWR_AGND")
+		(lib_id "class_board:PWR_GND")
 		(at 389.89 111.76 0)
 		(unit 1)
@@
 		(fields_autoplaced yes)
 		(property "Reference" "#PWR3024"
-			(at 387.35 108.458 0)
+			(at 389.89 111.76 0)
 			(hide yes)
 			(show_name no)
@@
 					(size 1.27 1.27)
 				)
-				(justify left bottom)
 			)
 		)
-		(property "Value" "AGND"
-			(at 389.89 115.57 0)
+		(property "Value" "GND"
+			(at 389.89 116.84 0)
 			(show_name no)
 			(do_not_autoplace no)
@@
 			)
 		)
-		(property "Description" "Power symbol: AGND"
+		(property "Description" "Power symbol: GND"
 			(at 389.89 111.76 0)
 			(hide yes)
@@
 	)
 	(symbol
-		(lib_id "class_board:PWR_AGND")
+		(lib_id "class_board:PWR_GND")
 		(at 139.7 86.36 0)
 		(unit 1)
@@
 		(fields_autoplaced yes)
 		(property "Reference" "#PWR3011"
-			(at 137.16 83.058 0)
+			(at 139.7 86.36 0)
 			(hide yes)
 			(show_name no)
@@
 					(size 1.27 1.27)
 				)
-				(justify left bottom)
 			)
 		)
-		(property "Value" "AGND"
-			(at 139.7 90.17 0)
+		(property "Value" "GND"
+			(at 139.7 91.44 0)
 			(show_name no)
 			(do_not_autoplace no)
@@
 			)
 		)
-		(property "Description" "Power symbol: AGND"
+		(property "Description" "Power symbol: GND"
 			(at 139.7 86.36 0)
 			(hide yes)
@@
 	)
 	(symbol
-		(lib_id "class_board:PWR_AGND")
+		(lib_id "class_board:PWR_GND")
 		(at 402.59 111.76 0)
 		(unit 1)
@@
 		(fields_autoplaced yes)
 		(property "Reference" "#PWR3026"
-			(at 400.05 108.458 0)
+			(at 402.59 111.76 0)
 			(hide yes)
 			(show_name no)
@@
 					(size 1.27 1.27)
 				)
-				(justify left bottom)
 			)
 		)
-		(property "Value" "AGND"
-			(at 402.59 115.57 0)
+		(property "Value" "GND"
+			(at 402.59 116.84 0)
 			(show_name no)
 			(do_not_autoplace no)
@@
 			)
 		)
-		(property "Description" "Power symbol: AGND"
+		(property "Description" "Power symbol: GND"
 			(at 402.59 111.76 0)
 			(hide yes)
@@
 	)
 	(symbol
-		(lib_id "class_board:PWR_AGND")
+		(lib_id "class_board:PWR_GND")
 		(at 402.59 147.32 0)
 		(unit 1)
@@
 		(fields_autoplaced yes)
 		(property "Reference" "#PWR3030"
-			(at 400.05 144.018 0)
+			(at 402.59 147.32 0)
 			(hide yes)
 			(show_name no)
@@
 					(size 1.27 1.27)
 				)
-				(justify left bottom)
 			)
 		)
-		(property "Value" "AGND"
-			(at 402.59 151.13 0)
+		(property "Value" "GND"
+			(at 402.59 152.4 0)
 			(show_name no)
 			(do_not_autoplace no)
@@
 			)
 		)
-		(property "Description" "Power symbol: AGND"
+		(property "Description" "Power symbol: GND"
 			(at 402.59 147.32 0)
 			(hide yes)
@@
 	)
 	(symbol
-		(lib_id "class_board:PWR_AGND")
+		(lib_id "class_board:PWR_GND")
 		(at 389.89 147.32 0)
 		(unit 1)
@@
 		(fields_autoplaced yes)
 		(property "Reference" "#PWR3028"
-			(at 387.35 144.018 0)
+			(at 389.89 147.32 0)
 			(hide yes)
 			(show_name no)
@@
 					(size 1.27 1.27)
 				)
-				(justify left bottom)
 			)
 		)
-		(property "Value" "AGND"
-			(at 389.89 151.13 0)
+		(property "Value" "GND"
+			(at 389.89 152.4 0)
 			(show_name no)
 			(do_not_autoplace no)
@@
 			)
 		)
-		(property "Description" "Power symbol: AGND"
+		(property "Description" "Power symbol: GND"
 			(at 389.89 147.32 0)
 			(hide yes)
@@
 	)
 	(symbol
-		(lib_id "class_board:PWR_AGND")
+		(lib_id "class_board:PWR_GND")
 		(at 287.02 135.89 180)
 		(unit 1)
@@
 		(fields_autoplaced yes)
 		(property "Reference" "#PWR3018"
-			(at 284.48 132.588 0)
+			(at 287.02 135.89 0)
 			(hide yes)
 			(show_name no)
@@
 					(size 1.27 1.27)
 				)
-				(justify left bottom)
 			)
 		)
-		(property "Value" "AGND"
-			(at 287.02 131.06 0)
+		(property "Value" "GND"
+			(at 287.02 130.81 0)
 			(show_name no)
 			(do_not_autoplace no)
@@
 			)
 		)
-		(property "Description" "Power symbol: AGND"
+		(property "Description" "Power symbol: GND"
 			(at 287.02 135.89 0)
 			(hide yes)
