File: hardware/sheets/nmr_tx.kicad_sch (KiCad schematic)
At the start: 46 parts, among them J802 KF301-5.0-2P, U801 AD9834BRUZ, U802 OPA564AIDWPR

Commit message: hardware: three LCSC numbers corrected (C701/C702 3.9 pF -> C519107, R722 9.1 k -> C23260, 100 uF 35 V -> C37309); library, sheets and gapped copies regenerated, ERC 0 errors; PROTOCOL: hbridge/polarizer commands, presence flags in info
Found by bom/verification/jlc_check.py in the course repo (full-BOM JLC check).

Co-Authored-By: Claude Fable 5.1 <noreply@anthropic.com>
Parts:
- C813: LCSC C72479 -> C37309
Changed lines of the file:
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@@
     (property "Value" "100uF 35V" (at 251.46 205.232 0) (show_name no) (effects (font (size 1.27 1.27)) (justify left top)))
     (property "Footprint" "class_board:CAP-SMD_BD8.0-L8.3-W8.3-LS9.3-FD" (at 254 200.66 0) (show_name no) (effects (font (size 1.27 1.27)) (hide yes)))
-    (property "Datasheet" "https://www.lcsc.com/product-detail/C72479.html" (at 254 200.66 0) (show_name no) (effects (font (size 1.27 1.27)) (hide yes)))
+    (property "Datasheet" "https://www.lcsc.com/product-detail/C37309.html" (at 254 200.66 0) (show_name no) (effects (font (size 1.27 1.27)) (hide yes)))
     (property "Description" "Aluminium electrolytic 100 uF 35 V, SMD can 8x10 mm (ROQANG RVT1V101M0810) - +VEXT bulk; PIN 1 = +" (at 254 200.66 0) (show_name no) (effects (font (size 1.27 1.27)) (hide yes)))
-    (property "LCSC" "C72479" (at 254 200.66 0) (show_name no) (effects (font (size 1.27 1.27)) (hide yes)))
+    (property "LCSC" "C37309" (at 254 200.66 0) (show_name no) (effects (font (size 1.27 1.27)) (hide yes)))
     (property "JLC_CLASS" "Extended" (at 254 200.66 0) (show_name no) (effects (font (size 1.27 1.27)) (hide yes)))
     (property "MPN" "RVT1V101M0810" (at 254 200.66 0) (show_name no) (effects (font (size 1.27 1.27)) (hide yes)))

Commit message: hardware: chip resistors and ceramic capacitors on KiCad standard footprints (Decision #47); schematic, library and gapped copies regenerated, ERC 0 errors
Co-Authored-By: Claude Fable 5.1 <noreply@anthropic.com>
Parts:
- C801, C802, C803, C804, C805, C807, C808, C809, C810, C812, C814, C816, C817: footprint class_board:C0603 -> Capacitor_SMD:C_0603_1608Metric
- C806, C811: footprint class_board:C0805 -> Capacitor_SMD:C_0805_2012Metric
- C818: footprint class_board:C1206 -> Capacitor_SMD:C_1206_3216Metric
- R801, R802, R803, R804, R805, R806, R807, R808, R809, R810, R811, R812, R815, R816, R817, R818: footprint class_board:R0603 -> Resistor_SMD:R_0603_1608Metric
- R813: footprint class_board:R2512 -> Resistor_SMD:R_2512_6332Metric
- R814: footprint class_board:R0805 -> Resistor_SMD:R_0805_2012Metric

Commit message: hardware: panel stacked on the back (180 x 100, three 2x20 headers, 17 SMA, TTL strip, TX terminal, Qwiic); TTL/fast/TX-coil/Qwiic connectors leave the main board; mains-safe relay channels (JQC-3FF 10 A, MAINS net class + DRC rules); library, sheets, gapped copies, docs regenerated; ERC 0 errors
Decisions #45-#50 in the course repo. The main-board PCB is unchanged: Update PCB from Schematic, header placement, relay re-spacing and connector rotation are the instructor's GUI steps on the master.

Co-Authored-By: Claude Fable 5.1 <noreply@anthropic.com>
Parts:
- removed J802: KF301-5.0-2P, class_board:CONN-TH_P5.00_KF301-5.0-2P, symbol class_board:KF301-5.0-2P
Other:
- note added: "-> the TX SMA and the 2P screw terminal on the panel. Route TX and its return as a close pair,"
- note added: "TX leaves this sheet as a global label -> panel link J6 pins 19 and 21 (AGND on 20 and 22)"
- note added: "loop area < 1 cm2; up to 1 A of coil current must never share copper with the receiver pour."
- note removed: "TX leaves on the front-panel link (pin 39 -> panel SMA J801) and on J802 KF301-5.0-2P at the"
- note removed: "board edge (pin 1 = TX, pin 2 = GND). Route TX and its return as a close pair, loop area < 1 cm2;"
- note removed: "up to 1 A of coil current must never share copper with the receiver pour (re-spec 8.2)."
Changed lines of the file:
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@@
   (junction (at 358.14 123.19) (diameter 0) (color 0 0 0 0))
   (junction (at 372.11 110.49) (diameter 0) (color 0 0 0 0))
-  (junction (at 372.11 146.05) (diameter 0) (color 0 0 0 0))
   (no_connect (at 144.78 114.3))
   (no_connect (at 266.7 133.35))
@@
   (wire (pts (xy 372.11 102.87) (xy 372.11 100.33)) (stroke (width 0) (type default)))
   (wire (pts (xy 367.03 127) (xy 367.03 146.05)) (stroke (width 0) (type default)))
-  (wire (pts (xy 367.03 146.05) (xy 381 146.05)) (stroke (width 0) (type default)))
+  (wire (pts (xy 367.03 146.05) (xy 372.11 146.05)) (stroke (width 0) (type default)))
   (wire (pts (xy 372.11 146.05) (xy 372.11 152.4)) (stroke (width 0) (type default)))
-  (wire (pts (xy 381 143.51) (xy 375.92 143.51)) (stroke (width 0) (type default)))
   (text "NMR TX (section B) — AD9834 DDS + reconstruction filter + OPA564 power stage -> TX" (exclude_from_sim no) (at 12.7 14 0) (effects (font (size 3 3) (bold yes)) (justify left bottom)))
   (text "DDS: AD9834BRUZ, MCLK = CLK0_MCLK = 50.000 MHz from the Si5351A on the RX sheet; df = f_MCLK / 2^28 = 0.186 Hz per LSB. R801 6.80 k on FS ADJUST -> I_OUT,FS = 18 x 1.20 V / 6.80 k = 3.18 mA;" (exclude_from_sim no) (at 12.7 19 0) (effects (font (size 1.5 1.5)) (justify left bottom)))
@@
   (text "spare for an external gain resistor." (exclude_from_sim no) (at 214 218.4 0) (effects (font (size 1.2 1.2)) (justify left bottom)))
   (text "-20 dB pad: 100/(910+100) = 0.099 into a high-Z load." (exclude_from_sim no) (at 303 96 0) (effects (font (size 1.2 1.2)) (justify left bottom)))
-  (text "TX leaves on the front-panel link (pin 39 -> panel SMA J801) and on J802 KF301-5.0-2P at the" (exclude_from_sim no) (at 300 195 0) (effects (font (size 1.2 1.2)) (justify left bottom)))
-  (text "board edge (pin 1 = TX, pin 2 = GND). Route TX and its return as a close pair, loop area < 1 cm2;" (exclude_from_sim no) (at 300 198.2 0) (effects (font (size 1.2 1.2)) (justify left bottom)))
-  (text "up to 1 A of coil current must never share copper with the receiver pour (re-spec 8.2)." (exclude_from_sim no) (at 300 201.4 0) (effects (font (size 1.2 1.2)) (justify left bottom)))
+  (text "TX leaves this sheet as a global label -> panel link J6 pins 19 and 21 (AGND on 20 and 22)" (exclude_from_sim no) (at 300 195 0) (effects (font (size 1.2 1.2)) (justify left bottom)))
+  (text "-> the TX SMA and the 2P screw terminal on the panel. Route TX and its return as a close pair," (exclude_from_sim no) (at 300 198.2 0) (effects (font (size 1.2 1.2)) (justify left bottom)))
+  (text "loop area < 1 cm2; up to 1 A of coil current must never share copper with the receiver pour." (exclude_from_sim no) (at 300 201.4 0) (effects (font (size 1.2 1.2)) (justify left bottom)))
   (text "Level plan from 0.636 V pp at the DDS output (re-spec 2.3). Top row = the 89.4 kHz NMR setting: +-7.95 V into 1419 R = 5.6 mA = t90 417 us." (exclude_from_sim no) (at 38.1 198 0) (effects (font (size 1.3 1.3)) (justify left bottom)))
   (text "Firmware (re-spec 9.1 / 9.3): hold DDS_RESET high while writing, B28 = 1, PIN/SW set for hardware PSELECT; the carrier free-runs and is gated ONLY by TX_EN." (exclude_from_sim no) (at 38.1 222 0) (effects (font (size 1.3 1.3)) (justify left bottom)))
@@
     (instances (project "class-board" (path "/21416d14-3056-576f-bbf8-3b43eaeb7e71/bbb6eea2-e7dc-5d96-9a3a-152d51422209" (reference "#PWR8036") (unit 1))))
   )
-  (symbol (lib_id "class_board:KF301-5.0-2P") (at 388.62 144.78 180) (unit 1)
-    (exclude_from_sim no) (in_bom yes) (on_board yes) (dnp no) (fields_autoplaced yes)
-    (property "Reference" "J802" (at 383.54 140.208 0) (show_name no) (effects (font (size 1.27 1.27)) (justify left bottom)))
-    (property "Value" "KF301-5.0-2P" (at 383.54 149.352 0) (show_name no) (effects (font (size 1.27 1.27)) (justify left top)))
-    (property "Footprint" "class_board:CONN-TH_P5.00_KF301-5.0-2P" (at 388.62 144.78 0) (show_name no) (effects (font (size 1.27 1.27)) (hide yes)))
-    (property "Datasheet" "https://www.lcsc.com/datasheet/lcsc_datasheet_2303171000_Cixi-Kefa-Elec-KF301-5-0-2P_C474881.pdf" (at 388.62 144.78 0) (show_name no) (effects (font (size 1.27 1.27)) (hide yes)))
-    (property "Description" "Screw terminal 5.0 mm 2P, 300 V 16 A" (at 388.62 144.78 0) (show_name no) (effects (font (size 1.27 1.27)) (hide yes)))
-    (property "LCSC" "C474881" (at 388.62 144.78 0) (show_name no) (effects (font (size 1.27 1.27)) (hide yes)))
-    (property "JLC_CLASS" "Extended" (at 388.62 144.78 0) (show_name no) (effects (font (size 1.27 1.27)) (hide yes)))
-    (property "MPN" "KF301-5.0-2P" (at 388.62 144.78 0) (show_name no) (effects (font (size 1.27 1.27)) (hide yes)))
-    (property "Manufacturer" "Cixi Kefa" (at 388.62 144.78 0) (show_name no) (effects (font (size 1.27 1.27)) (hide yes)))
-    (property "Block" "NMR_TX" (at 388.62 144.78 0) (show_name no) (effects (font (size 1.27 1.27)) (hide yes)))
-    (pin "1")
-    (pin "2")
-    (instances (project "class-board" (path "/21416d14-3056-576f-bbf8-3b43eaeb7e71/bbb6eea2-e7dc-5d96-9a3a-152d51422209" (reference "J802") (unit 1))))
-  )
-  (symbol (lib_id "class_board:PWR_GND") (at 375.92 143.51 270) (unit 1)
-    (exclude_from_sim no) (in_bom no) (on_board yes) (dnp no) (fields_autoplaced yes)
-    (property "Reference" "#PWR8037" (at 373.38 140.208 0) (show_name no) (effects (font (size 1.27 1.27)) (justify left bottom) (hide yes)))
-    (property "Value" "GND" (at 372.618 143.51 0) (show_name no) (effects (font (size 1.27 1.27)) (justify right)))
-    (property "Footprint" "" (at 375.92 143.51 0) (show_name no) (effects (font (size 1.27 1.27)) (hide yes)))
-    (property "Datasheet" "" (at 375.92 143.51 0) (show_name no) (effects (font (size 1.27 1.27)) (hide yes)))
-    (property "Description" "Power symbol: GND" (at 375.92 143.51 0) (show_name no) (effects (font (size 1.27 1.27)) (hide yes)))
-    (pin "1")
-    (instances (project "class-board" (path "/21416d14-3056-576f-bbf8-3b43eaeb7e71/bbb6eea2-e7dc-5d96-9a3a-152d51422209" (reference "#PWR8037") (unit 1))))
-  )
 )

Commit message: Schematic spacing rework: all nine sheets checker-clean, netlist fixes (LM66100 inputs off GND, TCXO divider joined), arrow rails, A2 for b5/c_switch/nmr_tx/nmr_rx; sch_check.py + net_diff.py; renders in docs/sch
Co-Authored-By: Claude Fable 5.1 <noreply@anthropic.com>
Other:
- note added: "Both lines go to TCA9535 spare pins P1.5 / P1.6 — global labels until the expander sheet claims them."
- note removed: "Both lines go to TCA9535 spare pins P1.5 / P1.6 — global labels until"
- note removed: "the expander sheet claims them."
- moved on the sheet: C801, C802, C803, C804, C805, C806, C807, C808, C809, C810, C811, C812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

Commit message: Boards as hand-reworked by the instructor 2026-09-18 (Decision #66): three 2x20 links re-placed, jumpers -> headers, TCXO removed, 16 SMA; layout and routing in progress; review in the course repo notes
Co-Authored-By: Claude Fable 5.1 <noreply@anthropic.com>
Parts:
- removed JP801, JP802: SolderJumper_3_Bridged12, class_board:SolderJumper-3_P1.3mm_Bridged12_RoundedPad1.0x1.5mm, symbol class_board:SolderJumper_3_Bridged12
- added J10, J11: C2937625_-_Conn_01x03, DDS_Library:C2937625-HDR-TH_3P-P2.54-V-M, symbol DDS_Library:C2937625_-_Conn_01x03
Connections:
- net TX: now also J11.2 (Pin_2)
- net TX_FB: now also J10.1 (Pin_1)
- net at R808.1: now also J10.2 (Pin_2)
- net at R815.2, R816.1: now also J11.3 (Pin_3)
- net at C818.2, R815.1: now also J11.1 (Pin_1)
Other:
- moved on the sheet: C813, R807, R808, R811, R812, R817, R818

Commit message: Schematic review fixes, part 2 (Konnect): panel RX/AUX labels + SMA labels swapped to match the main board (copper unchanged); TX_VMID -> R820 47k -> TX_IN (C810 couples into TX_IN); Q901 D/S corrected + D932 to +VEXT; R950 10k Q904 gate-source; R712 permanent (J3 pin 1 tied to pin 2); U302/C308 on +5VA; panel 6N137 VCC/VE + C401/C402 on +5V_RAW; R521-R528 DIO pull-downs; front_panel_link sheet removed from the root; change notes on six sheets; panel silk: pairing labels corrected, stale J3 texts deleted, TX/RX/AUX labels fixed, OUT1..7. ERC unchanged (2 cosmetic), panel DRC 0/0; netlist diff = intended changes only
Co-Authored-By: Claude Fable 5.1 <noreply@anthropic.com>
Parts:
- added R820: 47k, Resistor_SMD:R_0603_1608Metric, symbol Device:R
Connections:
- net TX_VMID: now also R820.1; no longer C810.2, U802.5 (+IN)
- new net TX_IN: C810.2, R820.2, U802.5 (+IN)
Other:
- note added: "2026-10-01: the bias node TX_VMID (R805/R806, C811/C812) now feeds the OPA564 +IN through R820 47k; C810 couples the DDS signal into the new node TX_IN. Before, C810 was coupled straight into the 10uF-bypassed bias node and almost no signal reached the amplifier."

Commit message: hardware: instructor 2026-10-01 saves synced (one GND net on both boards, PCB updated, R951-R958, headers DNP per Decision #73) + nmr_tx R808 -> TX_VMID, C813 removed, R805/R806 10 k (review B2)
Co-Authored-By: Claude Fable 5.1 <noreply@anthropic.com>
Parts:
- removed C813: 100uF 35V, class_board:CAP-SMD_BD8.0-L8.3-W8.3-LS9.3-FD, symbol class_board:CP_100uF_35V
- J10, J11: now not fitted; now left out of the parts list
- R805, R806: value 100k -> 10k; symbol class_board:R0603_100k -> class_board:R0603_10k; LCSC C25803 -> C25804
Connections:
- net AGND is gone; now on net GND: C801.2, C802.2, C803.2, C804.2, C806.2, C807.2, C808.2, C809.2, R801.2, R802.2, R803.2, R804.2, R817.2, R818.2, U801.18 (AGND), U801.7 (DGND), U801.9 (FSELECT)
- net TX_VMID: now also R808.2
Other:
- note added: "G = 1 + R807/R808 = 1 + 6490/270 = 25.0 at DC too: R808 returns to TX_VMID (2026-10-01; C813 100 uF to GND removed), so -IN keeps"
- note added: "J10 / R808"
- note added: "R805/R806 10 k (were 100 k) stiffen the bias node. J10 1-2 fits the gain leg (open = unity gain for bring-up); pad 3 is a spare."
- note added: "its DC point while the amplifier is disabled between pulses (with C813 it drifted and the first pulses clipped); output = TX_VMID + 25 x V_OS."
- note removed: "G = 1 + R807/R808 = 1 + 6490/270 = 25.0. C813 blocks DC in the gain leg, so the DC gain is 1 and the output"
- note removed: "JP801 / R808"
- note removed: "sits at V_mid (f_HP = 5.9 Hz). JP801 (1-2 bridged) opens the gain leg for a unity-gain bring-up; pad 3 is a"
- note removed: "spare for an external gain resistor."
