File: hardware/sheets/nmr_tx.kicad_sch (KiCad schematic)
At the start: 45 parts, among them J10 C2937625_-_Conn_01x03, J11 C2937625_-_Conn_01x03, U801 AD9834BRUZ, U802 OPA564AIDWPR

Commit message: Instructor 2026-10-01 afternoon saves (after the review: Update PCB for the nmr_tx change and further sheet edits); ignore the board STEP export
Co-Authored-By: Claude Fable 5.1 <noreply@anthropic.com>
Parts:
- J10, J11: now fitted; now in the parts list

Commit message: Final boards (2026-10-01 23:44/23:48 saves) and re-exported release STEP models
- class-board and front-panel: DNP + out-of-BOM flags on the hand-soldered connectors, panel 3D-model paths on TIGP_BOARD_LIB, schematic sheets in step
- hardware/release: class-board.step and front-panel.step re-exported from these boards (filters as before, now without --no-dnp so the hand-soldered connectors keep their bodies; panel exported directly, no path-redirect copy); the STL meshes are unchanged (same triangles and bounding boxes)
- README: export note

Co-Authored-By: Claude Fable 5.1 <noreply@anthropic.com>
Parts:
- R811, R812: now left out of the parts list
Changed lines of the file:
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@@
 		(body_style 1)
 		(exclude_from_sim no)
-		(in_bom yes)
+		(in_bom no)
 		(on_board yes)
 		(in_pos_files yes)
@@
 		(body_style 1)
 		(exclude_from_sim no)
-		(in_bom yes)
+		(in_bom no)
 		(on_board yes)
 		(in_pos_files yes)

Commit message: Boards as ordered: instructor saves 2026-10-05 04:34 (J1/R1/R2/TP1/FID3 nudged, DNP flags on D934 R715 R716 R811 R812), JLC production files 04:03/04:04
Co-Authored-By: Claude Fable 5.1 <noreply@anthropic.com>
Parts:
- R811, R812: value 10k -> DNP-10k
Changed lines of the file:
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@@
 			)
 		)
-		(property "Value" "10k"
+		(property "Value" "DNP-10k"
 			(at 425.45 206.248 0)
 			(show_name no)
@@
 			)
 		)
-		(property "Value" "10k"
+		(property "Value" "DNP-10k"
 			(at 438.15 206.248 0)
 			(show_name no)
