File: hardware/sheets/b1_inputs.kicad_sch (KiCad schematic)
At the start: 39 parts, among them J14 C2937625_-_Conn_01x03, J15 C2937625_-_Conn_01x03, J6 Panel link 2x20 female, U101 ADS8688IDBTR

Commit message: hardware: instructor 2026-10-01 saves synced (one GND net on both boards, PCB updated, R951-R958, headers DNP per Decision #73) + nmr_tx R808 -> TX_VMID, C813 removed, R805/R806 10 k (review B2)
Co-Authored-By: Claude Fable 5.1 <noreply@anthropic.com>
Parts:
- removed TP101: AGND, class_board:TestPoint_Pad_D1.5mm, symbol class_board:TestPoint
- J14, J15: now not fitted; now left out of the parts list
- J6: now not fitted
Connections:
- net AGND is gone; now on net GND: C101.2, C102.2, C103.2, C104.2, C105.2, C106.2, C111.2, C112.2, C113.2, C114.2, C115.2, C116.2, C117.2, C118.2, J6.15, J6.17, J6.19, J6.21, J6.23, J6.25, J6.27, J6.29, J6.31, J6.33, J6.35, J6.37, J6.39, U101.10 (AUX_IN), U101.11 (AUX_GND), U101.13 (AIN_6GND), U101.15 (AIN_7GND), U101.17 (AIN_0GND), U101.19 (AIN_1GND), U101.20 (AIN_2GND), U101.22 (AIN_3GND), U101.24 (AIN_4GND), U101.26 (AIN_5GND), U101.28 (AGND), U101.29 (AGND), U101.31 (AGND), U101.32 (AGND), U101.4 (~{REFSEL}), U101.6 (REFGND), U101.8 (AGND)

Commit message: Instructor 2026-10-01 afternoon saves (after the review: Update PCB for the nmr_tx change and further sheet edits); ignore the board STEP export
Co-Authored-By: Claude Fable 5.1 <noreply@anthropic.com>
Parts:
- J14, J15: now fitted; now in the parts list
Changed lines of the file:
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@@
 		(body_style 1)
 		(exclude_from_sim no)
-		(in_bom no)
+		(in_bom yes)
 		(on_board yes)
 		(in_pos_files yes)
-		(dnp yes)
+		(dnp no)
 		(property "Reference" "J14"
 			(at 231.14 187.9601 90)
@@
 		(body_style 1)
 		(exclude_from_sim no)
-		(in_bom no)
+		(in_bom yes)
 		(on_board yes)
 		(in_pos_files yes)
-		(dnp yes)
+		(dnp no)
 		(property "Reference" "J15"
 			(at 231.14 207.0101 90)

Commit message: Final boards (2026-10-01 23:44/23:48 saves) and re-exported release STEP models
- class-board and front-panel: DNP + out-of-BOM flags on the hand-soldered connectors, panel 3D-model paths on TIGP_BOARD_LIB, schematic sheets in step
- hardware/release: class-board.step and front-panel.step re-exported from these boards (filters as before, now without --no-dnp so the hand-soldered connectors keep their bodies; panel exported directly, no path-redirect copy); the STL meshes are unchanged (same triangles and bounding boxes)
- README: export note

Co-Authored-By: Claude Fable 5.1 <noreply@anthropic.com>
Parts:
- J6: now fitted; now in the parts list
Changed lines of the file:
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@@
 		(body_style 1)
 		(exclude_from_sim no)
-		(in_bom no)
+		(in_bom yes)
 		(on_board yes)
 		(in_pos_files yes)
-		(dnp yes)
+		(dnp no)
 		(property "Reference" "J6"
 			(at 147.32 100.838 0)
