File: hardware/sheets/base_mcu.kicad_sch (KiCad schematic)
At the start: 19 parts, among them J1 DevKit J1 (left row), J2 DevKit J3 (right row)

Commit message: Final boards (2026-10-01 23:44/23:48 saves) and re-exported release STEP models
- class-board and front-panel: DNP + out-of-BOM flags on the hand-soldered connectors, panel 3D-model paths on TIGP_BOARD_LIB, schematic sheets in step
- hardware/release: class-board.step and front-panel.step re-exported from these boards (filters as before, now without --no-dnp so the hand-soldered connectors keep their bodies; panel exported directly, no path-redirect copy); the STL meshes are unchanged (same triangles and bounding boxes)
- README: export note

Co-Authored-By: Claude Fable 5.1 <noreply@anthropic.com>
Parts:
- FID1, FID2, FID3, H1, H2, H3, H4: now in the parts list
- J1, J2: now fitted; now in the parts list
Changed lines of the file:
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@@
 		(body_style 1)
 		(exclude_from_sim no)
-		(in_bom no)
+		(in_bom yes)
 		(on_board yes)
 		(in_pos_files yes)
@@
 		(body_style 1)
 		(exclude_from_sim no)
-		(in_bom no)
+		(in_bom yes)
 		(on_board yes)
 		(in_pos_files yes)
@@
 		(body_style 1)
 		(exclude_from_sim no)
-		(in_bom no)
+		(in_bom yes)
 		(on_board yes)
 		(in_pos_files yes)
@@
 		(body_style 1)
 		(exclude_from_sim no)
-		(in_bom no)
+		(in_bom yes)
 		(on_board yes)
 		(in_pos_files yes)
-		(dnp yes)
+		(dnp no)
 		(fields_autoplaced yes)
 		(property "Reference" "J1"
@@
 		(body_style 1)
 		(exclude_from_sim no)
-		(in_bom no)
+		(in_bom yes)
 		(on_board yes)
 		(in_pos_files yes)
-		(dnp yes)
+		(dnp no)
 		(fields_autoplaced yes)
 		(property "Reference" "J2"
@@
 		(body_style 1)
 		(exclude_from_sim no)
-		(in_bom no)
+		(in_bom yes)
 		(on_board yes)
 		(in_pos_files yes)
@@
 		(body_style 1)
 		(exclude_from_sim no)
-		(in_bom no)
+		(in_bom yes)
 		(on_board yes)
 		(in_pos_files yes)
@@
 		(body_style 1)
 		(exclude_from_sim no)
-		(in_bom no)
+		(in_bom yes)
 		(on_board yes)
 		(in_pos_files yes)
@@
 		(body_style 1)
 		(exclude_from_sim no)
-		(in_bom no)
+		(in_bom yes)
 		(on_board yes)
 		(in_pos_files yes)
