File: hardware/sheets/b2_power.kicad_sch (KiCad schematic)
At the start: 54 parts, among them J201 USB-C 16P, J202 DC005-T20, U201 LM66100DCKR, U202 LM66100DCKR, U203 78L05G-AB3-R, U204 AMS1117-3.3

Commit message: hardware: chip resistors and ceramic capacitors on KiCad standard footprints (Decision #47); schematic, library and gapped copies regenerated, ERC 0 errors
Co-Authored-By: Claude Fable 5.1 <noreply@anthropic.com>
Parts:
- C201, C206, C207, C214: footprint class_board:C1206 -> Capacitor_SMD:C_1206_3216Metric
- C202, C208, C209, C210, C212, C215: footprint class_board:C0603 -> Capacitor_SMD:C_0603_1608Metric
- C203, C204, C211, C213, C216, C217: footprint class_board:C0805 -> Capacitor_SMD:C_0805_2012Metric
- R201, R202, R203, R204, R205, R206, R207, R208, R209, R210, R211, R212: footprint class_board:R0603 -> Resistor_SMD:R_0603_1608Metric

Commit message: Schematic spacing rework: all nine sheets checker-clean, netlist fixes (LM66100 inputs off GND, TCXO divider joined), arrow rails, A2 for b5/c_switch/nmr_tx/nmr_rx; sch_check.py + net_diff.py; renders in docs/sch
Co-Authored-By: Claude Fable 5.1 <noreply@anthropic.com>
Connections:
- net GND: no longer C203.1, C204.1, D201.1 (K), D202.1 (K), F201.2, F202.2, U201.1 (VIN), U202.1 (VIN)
- new net: C203.1, D201.1 (K), F201.2, U201.1 (VIN)
- new net: C204.1, D202.1 (K), F202.2, U202.1 (VIN)
Other:
- note added: "-12V: module #2 with +Vo on AGND; FB in the -Vo line; 3 x 2.2k bleeder (16 mA) + LED keep the 10 % minimum load"
- note removed: "-12V: module #2 with +Vo on AGND; FB in the -Vo line; 3 x 2.2k bleeder (16 mA) + LED keep the 10 % minimum load without the OPT chain"
- moved on the sheet: C201, C202, C206, C207, C208, C209, C210, C211, C212, C213, C214, C215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

Commit message: Boards as hand-reworked by the instructor 2026-09-18 (Decision #66): three 2x20 links re-placed, jumpers -> headers, TCXO removed, 16 SMA; layout and routing in progress; review in the course repo notes
Co-Authored-By: Claude Fable 5.1 <noreply@anthropic.com>
Connections:
- net USB_DN renamed USB_D_N
- net USB_DP renamed USB_D_P
Other:
- moved on the sheet: C201, C202, C213, C214, C215, D203, D204, R209, R210, U204

Commit message: WIP main board routing + schematic (instructor), 2026-09-21 05:04
Co-Authored-By: Claude Fable 5.1 <noreply@anthropic.com>
Parts:
- TP201: value TP -> 5V_RAW
- TP202: value TP -> +3V3
- TP203: value TP -> +12V
- TP204: value TP -> -12V
- TP205: value TP -> +5VA
- TP206: value TP -> AGND
Other:
- moved on the sheet: TP201
Changed lines of the file:
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@@
 	(wire
 		(pts
-			(xy 39.37 240.03) (xy 39.37 242.57)
+			(xy 39.37 238.76) (xy 39.37 242.57)
 		)
 		(stroke
@@
 			)
 		)
-		(property "Value" "TP"
+		(property "Value" "-12V"
 			(at 83.82 240.792 0)
 			(show_name no)
@@
 			)
 		)
-		(property "Value" "TP"
+		(property "Value" "+3V3"
 			(at 53.34 240.792 0)
 			(show_name no)
@@
 	(symbol
 		(lib_id "class_board:TestPoint")
-		(at 39.37 240.03 0)
+		(at 39.37 238.76 0)
 		(unit 1)
 		(body_style 1)
@@
 		(fields_autoplaced yes)
 		(property "Reference" "TP201"
-			(at 38.1 235.204 0)
+			(at 38.1 233.934 0)
 			(show_name no)
 			(do_not_autoplace no)
@@
 			)
 		)
-		(property "Value" "TP"
-			(at 38.1 240.792 0)
+		(property "Value" "5V_RAW"
+			(at 38.1 239.522 0)
 			(show_name no)
 			(do_not_autoplace no)
@@
 		)
 		(property "Footprint" "class_board:TestPoint_Pad_D1.5mm"
-			(at 39.37 240.03 0)
+			(at 39.37 238.76 0)
 			(hide yes)
 			(show_name no)
@@
 		)
 		(property "Datasheet" ""
-			(at 39.37 240.03 0)
+			(at 39.37 238.76 0)
 			(hide yes)
 			(show_name no)
@@
 		)
 		(property "Description" "Test point pad 1.5 mm"
-			(at 39.37 240.03 0)
+			(at 39.37 238.76 0)
 			(hide yes)
 			(show_name no)
@@
 		)
 		(property "Block" "B2"
-			(at 39.37 240.03 0)
+			(at 39.37 238.76 0)
 			(hide yes)
 			(show_name no)
@@
 			)
 		)
-		(property "Value" "TP"
+		(property "Value" "AGND"
 			(at 114.3 240.792 0)
 			(show_name no)
@@
 			)
 		)
-		(property "Value" "TP"
+		(property "Value" "+12V"
 			(at 68.58 240.792 0)
 			(show_name no)
@@
 			)
 		)
-		(property "Value" "TP"
+		(property "Value" "+5VA"
 			(at 99.06 240.792 0)
 			(show_name no)

Commit message: hardware: instructor 2026-10-01 saves synced (one GND net on both boards, PCB updated, R951-R958, headers DNP per Decision #73) + nmr_tx R808 -> TX_VMID, C813 removed, R805/R806 10 k (review B2)
Co-Authored-By: Claude Fable 5.1 <noreply@anthropic.com>
Parts:
- removed TP206: AGND, class_board:TestPoint_Pad_D1.5mm, symbol class_board:TestPoint
Connections:
- net AGND is gone; now on net GND: C206.2, C207.2, C208.2, C209.2, C210.2, C211.2, C212.2, D205.1 (K), D206.2 (A), PS201.4 (-VO), PS202.6 (+VO), R203.2, R204.2, R205.2, R206.2, R207.2, R208.2, U203.2 (GND)

Commit message: LED polarity fixed in the design (synced from the class repo main aaaec0f)
Co-Authored-By: Claude Fable 5.1 <noreply@anthropic.com>
Connections:
- net GND: now also D203.2 (K), D204.2 (K), D205.2 (K), D206.1 (A); no longer D203.1 (K), D204.1 (K), D205.1 (K), D206.2 (A)
- net at R209.2: now also D203.1 (A); no longer D203.2 (A)
- net at R210.2: now also D204.1 (A); no longer D204.2 (A)
- net at R211.2: now also D205.1 (A); no longer D205.2 (A)
- net at R212.2: now also D206.2 (K); no longer D206.1 (K)
