File: hardware/student/c_switch_gapped.kicad_sch (KiCad schematic)
At the start: 27 parts, among them J901 KF301-5.0-2P, J903 KF301-5.0-2P, J905 KF301-5.0-3P, Q901 AOD4185, Q904 AOD4184A, U903 DRV8871DDAR, U904 UCC27517DBVR

Commit message: hardware: three LCSC numbers corrected (C701/C702 3.9 pF -> C519107, R722 9.1 k -> C23260, 100 uF 35 V -> C37309); library, sheets and gapped copies regenerated, ERC 0 errors; PROTOCOL: hbridge/polarizer commands, presence flags in info
Found by bom/verification/jlc_check.py in the course repo (full-BOM JLC check).

Co-Authored-By: Claude Fable 5.1 <noreply@anthropic.com>
Parts:
- C921, C940: LCSC C72479 -> C37309
Changed lines of the file:
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@@
     (property "Value" "100uF 35V" (at 130.81 99.822 0) (show_name no) (effects (font (size 1.27 1.27)) (justify left top)))
     (property "Footprint" "class_board:CAP-SMD_BD8.0-L8.3-W8.3-LS9.3-FD" (at 133.35 95.25 0) (show_name no) (effects (font (size 1.27 1.27)) (hide yes)))
-    (property "Datasheet" "https://www.lcsc.com/product-detail/C72479.html" (at 133.35 95.25 0) (show_name no) (effects (font (size 1.27 1.27)) (hide yes)))
+    (property "Datasheet" "https://www.lcsc.com/product-detail/C37309.html" (at 133.35 95.25 0) (show_name no) (effects (font (size 1.27 1.27)) (hide yes)))
     (property "Description" "Aluminium electrolytic 100 uF 35 V, SMD can 8x10 mm (ROQANG RVT1V101M0810) - +VEXT bulk; PIN 1 = +" (at 133.35 95.25 0) (show_name no) (effects (font (size 1.27 1.27)) (hide yes)))
-    (property "LCSC" "C72479" (at 133.35 95.25 0) (show_name no) (effects (font (size 1.27 1.27)) (hide yes)))
+    (property "LCSC" "C37309" (at 133.35 95.25 0) (show_name no) (effects (font (size 1.27 1.27)) (hide yes)))
     (property "JLC_CLASS" "Extended" (at 133.35 95.25 0) (show_name no) (effects (font (size 1.27 1.27)) (hide yes)))
     (property "MPN" "RVT1V101M0810" (at 133.35 95.25 0) (show_name no) (effects (font (size 1.27 1.27)) (hide yes)))
@@
     (property "Value" "100uF 35V" (at 246.38 87.122 0) (show_name no) (effects (font (size 1.27 1.27)) (justify left top)))
     (property "Footprint" "class_board:CAP-SMD_BD8.0-L8.3-W8.3-LS9.3-FD" (at 248.92 82.55 0) (show_name no) (effects (font (size 1.27 1.27)) (hide yes)))
-    (property "Datasheet" "https://www.lcsc.com/product-detail/C72479.html" (at 248.92 82.55 0) (show_name no) (effects (font (size 1.27 1.27)) (hide yes)))
+    (property "Datasheet" "https://www.lcsc.com/product-detail/C37309.html" (at 248.92 82.55 0) (show_name no) (effects (font (size 1.27 1.27)) (hide yes)))
     (property "Description" "Aluminium electrolytic 100 uF 35 V, SMD can 8x10 mm (ROQANG RVT1V101M0810) - +VEXT bulk; PIN 1 = +" (at 248.92 82.55 0) (show_name no) (effects (font (size 1.27 1.27)) (hide yes)))
-    (property "LCSC" "C72479" (at 248.92 82.55 0) (show_name no) (effects (font (size 1.27 1.27)) (hide yes)))
+    (property "LCSC" "C37309" (at 248.92 82.55 0) (show_name no) (effects (font (size 1.27 1.27)) (hide yes)))
     (property "JLC_CLASS" "Extended" (at 248.92 82.55 0) (show_name no) (effects (font (size 1.27 1.27)) (hide yes)))
     (property "MPN" "RVT1V101M0810" (at 248.92 82.55 0) (show_name no) (effects (font (size 1.27 1.27)) (hide yes)))

Commit message: hardware: chip resistors and ceramic capacitors on KiCad standard footprints (Decision #47); schematic, library and gapped copies regenerated, ERC 0 errors
Co-Authored-By: Claude Fable 5.1 <noreply@anthropic.com>
Parts:
- C920, C930, C931, C941: footprint class_board:C0603 -> Capacitor_SMD:C_0603_1608Metric
- R920, R921, R930, R931, R932, R940, R941: footprint class_board:R0603 -> Resistor_SMD:R_0603_1608Metric
- R933: footprint class_board:R2512 -> Resistor_SMD:R_2512_6332Metric
