File: hardware/student/b1_inputs_gapped.kicad_sch (KiCad schematic)
At the start: 33 parts, among them U101 ADS8688IDBTR

Commit message: hardware: chip resistors and ceramic capacitors on KiCad standard footprints (Decision #47); schematic, library and gapped copies regenerated, ERC 0 errors
Co-Authored-By: Claude Fable 5.1 <noreply@anthropic.com>
Parts:
- C103, C104, C108, C111, C112, C113, C115, C116, C117, C118: footprint class_board:C0603 -> Capacitor_SMD:C_0603_1608Metric
- C105: footprint class_board:C1206 -> Capacitor_SMD:C_1206_3216Metric
- C106, C107: footprint class_board:C0805 -> Capacitor_SMD:C_0805_2012Metric
- R101, R102, R111, R112, R113, R115, R116, R117, R118: footprint class_board:R0603 -> Resistor_SMD:R_0603_1608Metric
