File: hardware/student/b3_outputs_gapped.kicad_sch (KiCad schematic)
At the start: 19 parts, among them U301 DAC8563SDGSR, U302 74HCT125PW, U303 OPA2192IDR

Commit message: hardware: chip resistors and ceramic capacitors on KiCad standard footprints (Decision #47); schematic, library and gapped copies regenerated, ERC 0 errors
Co-Authored-By: Claude Fable 5.1 <noreply@anthropic.com>
Parts:
- C301, C302, C304, C305, C308: footprint class_board:C0603 -> Capacitor_SMD:C_0603_1608Metric
- C303, C306, C307: footprint class_board:C0805 -> Capacitor_SMD:C_0805_2012Metric
- R301, R302, R303, R304, R309, R311: footprint class_board:R0603 -> Resistor_SMD:R_0603_1608Metric
