File: hardware/student/b5_dio_trig_gapped.kicad_sch (KiCad schematic)
At the start: 35 parts, among them J502 KF301-5.0-2P, J503 KF301-5.0-2P, J504 KF301-5.0-2P, J505 KF301-5.0-2P, J506 KF301-5.0-2P, J507 KF301-5.0-2P, U501 SN74AHCT541PWR, U503 SN74LVC1T45DBVR, U504 SN74LVC1G17DBVR, U505 TCA9535PWR, X501 10 MHz TCXO

Commit message: hardware: chip resistors and ceramic capacitors on KiCad standard footprints (Decision #47); schematic, library and gapped copies regenerated, ERC 0 errors
Co-Authored-By: Claude Fable 5.1 <noreply@anthropic.com>
Parts:
- C503, C504, C505, C506, C507: footprint class_board:C0603 -> Capacitor_SMD:C_0603_1608Metric
- R501, R502, R503, R504, R505, R506, R507, R508, R511, R512, R513, R514, R515: footprint class_board:R0603 -> Resistor_SMD:R_0603_1608Metric

Commit message: hardware: panel stacked on the back (180 x 100, three 2x20 headers, 17 SMA, TTL strip, TX terminal, Qwiic); TTL/fast/TX-coil/Qwiic connectors leave the main board; mains-safe relay channels (JQC-3FF 10 A, MAINS net class + DRC rules); library, sheets, gapped copies, docs regenerated; ERC 0 errors
Decisions #45-#50 in the course repo. The main-board PCB is unchanged: Update PCB from Schematic, header placement, relay re-spacing and connector rotation are the instructor's GUI steps on the master.

Co-Authored-By: Claude Fable 5.1 <noreply@anthropic.com>
Parts:
- removed J502, J503, J504, J505, J506, J507: KF301-5.0-2P, class_board:CONN-TH_P5.00_KF301-5.0-2P, symbol class_board:KF301-5.0-2P
- removed R501: 1k, Resistor_SMD:R_0603_1608Metric, symbol class_board:R0603_1k
Other:
- note added: "74AHCT541 (TTL-compatible inputs accept 3.3 V) buffers DIO1..8 to 5 V; 1 k series per output limits a shorted output to 5 mA (students!). Outputs are static/slow (kHz): 1 k x 100 pF cable = 100 ns. v0.8: TTL1..8 and FASTTTL1/2 leave on the panel link, not on board-edge terminals."
- note added: "74HCT125: FAST_OUT1/2 (MCPWM/RMT) -> 49.9 R series -> the panel link -> the two fast SMAs on the panel; drive +-6 mA rated, so a 50 R termination gives ~1 V: fast outs are for high-impedance TTL loads."
- note added: "FASTTTL1/2 leave this sheet as global labels -> panel link J7 -> the two fast SMAs"
- note added: "TTL1..TTL8 leave this sheet as global labels -> panel link J7 -> the 10-way screw-terminal"
- note added: "on the front panel (49.9 R series). The edge terminals J506/J507 are gone (v0.8)."
- note added: "strip on the front panel (TTL1..8 + 2 x GND). The board-edge terminals J501-J505 are gone (v0.8)."
- note removed: "74AHCT541 (TTL-compatible inputs accept 3.3 V) buffers DIO1..8 to 5 V; 1 k series per output limits a shorted output to 5 mA (students!). Outputs are static/slow (kHz): 1 k x 100 pF cable = 100 ns."
- note removed: "74HCT125: FAST_OUT1/2 (MCPWM/RMT) -> 49.9 R series -> terminals; drive +-6 mA rated, so a 50 R termination gives ~1 V: fast outs are for high-impedance TTL loads."
- note removed: "J501-J504: TTL1..TTL8 (5 V TTL out, 1 k series); J505: GND GND"
- note removed: "J506/J507: FASTTTL1/2 + GND (5 V TTL, 49.9 R series)"

Commit message: v0.7d: relays and mains removed, MODULE OUT 1-7 (5 V TTL) on a shrouded 2x6 header on the front panel, isolated inputs moved to the panel, section C = the front-panel board (4-layer, 18 mm SMA grid, OLED clear of headers, unrouted student copy), main board re-placed; workbook, tutor guide, firmware docs, hardware docs updated (Decision #58)
Co-Authored-By: Claude Fable 5.1 <noreply@anthropic.com>
Parts:
- removed TP502, TP503, TP504: TP, class_board:TestPoint_Pad_D1.5mm, symbol class_board:TestPoint
Connections:
- net EXP_P15 renamed MOD5
- net EXP_P16 renamed MOD6
- net EXP_P17 renamed MOD7
- net RLY_IN1 renamed MOD1
- net RLY_IN2 renamed MOD2
- net RLY_IN3 renamed MOD3
- net RLY_IN4 renamed MOD4
Other:
- note added: "P00..P07 = DIO1..8 into the 74AHCT541 above; P10..P13 and P15..P17 = MODULE OUT 1..7, the 3.3 V module outputs, to the panel link J8 (v0.7d)."
- note added: "P14 is NOT free: it is EXP_P14, the /CLR of the 74HC74 Johnson counter on the NMR receiver sheet (TP501 is its test point). MODULE OUT 8 is"
- note added: "mapping is unchanged. Every port is an input after power-up and after a reset: the pull-down on the panel buffer decides the state of a module."
- note added: "reserved: J8 pin 33 is not connected on this board and the panel pulls it down. MOD1..MOD4 keep the ports the relay gates used, so the firmware"
- note added: "v0.7: DIO1..8 keep their names but are no longer MCU pins — they come from the TCA9535 I2C expander U505 (address 0x20, A0 = A1 = A2 = GND), P00..P07. The 541 runs at +5V_RAW while the expander drives 3.3 V: the AHCT TTL thresholds (VIH 2.0 V) accept that. v0.7d: P10..P13 and P15..P17 = MODULE OUT 1..7 to the panel link J8 (P10..P13 are the ports the four relay gates used); P14 stays EXP_P14, the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"
- note removed: "Every port is an input after power-up and after a reset: the relay gate pull-downs (B4) are what set the safe state."
- note removed: "P00..P07 = DIO1..8 into the 74AHCT541 above, P10..P13 = RLY_IN1..4 to the relay gates (B4), P14..P17 spare on TP501..TP504."
- note removed: "v0.7: DIO1..8 keep their names but are no longer MCU pins — they come from the TCA9535 I2C expander U505 (address 0x20, A0 = A1 = A2 = GND), P00..P07. The 541 runs at +5V_RAW while the expander drives 3.3 V: the AHCT TTL thresholds (VIH 2.0 V) accept that. P10..P13 = RLY_IN1..4 (relay gates, B4), P14..P17 = spare on test points EXP_P14..P17."
