File: hardware/student/nmr_rx_gapped.kicad_sch (KiCad schematic)
At the start: 88 parts, among them U701 SI5351A-B-GT, U702 74HC74D,653, U703 OPA1656IDR, U704 DG419DY-T1-E3, U705 OPA1612AIDR, U706 OPA1612AIDR, U901 TS5A23157DGSR, U902 TS5A23157DGSR, Y701 25 MHz

Commit message: hardware: three LCSC numbers corrected (C701/C702 3.9 pF -> C519107, R722 9.1 k -> C23260, 100 uF 35 V -> C37309); library, sheets and gapped copies regenerated, ERC 0 errors; PROTOCOL: hbridge/polarizer commands, presence flags in info
Found by bom/verification/jlc_check.py in the course repo (full-BOM JLC check).

Co-Authored-By: Claude Fable 5.1 <noreply@anthropic.com>
Parts:
- C701, C702: symbol class_board:C0603_100nF -> class_board:C0603_4pF; JLC_CLASS Basic -> Extended; LCSC C14663 -> C519107; MPN CC0603KRX7R9BB104 -> CC0603BRNPO9BN3R9; Manufacturer Yageo -> YAGEO
- R722: symbol class_board:R0603_10k -> class_board:R0603_9R09k; LCSC C25804 -> C23260; MPN 0603WAF1002T5E -> 0603WAF9101T5E
Changed lines of the file:
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@@
     (instances (project "class-board" (path "/21416d14-3056-576f-bbf8-3b43eaeb7e71/27fece37-25e5-55f8-9b4c-3407e1c1ba01" (reference "TP701") (unit 1))))
   )
-  (symbol (lib_id "class_board:C0603_100nF") (at 350.52 59.69 90) (unit 1)
+  (symbol (lib_id "class_board:C0603_4pF") (at 350.52 59.69 90) (unit 1)
     (exclude_from_sim no) (in_bom yes) (on_board yes) (dnp no) (fields_autoplaced yes)
     (property "Reference" "C701" (at 346.71 56.388 0) (show_name no) (effects (font (size 1.27 1.27)) (justify left bottom)))
     (property "Value" "3.9pF" (at 346.71 62.992 0) (show_name no) (effects (font (size 1.27 1.27)) (justify left top)))
     (property "Footprint" "class_board:C0603" (at 350.52 59.69 0) (show_name no) (effects (font (size 1.27 1.27)) (hide yes)))
-    (property "Datasheet" "https://www.lcsc.com/product-detail/C14663.html" (at 350.52 59.69 0) (show_name no) (effects (font (size 1.27 1.27)) (hide yes)))
-    (property "Description" "Capacitor 100 nF 50 V X7R 0603 (Yageo CC0603KRX7R9BB104)" (at 350.52 59.69 0) (show_name no) (effects (font (size 1.27 1.27)) (hide yes)))
-    (property "LCSC" "C14663" (at 350.52 59.69 0) (show_name no) (effects (font (size 1.27 1.27)) (hide yes)))
-    (property "JLC_CLASS" "Basic" (at 350.52 59.69 0) (show_name no) (effects (font (size 1.27 1.27)) (hide yes)))
-    (property "MPN" "CC0603KRX7R9BB104" (at 350.52 59.69 0) (show_name no) (effects (font (size 1.27 1.27)) (hide yes)))
-    (property "Manufacturer" "Yageo" (at 350.52 59.69 0) (show_name no) (effects (font (size 1.27 1.27)) (hide yes)))
+    (property "Datasheet" "https://www.lcsc.com/product-detail/C519107.html" (at 350.52 59.69 0) (show_name no) (effects (font (size 1.27 1.27)) (hide yes)))
+    (property "Description" "Capacitor 3.9 pF 50 V NP0 0603 (Si5351 crystal load; circuits note 1.2 asks for 4 pF - 3.9 pF is the stocked NP0 value, XTAL_CL = 10 pF unchanged) (YAGEO CC0603BRNPO9BN3R9)" (at 350.52 59.69 0) (show_name no) (effects (font (size 1.27 1.27)) (hide yes)))
+    (property "LCSC" "C519107" (at 350.52 59.69 0) (show_name no) (effects (font (size 1.27 1.27)) (hide yes)))
+    (property "JLC_CLASS" "Extended" (at 350.52 59.69 0) (show_name no) (effects (font (size 1.27 1.27)) (hide yes)))
+    (property "MPN" "CC0603BRNPO9BN3R9" (at 350.52 59.69 0) (show_name no) (effects (font (size 1.27 1.27)) (hide yes)))
+    (property "Manufacturer" "YAGEO" (at 350.52 59.69 0) (show_name no) (effects (font (size 1.27 1.27)) (hide yes)))
     (property "Block" "NMR_RX" (at 350.52 59.69 0) (show_name no) (effects (font (size 1.27 1.27)) (hide yes)))
     (pin "1")
@@
     (instances (project "class-board" (path "/21416d14-3056-576f-bbf8-3b43eaeb7e71/27fece37-25e5-55f8-9b4c-3407e1c1ba01" (reference "#PWR7013") (unit 1))))
   )
-  (symbol (lib_id "class_board:C0603_100nF") (at 350.52 68.58 90) (unit 1)
+  (symbol (lib_id "class_board:C0603_4pF") (at 350.52 68.58 90) (unit 1)
     (exclude_from_sim no) (in_bom yes) (on_board yes) (dnp no) (fields_autoplaced yes)
     (property "Reference" "C702" (at 346.71 65.278 0) (show_name no) (effects (font (size 1.27 1.27)) (justify left bottom)))
     (property "Value" "3.9pF" (at 346.71 71.882 0) (show_name no) (effects (font (size 1.27 1.27)) (justify left top)))
     (property "Footprint" "class_board:C0603" (at 350.52 68.58 0) (show_name no) (effects (font (size 1.27 1.27)) (hide yes)))
-    (property "Datasheet" "https://www.lcsc.com/product-detail/C14663.html" (at 350.52 68.58 0) (show_name no) (effects (font (size 1.27 1.27)) (hide yes)))
-    (property "Description" "Capacitor 100 nF 50 V X7R 0603 (Yageo CC0603KRX7R9BB104)" (at 350.52 68.58 0) (show_name no) (effects (font (size 1.27 1.27)) (hide yes)))
-    (property "LCSC" "C14663" (at 350.52 68.58 0) (show_name no) (effects (font (size 1.27 1.27)) (hide yes)))
-    (property "JLC_CLASS" "Basic" (at 350.52 68.58 0) (show_name no) (effects (font (size 1.27 1.27)) (hide yes)))
-    (property "MPN" "CC0603KRX7R9BB104" (at 350.52 68.58 0) (show_name no) (effects (font (size 1.27 1.27)) (hide yes)))
-    (property "Manufacturer" "Yageo" (at 350.52 68.58 0) (show_name no) (effects (font (size 1.27 1.27)) (hide yes)))
+    (property "Datasheet" "https://www.lcsc.com/product-detail/C519107.html" (at 350.52 68.58 0) (show_name no) (effects (font (size 1.27 1.27)) (hide yes)))
+    (property "Description" "Capacitor 3.9 pF 50 V NP0 0603 (Si5351 crystal load; circuits note 1.2 asks for 4 pF - 3.9 pF is the stocked NP0 value, XTAL_CL = 10 pF unchanged) (YAGEO CC0603BRNPO9BN3R9)" (at 350.52 68.58 0) (show_name no) (effects (font (size 1.27 1.27)) (hide yes)))
+    (property "LCSC" "C519107" (at 350.52 68.58 0) (show_name no) (effects (font (size 1.27 1.27)) (hide yes)))
+    (property "JLC_CLASS" "Extended" (at 350.52 68.58 0) (show_name no) (effects (font (size 1.27 1.27)) (hide yes)))
+    (property "MPN" "CC0603BRNPO9BN3R9" (at 350.52 68.58 0) (show_name no) (effects (font (size 1.27 1.27)) (hide yes)))
+    (property "Manufacturer" "YAGEO" (at 350.52 68.58 0) (show_name no) (effects (font (size 1.27 1.27)) (hide yes)))
     (property "Block" "NMR_RX" (at 350.52 68.58 0) (show_name no) (effects (font (size 1.27 1.27)) (hide yes)))
     (pin "1")
@@
     (instances (project "class-board" (path "/21416d14-3056-576f-bbf8-3b43eaeb7e71/27fece37-25e5-55f8-9b4c-3407e1c1ba01" (reference "#PWR7071") (unit 1))))
   )
-  (symbol (lib_id "class_board:R0603_10k") (at 406.4 215.9 90) (unit 1)
+  (symbol (lib_id "class_board:R0603_9R09k") (at 406.4 215.9 90) (unit 1)
     (exclude_from_sim no) (in_bom yes) (on_board yes) (dnp no) (fields_autoplaced yes)
     (property "Reference" "R722" (at 402.59 212.598 0) (show_name no) (effects (font (size 1.27 1.27)) (justify left bottom)))
     (property "Value" "9.1k" (at 402.59 219.202 0) (show_name no) (effects (font (size 1.27 1.27)) (justify left top)))
     (property "Footprint" "class_board:R0603" (at 406.4 215.9 0) (show_name no) (effects (font (size 1.27 1.27)) (hide yes)))
-    (property "Datasheet" "https://www.lcsc.com/product-detail/C25804.html" (at 406.4 215.9 0) (show_name no) (effects (font (size 1.27 1.27)) (hide yes)))
-    (property "Description" "Resistor 10k 1% 0603 100 mW (Uniroyal 0603WAF1002T5E)" (at 406.4 215.9 0) (show_name no) (effects (font (size 1.27 1.27)) (hide yes)))
-    (property "LCSC" "C25804" (at 406.4 215.9 0) (show_name no) (effects (font (size 1.27 1.27)) (hide yes)))
+    (property "Datasheet" "https://www.lcsc.com/product-detail/C23260.html" (at 406.4 215.9 0) (show_name no) (effects (font (size 1.27 1.27)) (hide yes)))
+    (property "Description" "Resistor 9.1 kOhm 1% 0603 fitted where the design says 9.09 kOhm (stage-2 gain 10.01 instead of 10.00). The exact E96 9.09 kOhm is C23125 (Extended, 93 k stock) if the ratio must be exact (UNI-ROYAL 0603WAF9101T5E)" (at 406.4 215.9 0) (show_name no) (effects (font (size 1.27 1.27)) (hide yes)))
+    (property "LCSC" "C23260" (at 406.4 215.9 0) (show_name no) (effects (font (size 1.27 1.27)) (hide yes)))
     (property "JLC_CLASS" "Basic" (at 406.4 215.9 0) (show_name no) (effects (font (size 1.27 1.27)) (hide yes)))
-    (property "MPN" "0603WAF1002T5E" (at 406.4 215.9 0) (show_name no) (effects (font (size 1.27 1.27)) (hide yes)))
+    (property "MPN" "0603WAF9101T5E" (at 406.4 215.9 0) (show_name no) (effects (font (size 1.27 1.27)) (hide yes)))
     (property "Manufacturer" "UNI-ROYAL" (at 406.4 215.9 0) (show_name no) (effects (font (size 1.27 1.27)) (hide yes)))
     (property "Block" "NMR_RX" (at 406.4 215.9 0) (show_name no) (effects (font (size 1.27 1.27)) (hide yes)))

Commit message: hardware: chip resistors and ceramic capacitors on KiCad standard footprints (Decision #47); schematic, library and gapped copies regenerated, ERC 0 errors
Co-Authored-By: Claude Fable 5.1 <noreply@anthropic.com>
Parts:
- C701, C702, C703, C704, C705, C706, C707, C710, C711, C712, C720, C721, C724, C725, C901, C902, C903, C904, C906, C907, C908, C910, C912, C913, C914, C915, C916, C917, C918, C919: footprint class_board:C0603 -> Capacitor_SMD:C_0603_1608Metric
- C726, C727, C905: footprint class_board:C0805 -> Capacitor_SMD:C_0805_2012Metric
- R701, R702, R703, R704, R705, R706, R710, R711, R712, R713, R714, R721, R722, R723, R724, R901, R902, R903, R904, R905, R906, R907, R908, R909, R910, R912, R913, R914, R915, R916, R917, R918, R919, R923, R924: footprint class_board:R0603 -> Resistor_SMD:R_0603_1608Metric
