File: hardware/student/nmr_tx_gapped.kicad_sch (KiCad schematic)
At the start: 42 parts, among them J802 KF301-5.0-2P, U801 AD9834BRUZ, U802 OPA564AIDWPR

Commit message: hardware: three LCSC numbers corrected (C701/C702 3.9 pF -> C519107, R722 9.1 k -> C23260, 100 uF 35 V -> C37309); library, sheets and gapped copies regenerated, ERC 0 errors; PROTOCOL: hbridge/polarizer commands, presence flags in info
Found by bom/verification/jlc_check.py in the course repo (full-BOM JLC check).

Co-Authored-By: Claude Fable 5.1 <noreply@anthropic.com>
Parts:
- C813: LCSC C72479 -> C37309
Changed lines of the file:
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@@
     (property "Value" "100uF 35V" (at 251.46 205.232 0) (show_name no) (effects (font (size 1.27 1.27)) (justify left top)))
     (property "Footprint" "class_board:CAP-SMD_BD8.0-L8.3-W8.3-LS9.3-FD" (at 254 200.66 0) (show_name no) (effects (font (size 1.27 1.27)) (hide yes)))
-    (property "Datasheet" "https://www.lcsc.com/product-detail/C72479.html" (at 254 200.66 0) (show_name no) (effects (font (size 1.27 1.27)) (hide yes)))
+    (property "Datasheet" "https://www.lcsc.com/product-detail/C37309.html" (at 254 200.66 0) (show_name no) (effects (font (size 1.27 1.27)) (hide yes)))
     (property "Description" "Aluminium electrolytic 100 uF 35 V, SMD can 8x10 mm (ROQANG RVT1V101M0810) - +VEXT bulk; PIN 1 = +" (at 254 200.66 0) (show_name no) (effects (font (size 1.27 1.27)) (hide yes)))
-    (property "LCSC" "C72479" (at 254 200.66 0) (show_name no) (effects (font (size 1.27 1.27)) (hide yes)))
+    (property "LCSC" "C37309" (at 254 200.66 0) (show_name no) (effects (font (size 1.27 1.27)) (hide yes)))
     (property "JLC_CLASS" "Extended" (at 254 200.66 0) (show_name no) (effects (font (size 1.27 1.27)) (hide yes)))
     (property "MPN" "RVT1V101M0810" (at 254 200.66 0) (show_name no) (effects (font (size 1.27 1.27)) (hide yes)))

Commit message: hardware: chip resistors and ceramic capacitors on KiCad standard footprints (Decision #47); schematic, library and gapped copies regenerated, ERC 0 errors
Co-Authored-By: Claude Fable 5.1 <noreply@anthropic.com>
Parts:
- C801, C802, C803, C804, C805, C807, C808, C809, C810, C812, C814, C817: footprint class_board:C0603 -> Capacitor_SMD:C_0603_1608Metric
- C806, C811: footprint class_board:C0805 -> Capacitor_SMD:C_0805_2012Metric
- C818: footprint class_board:C1206 -> Capacitor_SMD:C_1206_3216Metric
- R801, R802, R803, R804, R805, R806, R807, R808, R809, R810, R811, R812, R815, R816, R817, R818: footprint class_board:R0603 -> Resistor_SMD:R_0603_1608Metric
- R814: footprint class_board:R0805 -> Resistor_SMD:R_0805_2012Metric

Commit message: hardware: panel stacked on the back (180 x 100, three 2x20 headers, 17 SMA, TTL strip, TX terminal, Qwiic); TTL/fast/TX-coil/Qwiic connectors leave the main board; mains-safe relay channels (JQC-3FF 10 A, MAINS net class + DRC rules); library, sheets, gapped copies, docs regenerated; ERC 0 errors
Decisions #45-#50 in the course repo. The main-board PCB is unchanged: Update PCB from Schematic, header placement, relay re-spacing and connector rotation are the instructor's GUI steps on the master.

Co-Authored-By: Claude Fable 5.1 <noreply@anthropic.com>
Parts:
- removed J802: KF301-5.0-2P, class_board:CONN-TH_P5.00_KF301-5.0-2P, symbol class_board:KF301-5.0-2P
Other:
- note added: "-> the TX SMA and the 2P screw terminal on the panel. Route TX and its return as a close pair,"
- note added: "TX leaves this sheet as a global label -> panel link J6 pins 19 and 21 (AGND on 20 and 22)"
- note added: "loop area < 1 cm2; up to 1 A of coil current must never share copper with the receiver pour."
- note removed: "TX leaves on the front-panel link (pin 39 -> panel SMA J801) and on J802 KF301-5.0-2P at the"
- note removed: "board edge (pin 1 = TX, pin 2 = GND). Route TX and its return as a close pair, loop area < 1 cm2;"
- note removed: "up to 1 A of coil current must never share copper with the receiver pour (re-spec 8.2)."
Changed lines of the file:
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@@
   (junction (at 358.14 123.19) (diameter 0) (color 0 0 0 0))
   (junction (at 372.11 110.49) (diameter 0) (color 0 0 0 0))
-  (junction (at 372.11 146.05) (diameter 0) (color 0 0 0 0))
   (no_connect (at 144.78 114.3))
   (no_connect (at 266.7 133.35))
@@
   (wire (pts (xy 372.11 102.87) (xy 372.11 100.33)) (stroke (width 0) (type default)))
   (wire (pts (xy 367.03 127) (xy 367.03 146.05)) (stroke (width 0) (type default)))
-  (wire (pts (xy 367.03 146.05) (xy 381 146.05)) (stroke (width 0) (type default)))
+  (wire (pts (xy 367.03 146.05) (xy 372.11 146.05)) (stroke (width 0) (type default)))
   (wire (pts (xy 372.11 146.05) (xy 372.11 152.4)) (stroke (width 0) (type default)))
-  (wire (pts (xy 381 143.51) (xy 375.92 143.51)) (stroke (width 0) (type default)))
   (text "NMR TX (section B) — AD9834 DDS + reconstruction filter + OPA564 power stage -> TX" (exclude_from_sim no) (at 12.7 14 0) (effects (font (size 3 3) (bold yes)) (justify left bottom)))
   (text "DDS: AD9834BRUZ, MCLK = CLK0_MCLK = 50.000 MHz from the Si5351A on the RX sheet; df = f_MCLK / 2^28 = 0.186 Hz per LSB. R801 6.80 k on FS ADJUST -> I_OUT,FS = 18 x 1.20 V / 6.80 k = 3.18 mA;" (exclude_from_sim no) (at 12.7 19 0) (effects (font (size 1.5 1.5)) (justify left bottom)))
@@
   (text "spare for an external gain resistor." (exclude_from_sim no) (at 214 218.4 0) (effects (font (size 1.2 1.2)) (justify left bottom)))
   (text "-20 dB pad: 100/(910+100) = 0.099 into a high-Z load." (exclude_from_sim no) (at 303 96 0) (effects (font (size 1.2 1.2)) (justify left bottom)))
-  (text "TX leaves on the front-panel link (pin 39 -> panel SMA J801) and on J802 KF301-5.0-2P at the" (exclude_from_sim no) (at 300 195 0) (effects (font (size 1.2 1.2)) (justify left bottom)))
-  (text "board edge (pin 1 = TX, pin 2 = GND). Route TX and its return as a close pair, loop area < 1 cm2;" (exclude_from_sim no) (at 300 198.2 0) (effects (font (size 1.2 1.2)) (justify left bottom)))
-  (text "up to 1 A of coil current must never share copper with the receiver pour (re-spec 8.2)." (exclude_from_sim no) (at 300 201.4 0) (effects (font (size 1.2 1.2)) (justify left bottom)))
+  (text "TX leaves this sheet as a global label -> panel link J6 pins 19 and 21 (AGND on 20 and 22)" (exclude_from_sim no) (at 300 195 0) (effects (font (size 1.2 1.2)) (justify left bottom)))
+  (text "-> the TX SMA and the 2P screw terminal on the panel. Route TX and its return as a close pair," (exclude_from_sim no) (at 300 198.2 0) (effects (font (size 1.2 1.2)) (justify left bottom)))
+  (text "loop area < 1 cm2; up to 1 A of coil current must never share copper with the receiver pour." (exclude_from_sim no) (at 300 201.4 0) (effects (font (size 1.2 1.2)) (justify left bottom)))
   (text "Level plan from 0.636 V pp at the DDS output (re-spec 2.3). Top row = the 89.4 kHz NMR setting: +-7.95 V into 1419 R = 5.6 mA = t90 417 us." (exclude_from_sim no) (at 38.1 198 0) (effects (font (size 1.3 1.3)) (justify left bottom)))
   (text "Firmware (re-spec 9.1 / 9.3): hold DDS_RESET high while writing, B28 = 1, PIN/SW set for hardware PSELECT; the carrier free-runs and is gated ONLY by TX_EN." (exclude_from_sim no) (at 38.1 222 0) (effects (font (size 1.3 1.3)) (justify left bottom)))
@@
     (instances (project "class-board" (path "/21416d14-3056-576f-bbf8-3b43eaeb7e71/bbb6eea2-e7dc-5d96-9a3a-152d51422209" (reference "#PWR8036") (unit 1))))
   )
-  (symbol (lib_id "class_board:KF301-5.0-2P") (at 388.62 144.78 180) (unit 1)
-    (exclude_from_sim no) (in_bom yes) (on_board yes) (dnp no) (fields_autoplaced yes)
-    (property "Reference" "J802" (at 383.54 140.208 0) (show_name no) (effects (font (size 1.27 1.27)) (justify left bottom)))
-    (property "Value" "KF301-5.0-2P" (at 383.54 149.352 0) (show_name no) (effects (font (size 1.27 1.27)) (justify left top)))
-    (property "Footprint" "class_board:CONN-TH_P5.00_KF301-5.0-2P" (at 388.62 144.78 0) (show_name no) (effects (font (size 1.27 1.27)) (hide yes)))
-    (property "Datasheet" "https://www.lcsc.com/datasheet/lcsc_datasheet_2303171000_Cixi-Kefa-Elec-KF301-5-0-2P_C474881.pdf" (at 388.62 144.78 0) (show_name no) (effects (font (size 1.27 1.27)) (hide yes)))
-    (property "Description" "Screw terminal 5.0 mm 2P, 300 V 16 A" (at 388.62 144.78 0) (show_name no) (effects (font (size 1.27 1.27)) (hide yes)))
-    (property "LCSC" "C474881" (at 388.62 144.78 0) (show_name no) (effects (font (size 1.27 1.27)) (hide yes)))
-    (property "JLC_CLASS" "Extended" (at 388.62 144.78 0) (show_name no) (effects (font (size 1.27 1.27)) (hide yes)))
-    (property "MPN" "KF301-5.0-2P" (at 388.62 144.78 0) (show_name no) (effects (font (size 1.27 1.27)) (hide yes)))
-    (property "Manufacturer" "Cixi Kefa" (at 388.62 144.78 0) (show_name no) (effects (font (size 1.27 1.27)) (hide yes)))
-    (property "Block" "NMR_TX" (at 388.62 144.78 0) (show_name no) (effects (font (size 1.27 1.27)) (hide yes)))
-    (pin "1")
-    (pin "2")
-    (instances (project "class-board" (path "/21416d14-3056-576f-bbf8-3b43eaeb7e71/bbb6eea2-e7dc-5d96-9a3a-152d51422209" (reference "J802") (unit 1))))
-  )
-  (symbol (lib_id "class_board:PWR_GND") (at 375.92 143.51 270) (unit 1)
-    (exclude_from_sim no) (in_bom no) (on_board yes) (dnp no) (fields_autoplaced yes)
-    (property "Reference" "#PWR8037" (at 373.38 140.208 0) (show_name no) (effects (font (size 1.27 1.27)) (justify left bottom) (hide yes)))
-    (property "Value" "GND" (at 372.618 143.51 0) (show_name no) (effects (font (size 1.27 1.27)) (justify right)))
-    (property "Footprint" "" (at 375.92 143.51 0) (show_name no) (effects (font (size 1.27 1.27)) (hide yes)))
-    (property "Datasheet" "" (at 375.92 143.51 0) (show_name no) (effects (font (size 1.27 1.27)) (hide yes)))
-    (property "Description" "Power symbol: GND" (at 375.92 143.51 0) (show_name no) (effects (font (size 1.27 1.27)) (hide yes)))
-    (pin "1")
-    (instances (project "class-board" (path "/21416d14-3056-576f-bbf8-3b43eaeb7e71/bbb6eea2-e7dc-5d96-9a3a-152d51422209" (reference "#PWR8037") (unit 1))))
-  )
 )
