File: hardware/front-panel/front-panel.kicad_sch (KiCad schematic)
At the start: 30 parts, among them J1 Panel link 2x20 female, J10 SMA, J11 SMA, J12 SMA, J13 SMA, J14 SMA, J15 SMA, J16 SMA, J17 OLED 1x4 socket, J2 SMA, J3 SMA, J4 SMA, J5 SMA, J6 SMA, J7 SMA, J8 SMA, J9 SMA

Commit message: hardware: panel stacked on the back (180 x 100, three 2x20 headers, 17 SMA, TTL strip, TX terminal, Qwiic); TTL/fast/TX-coil/Qwiic connectors leave the main board; mains-safe relay channels (JQC-3FF 10 A, MAINS net class + DRC rules); library, sheets, gapped copies, docs regenerated; ERC 0 errors
Decisions #45-#50 in the course repo. The main-board PCB is unchanged: Update PCB from Schematic, header placement, relay re-spacing and connector rotation are the instructor's GUI steps on the master.

Co-Authored-By: Claude Fable 5.1 <noreply@anthropic.com>
Parts:
- removed J4, J5, J6, J7, J8, J9: SMA, class_board:SMA-TH_BWSMA-KE-Z001, symbol class_board:BWSMA-KE-Z001
- added H5, H6: M2, MountingHole:MountingHole_2.2mm_M2, symbol class_board:MountingHole
- added J18, J19, J20, J21, J22, J23, J24, J25, J26: SMA, class_board:SMA-TH_BWSMA-KE-Z001, symbol class_board:BWSMA-KE-Z001
- added J30: OLED 1x4 socket, right-angle, Connector_PinSocket_2.54mm:PinSocket_1x04_P2.54mm_Horizontal, symbol class_board:HDR_1x4_FEMALE
- added J31: KF128-2.54-10P, class_board:CONN-TH_10P-P2.54_KF128-2.54-10P, symbol class_board:KF128-2.54-10P
- added J32: KF128-5.0-2P, class_board:CONN-TH_P5.00_KF128-5.0-2P, symbol class_board:KF128-5.0-2P
- added J33: Qwiic (vertical), class_board:CONN-SMD_BM04B-SRSS-TB, symbol class_board:QWIIC_BM04B-SRSS
- J1: footprint class_board:HDR-TH_40P-P2.54-V-F-R2-C20-S2.54 -> Connector_PinSocket_2.54mm:PinSocket_2x20_P2.54mm_Vertical; Assembly (none) -> hand; JLC_CLASS Extended -> (none); LCSC C2977589 -> (none); MPN 2.54-2*20 -> 2x20 female header 8.5 mm; Manufacturer ZHOURI -> any; Purchase (none) -> C5124634; now left out of the parts list
- J17: value OLED 1x4 socket -> SMA; footprint class_board:PinSocket_1x04_P2.54mm_Vertical -> class_board:SMA-TH_BWSMA-KE-Z001; symbol class_board:HDR_1x4_FEMALE -> class_board:BWSMA-KE-Z001; LCSC C2894927 -> C496549; MPN PZ254-1-04-Z-8.5 -> BWSMA-KE-Z001; Manufacturer XFCN -> BAT Wireless
- J2, J3: value SMA -> Panel link 2x20 female; footprint class_board:SMA-TH_BWSMA-KE-Z001 -> Connector_PinSocket_2.54mm:PinSocket_2x20_P2.54mm_Vertical; symbol class_board:BWSMA-KE-Z001 -> class_board:HDR_2x20_FEMALE; Assembly (none) -> hand; JLC_CLASS Extended -> (none); LCSC C496549 -> (none); MPN BWSMA-KE-Z001 -> 2x20 female header 8.5 mm; Manufacturer BAT Wireless -> any; Purchase (none) -> C5124634; now left out of the parts list
- R1, R2, R3: footprint class_board:R0603 -> Resistor_SMD:R_0603_1608Metric
Connections:
- net +3V3: now also J2.27, J2.29, J3.5, R1.1, J30.2 (VCC), J33.2 (3V3); no longer J1.30, J17.2 (VCC)
- net AGND: now also J1.10, J1.12, J1.14, J1.16, J1.18, J1.2, J1.20, J1.22, J1.24, J1.26, J1.28, J1.30, J1.32, J1.34, J1.36, J1.38, J1.4, J1.40, J1.6, J1.8, J17.1 (GND), J17.2 (GND), J17.3 (GND), J17.4 (GND), J18.1 (GND), J18.2 (GND), J18.3 (GND), J18.4 (GND), J19.1 (GND), J19.2 (GND), J19.3 (GND), J19.4 (GND), J20.1 (GND), J20.2 (GND), J20.3 (GND), J20.4 (GND), J21.1 (GND), J21.2 (GND), J21.3 (GND), J21.4 (GND), J22.1 (GND), J22.2 (GND), J22.3 (GND), J22.4 (GND), J23.1 (GND), J23.2 (GND), J23.3 (GND), J23.4 (GND), J24.1 (GND), J24.2 (GND), J24.3 (GND), J24.4 (GND), J25.1 (GND), J25.2 (GND), J25.3 (GND), J25.4 (GND), J26.1 (GND), J26.2 (GND), J26.3 (GND), J26.4 (GND), J32.2; no longer J1.1, J1.11, J1.13, J1.15, J1.17, J1.19, J1.21, J1.23, J1.3, J1.37, J1.39, J1.7, J1.9, J2.1 (GND), J2.2 (GND), J2.3 (GND), J2.4 (GND), J3.1 (GND), J3.2 (GND), J3.3 (GND), J3.4 (GND)
- net AI1: now also J1.1, J16.5 (SIG); no longer J1.10
- net AI2: now also J1.3, J17.5 (SIG); no longer J1.12
- net AI3: now also J1.5, J18.5 (SIG); no longer J1.14
- net AI4: now also J1.7, J19.5 (SIG); no longer J1.16, J10.5 (SIG)
- net AI5: now also J1.9, J22.5 (SIG); no longer J1.18, J12.5 (SIG)
- net AI6: now also J1.11, J23.5 (SIG); no longer J1.20, J13.5 (SIG)
- net AI7: now also J1.13, J24.5 (SIG); no longer J1.22, J14.5 (SIG)
- net AI8: now also J1.15, J25.5 (SIG); no longer J1.24, J15.5 (SIG)
- net AO1: now also J1.25, J10.5 (SIG); no longer J1.2, J2.5 (SIG)
- net AO2: now also J1.27, J11.5 (SIG); no longer J1.4, J3.5 (SIG)
- net AUX: now also J1.23, J13.5 (SIG); no longer J1.8
- net GND: now also J2.10, J2.12, J2.14, J2.16, J2.18, J2.2, J2.20, J2.22, J2.24, J2.26, J2.28, J2.30, J2.32, J2.34, J2.36, J2.38, J2.4, J2.40, J2.6, J2.8, J3.10, J3.12, J3.14, J3.16, J3.18, J3.2, J3.20, J3.22, J3.24, J3.26, J3.28, J3.30, J3.32, J3.34, J3.36, J3.38, J3.4, J3.40, J3.6, J3.8, J30.1 (GND), J31.10, J31.9, J33.1 (GND), J33.5 (SHELL), J33.6 (SHELL); no longer J1.25, J1.27, J1.29, J1.31, J1.33, J1.35, J1.5, J17.1 (GND)
- net I2C_SCL: now also J2.25, J30.3 (SCL), J33.4 (SCL); no longer J1.28, J17.3 (SCL)
- net I2C_SDA: now also J2.23, J30.4 (SDA), J33.3 (SDA); no longer J1.26, J17.4 (SDA)
- net LED_ACT: now also J2.33; no longer J1.36
- net LED_WIFI: now also J2.31; no longer J1.34
- net RX: now also J1.17, J20.5 (SIG); no longer J1.38, J11.5 (SIG)
- net SPARE: now also J26.5 (SIG); no longer J16.5 (SIG)
- net TRIG_5V: now also J12.5 (SIG), J2.21; no longer J1.6
- net TX: now also J1.19, J1.21, J14.5 (SIG), J32.1; no longer J1.40
- removed net LED_PWR: J1.32, R1.1
- new net +5V_RAW: J3.1, J3.3
- new net FASTTTL1: J15.5 (SIG), J2.17
- new net FASTTTL2: J2.19, J21.5 (SIG)
- new net GPIO15: J3.13
- new net GPIO4: J3.7
- new net GPIO43: J3.15
- new net GPIO44: J3.17
- new net GPIO6: J3.9
- new net GPIO7: J3.11
- new net TTL1: J2.1, J31.1
- new net TTL2: J2.3, J31.2
- new net TTL3: J2.5, J31.3
- new net TTL4: J2.7, J31.4
- new net TTL5: J2.9, J31.5
- new net TTL6: J2.11, J31.6
- new net TTL7: J2.13, J31.7
- new net TTL8: J2.15, J31.8
- no-connect marks 0 -> 20
Other:
- note added: "0.96 in I2C OLED (0x3C) on a right-angle socket: the module lies flat, held by H5/H6 (M2)"
- note added: "17 SMA on a 20 mm grid (3 x 6, the 18th position is empty). Shields on AGND; the panel copper is AGND on both layers."
- note added: "AO1/AO2: +-10 V, 49.9 ohm back-terminated. AI1..AI8: +-10 V, 1 kohm series on the main board. TRIG: 5 V into open circuit, about 2.4 V into 50 ohm. FAST1/FAST2 = the main-board nets FASTTTL1 / FASTTTL2."
- note added: "FRONT PANEL - 2 layers, 180 x 100 mm; copper = AGND, joined to GND only at the main-board star point NT1"
- note added: "H1-H4: M3, same pattern as the main board (stand-offs). H5/H6: M2 for the OLED module."
- note added: "H5 / H6 are M2 (2.2 mm) holes for the OLED module; the shared library only has the M3 symbol, so their footprint is overridden to MountingHole:MountingHole_2.2mm_M2."
- note added: "J1 - analog (inner face): mates J6, the analog header"
- note added: "J2 - digital (inner face): mates J7, the digital header"
- note added: "J3 - power + spares (inner face): mates J8, the power + spares header"
- note added: "PWR is +3V3 from the link (1 kohm -> about 1 mA); WIFI / ACT come from GPIO43 / GPIO44 through JP1 / JP2 on the main board."
- note added: "Panel coordinates are mirrored in x against the main board (panel x = 180 - main x, panel y = main y), because the panel is drawn from its OUTER face. The main board's REAR edge is therefore the panel's TOP edge."
- note added: "Pins marked spare are not connected on the main board and are left unconnected here. SPARE (the 18th SMA position is empty; the fitted SPARE SMA) has its shield on AGND and its centre pin on TP1 only."
- note added: "Qwiic (vertical): sensor from the front; shell pads on GND"
- note added: "SPARE SMA: shield on AGND, centre pin on TP1 only (no link pin)"
- note added: "So the analog header J6 (main x = 12) is panel J1 at panel x = 168, the digital header J7 stays at x = 90, and the power header J8 (main x = 168) is panel J3 at panel x = 12."
- note added: "TTL1..8 out (5 V, 1 kohm series on the main board) + 2 x GND"
- note added: "TX coil terminal, beside the TX SMA (kept: user 2026-09-16)"
- note added: "The panel is passive: the rails come in through the link, so each one carries a power flag."
- note added: "The panel lies FLAT ON THE BACK of the main board (Decision #45). J1 / J2 / J3 are 2x20 FEMALE headers on the panel's INNER face (B.Cu); they mate J6 / J7 / J8, the male headers on the main board's bottom side."
- note added: "With that mirror, panel pad k mates main-board pin k on all three headers (the KiCad PinSocket footprint already carries the mating mirror). gen_panel.py proves it from the pad coordinates before the board is written."
- note added: "panel label: ACT"
- note added: "panel label: AI1 (40, 45) mm"
- note added: "panel label: AI2 (60, 45) mm"
- note added: "panel label: AI3 (80, 45) mm"
- note added: "panel label: AI4 (100, 45) mm"
- note added: "panel label: AI5 (40, 65) mm"
- note added: "panel label: AI6 (60, 65) mm"
- note added: "panel label: AI7 (80, 65) mm"
- note added: "panel label: AI8 (100, 65) mm"
- note added: "panel label: AO1 (40, 25) mm"
- note added: "panel label: AO2 (60, 25) mm"
- note added: "panel label: AUX (100, 25) mm"
- note added: "panel label: FAST1 (140, 25) mm"
- note added: "panel label: FAST2 (140, 45) mm"
- note added: "panel label: PWR"
- note added: "panel label: RX (120, 45) mm"
- note added: "panel label: SPARE (120, 65) mm"
- note added: "panel label: TRIG (80, 25) mm"
- note added: "panel label: TX (120, 25) mm"
- note added: "panel label: WIFI"
- note added: "panel x = 12 mm (main board x = 168 mm)"
- note added: "panel x = 168 mm (main board x = 12 mm)"
- note added: "panel x = 90 mm (main board x = 90 mm)"
- note removed: "0.96in I2C OLED module (GND VCC SCL SDA), address 0x3C, hangs below the socket"
- note removed: "FRONT PANEL - 2-layer 180 x 65 mm; copper = AGND, joined to GND only through the main-board star"
- note removed: "J1 is mounted on the BACK of the panel: female pad 2k-1 mates with link pin 2k and pad 2k with link pin 2k-1 (mirrored footprint). Net names follow the link pins (brief 7.8, v0.7 pins 37-40)."
- note removed: "LED_PWR = +3V3 from the link (pin 31); 1 k series -> ~1 mA"
- note removed: "RX (link pin 37) = NMR receive coil into the LNA (section A); TX (link pin 39) = NMR transmit coil from the OPA564 stage (section B); AGND on pins 38/40 beside them. SPARE: SMA shield to AGND, centre pin to test pad TP1 only."
- note removed: "SPARE SMA: fitted, shield to AGND, centre pin to TP1 only (no link pin)"
- note removed: "TRIG: 5 V into open circuit, about 2.4 V into 50 ohm (74LVC1T45 + 33 ohm). AI1..AI8 +-10 V, 1 kOhm series on the main board. AO1/AO2 +-10 V, 49.9 ohm back-terminated."
- note removed: "panel label: AI1"
- note removed: "panel label: AI2"
- note removed: "panel label: AI3"
- note removed: "panel label: AI4"
- note removed: "panel label: AI5"
- note removed: "panel label: AI6"
- note removed: "panel label: AI7"
- note removed: "panel label: AI8"
- note removed: "panel label: AO1"
- note removed: "panel label: AO2"
- note removed: "panel label: AUX"
- note removed: "panel label: RX"
- note removed: "panel label: SPARE"
- note removed: "panel label: TRIG"
- note removed: "panel label: TX"
- title: TIGP class board 2026 - front panel -> TIGP class board 2026 - front panel (180 x 100, stacked on the back)
- moved on the sheet: D1, D2, D3, FID1, FID2, H1, H2, H3, H4, J1, J10, J11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

Commit message: front panel: 3D models resolve from front-panel/ (path fix), OLED as one footprint with four M2 holes on an 8.5 mm vertical socket + box model, TTL/TX terminals flush with the bottom edge (instructor review 2026-09-17); DRC 0 errors
Co-Authored-By: Claude Fable 5.1 <noreply@anthropic.com>
Parts:
- removed H5, H6: M2, MountingHole:MountingHole_2.2mm_M2, symbol class_board:MountingHole
- J30: value OLED 1x4 socket, right-angle -> OLED 0.96in module on 1x4 socket 8.5 mm; footprint Connector_PinSocket_2.54mm:PinSocket_1x04_P2.54mm_Horizontal -> class_board:OLED-0.96in-4P-module-socket
Other:
- note added: "0.96 in I2C OLED (0x3C) on an 8.5 mm vertical socket: the module lies flat on four M2 stand-offs (holes in the footprint)"
- note added: "H1-H4: M3, same pattern as the main board (stand-offs). The OLED module's M2 holes are part of J30."
- note added: "J30 is one footprint: the vertical 8.5 mm 1x4 socket (JLC C2894927) plus the OLED module's outline and its four M2 (2.2 mm) holes. The module lies flat on four 11 mm M2 stand-offs; measure the real module's hole spacing (23.5 x 23.8 assumed) before the order."
- note removed: "0.96 in I2C OLED (0x3C) on a right-angle socket: the module lies flat, held by H5/H6 (M2)"
- note removed: "H1-H4: M3, same pattern as the main board (stand-offs). H5/H6: M2 for the OLED module."
- note removed: "H5 / H6 are M2 (2.2 mm) holes for the OLED module; the shared library only has the M3 symbol, so their footprint is overridden to MountingHole:MountingHole_2.2mm_M2."
Changed lines of the file:
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@@
   (text "So the analog header J6 (main x = 12) is panel J1 at panel x = 168, the digital header J7 stays at x = 90, and the power header J8 (main x = 168) is panel J3 at panel x = 12." (exclude_from_sim no) (at 14 29 0) (effects (font (size 1.4 1.4)) (justify left bottom)))
   (text "Pins marked spare are not connected on the main board and are left unconnected here. SPARE (the 18th SMA position is empty; the fitted SPARE SMA) has its shield on AGND and its centre pin on TP1 only." (exclude_from_sim no) (at 14 33 0) (effects (font (size 1.4 1.4)) (justify left bottom)))
-  (text "H5 / H6 are M2 (2.2 mm) holes for the OLED module; the shared library only has the M3 symbol, so their footprint is overridden to MountingHole:MountingHole_2.2mm_M2." (exclude_from_sim no) (at 14 37 0) (effects (font (size 1.4 1.4)) (justify left bottom)))
+  (text "J30 is one footprint: the vertical 8.5 mm 1x4 socket (JLC C2894927) plus the OLED module's outline and its four M2 (2.2 mm) holes. The module lies flat on four 11 mm M2 stand-offs; measure the real module's hole spacing (23.5 x 23.8 assumed) before the order." (exclude_from_sim no) (at 14 37 0) (effects (font (size 1.4 1.4)) (justify left bottom)))
   (text "AO1/AO2: +-10 V, 49.9 ohm back-terminated. AI1..AI8: +-10 V, 1 kohm series on the main board. TRIG: 5 V into open circuit, about 2.4 V into 50 ohm. FAST1/FAST2 = the main-board nets FASTTTL1 / FASTTTL2." (exclude_from_sim no) (at 14 41 0) (effects (font (size 1.4 1.4)) (justify left bottom)))
   (text "J1 - analog (inner face): mates J6, the analog header" (exclude_from_sim no) (at 45 100 0) (effects (font (size 1.6 1.6) (bold yes)) (justify left bottom)))
@@
   (text "TX coil terminal, beside the TX SMA (kept: user 2026-09-16)" (exclude_from_sim no) (at 128 355 0) (effects (font (size 1.3 1.3)) (justify left bottom)))
   (text "Qwiic (vertical): sensor from the front; shell pads on GND" (exclude_from_sim no) (at 198 355 0) (effects (font (size 1.3 1.3)) (justify left bottom)))
-  (text "0.96 in I2C OLED (0x3C) on a right-angle socket: the module lies flat, held by H5/H6 (M2)" (exclude_from_sim no) (at 278 355 0) (effects (font (size 1.3 1.3)) (justify left bottom)))
+  (text "0.96 in I2C OLED (0x3C) on an 8.5 mm vertical socket: the module lies flat on four M2 stand-offs (holes in the footprint)" (exclude_from_sim no) (at 278 355 0) (effects (font (size 1.3 1.3)) (justify left bottom)))
   (text "PWR is +3V3 from the link (1 kohm -> about 1 mA); WIFI / ACT come from GPIO43 / GPIO44 through JP1 / JP2 on the main board." (exclude_from_sim no) (at 355 340 0) (effects (font (size 1.3 1.3)) (justify left bottom)))
   (text "panel label: PWR" (exclude_from_sim no) (at 388 362 0) (effects (font (size 1.2 1.2)) (justify left bottom)))
@@
   (text "SPARE SMA: shield on AGND, centre pin on TP1 only (no link pin)" (exclude_from_sim no) (at 424 348 0) (effects (font (size 1.2 1.2)) (justify left bottom)))
   (text "The panel is passive: the rails come in through the link, so each one carries a power flag." (exclude_from_sim no) (at 60 396 0) (effects (font (size 1.2 1.2)) (justify left bottom)))
-  (text "H1-H4: M3, same pattern as the main board (stand-offs).   H5/H6: M2 for the OLED module." (exclude_from_sim no) (at 200 398 0) (effects (font (size 1.2 1.2)) (justify left bottom)))
+  (text "H1-H4: M3, same pattern as the main board (stand-offs). The OLED module's M2 holes are part of J30." (exclude_from_sim no) (at 200 398 0) (effects (font (size 1.2 1.2)) (justify left bottom)))
   (global_label "AI1" (shape bidirectional) (at 76.2 105.41 180) (fields_autoplaced yes) (effects (font (size 1.27 1.27)) (justify right)))
   (global_label "AI2" (shape bidirectional) (at 76.2 107.95 180) (fields_autoplaced yes) (effects (font (size 1.27 1.27)) (justify right)))
@@
     (exclude_from_sim no) (in_bom yes) (on_board yes) (dnp no) (fields_autoplaced yes)
     (property "Reference" "J30" (at 294.64 367.538 0) (show_name no) (effects (font (size 1.27 1.27)) (justify left bottom)))
-    (property "Value" "OLED 1x4 socket, right-angle" (at 294.64 381.762 0) (show_name no) (effects (font (size 1.27 1.27)) (justify left top)))
-    (property "Footprint" "Connector_PinSocket_2.54mm:PinSocket_1x04_P2.54mm_Horizontal" (at 299.72 374.65 0) (show_name no) (effects (font (size 1.27 1.27)) (hide yes)))
+    (property "Value" "OLED 0.96in module on 1x4 socket 8.5 mm" (at 294.64 381.762 0) (show_name no) (effects (font (size 1.27 1.27)) (justify left top)))
+    (property "Footprint" "class_board:OLED-0.96in-4P-module-socket" (at 299.72 374.65 0) (show_name no) (effects (font (size 1.27 1.27)) (hide yes)))
     (property "Datasheet" "https://www.lcsc.com/product-detail/C2894927.html" (at 299.72 374.65 0) (show_name no) (effects (font (size 1.27 1.27)) (hide yes)))
-    (property "Description" "1x4 2.54 mm female header, right-angle, so the 0.96in OLED module lies flat on the panel (GND VCC SCL SDA)" (at 299.72 374.65 0) (show_name no) (effects (font (size 1.27 1.27)) (hide yes)))
+    (property "Description" "0.96in I2C OLED module (GND VCC SCL SDA) on a vertical 8.5 mm 1x4 female header (C2894927); the footprint carries the module outline and its four M2 holes" (at 299.72 374.65 0) (show_name no) (effects (font (size 1.27 1.27)) (hide yes)))
     (property "LCSC" "C2894927" (at 299.72 374.65 0) (show_name no) (effects (font (size 1.27 1.27)) (hide yes)))
     (property "JLC_CLASS" "Extended" (at 299.72 374.65 0) (show_name no) (effects (font (size 1.27 1.27)) (hide yes)))
@@
     (instances (project "front-panel" (path "/9a1de069-fc88-5135-9eba-6be985ab8138" (reference "H4") (unit 1))))
   )
-  (symbol (lib_id "class_board:MountingHole") (at 299.72 405.13 0) (unit 1)
-    (exclude_from_sim no) (in_bom no) (on_board yes) (dnp no) (fields_autoplaced yes)
-    (property "Reference" "H5" (at 298.45 403.098 0) (show_name no) (effects (font (size 1.27 1.27)) (justify left bottom)))
-    (property "Value" "M2" (at 298.45 407.162 0) (show_name no) (effects (font (size 1.27 1.27)) (justify left top)))
-    (property "Footprint" "MountingHole:MountingHole_2.2mm_M2" (at 299.72 405.13 0) (show_name no) (effects (font (size 1.27 1.27)) (hide yes)))
-    (property "Datasheet" "" (at 299.72 405.13 0) (show_name no) (effects (font (size 1.27 1.27)) (hide yes)))
-    (property "Description" "Mounting hole 3.2 mm for M3" (at 299.72 405.13 0) (show_name no) (effects (font (size 1.27 1.27)) (hide yes)))
-    (property "Block" "PANEL" (at 299.72 405.13 0) (show_name no) (effects (font (size 1.27 1.27)) (hide yes)))
-    (instances (project "front-panel" (path "/9a1de069-fc88-5135-9eba-6be985ab8138" (reference "H5") (unit 1))))
-  )
-  (symbol (lib_id "class_board:MountingHole") (at 325.12 405.13 0) (unit 1)
-    (exclude_from_sim no) (in_bom no) (on_board yes) (dnp no) (fields_autoplaced yes)
-    (property "Reference" "H6" (at 323.85 403.098 0) (show_name no) (effects (font (size 1.27 1.27)) (justify left bottom)))
-    (property "Value" "M2" (at 323.85 407.162 0) (show_name no) (effects (font (size 1.27 1.27)) (justify left top)))
-    (property "Footprint" "MountingHole:MountingHole_2.2mm_M2" (at 325.12 405.13 0) (show_name no) (effects (font (size 1.27 1.27)) (hide yes)))
-    (property "Datasheet" "" (at 325.12 405.13 0) (show_name no) (effects (font (size 1.27 1.27)) (hide yes)))
-    (property "Description" "Mounting hole 3.2 mm for M3" (at 325.12 405.13 0) (show_name no) (effects (font (size 1.27 1.27)) (hide yes)))
-    (property "Block" "PANEL" (at 325.12 405.13 0) (show_name no) (effects (font (size 1.27 1.27)) (hide yes)))
-    (instances (project "front-panel" (path "/9a1de069-fc88-5135-9eba-6be985ab8138" (reference "H6") (unit 1))))
-  )
   (symbol (lib_id "class_board:Fiducial") (at 359.41 405.13 0) (unit 1)
