File: hardware/front-panel/front-panel.kicad_sch (KiCad schematic)
At the start: 78 parts, among them J1 Panel link 2x20 female, J10 SMA, J11 SMA, J12 SMA, J13 SMA, J14 SMA, J15 SMA, J16 SMA, J17 SMA, J18 SMA, J19 SMA, J2 Panel link 2x20 female, J20 SMA, J21 SMA, J22 SMA, J23 SMA, J24 SMA, J25 SMA, J26 SMA, J3 Panel link 2x20 female, J30 OLED 0.96in module on 1x4 soc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, J31 KF128-2.54-10P, J32 KF128-5.0-2P, J33 Qwiic (vertical), J40 Module header 2x6 (shrouded), J411 KF301-5.0-2P, J412 KF301-5.0-2P, Q411 MMBT5551, Q412 MMBT5551, Q421 MMBT5551, Q422 MMBT5551, U401 6N137S-TA1-L, U402 6N137S-TA1-L, U410 SN74AHCT541PWR

Commit message: front panel: OLED footprint per the real module (27 x 29 mm, holes 24 x 26 mm, header 1 mm below the top edge), panel + student copy regenerated, DRC 0/0 with zones filled
Co-Authored-By: Claude Fable 5.1 <noreply@anthropic.com>
Other:
- note added: "J30 is one footprint: the vertical 8.5 mm 1x4 socket (JLC C2894927) plus the OLED module's outline and its four M2 (2.2 mm) holes. The module lies flat on four 11 mm M2 stand-offs; hole spacing 24 x 26 mm (instructor, 2026-09-17), 2.4 mm holes; confirm on the delivered modules."
- note removed: "J30 is one footprint: the vertical 8.5 mm 1x4 socket (JLC C2894927) plus the OLED module's outline and its four M2 (2.2 mm) holes. The module lies flat on four 11 mm M2 stand-offs; measure the real module's hole spacing (23.5 x 23.8 assumed) before the order."
Changed lines of the file:
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@@
   (text "So the analog header J6 (main x = 12) is panel J1 at panel x = 168, the digital header J7 stays at x = 90, and the power header J8 (main x = 168) is panel J3 at panel x = 12." (exclude_from_sim no) (at 14 29 0) (effects (font (size 1.4 1.4)) (justify left bottom)))
   (text "Pins marked spare are not connected on the main board and are left unconnected here. SPARE (the 18th SMA position is empty; the fitted SPARE SMA) has its shield on AGND and its centre pin on TP1 only." (exclude_from_sim no) (at 14 33 0) (effects (font (size 1.4 1.4)) (justify left bottom)))
-  (text "J30 is one footprint: the vertical 8.5 mm 1x4 socket (JLC C2894927) plus the OLED module's outline and its four M2 (2.2 mm) holes. The module lies flat on four 11 mm M2 stand-offs; measure the real module's hole spacing (23.5 x 23.8 assumed) before the order." (exclude_from_sim no) (at 14 37 0) (effects (font (size 1.4 1.4)) (justify left bottom)))
+  (text "J30 is one footprint: the vertical 8.5 mm 1x4 socket (JLC C2894927) plus the OLED module's outline and its four M2 (2.2 mm) holes. The module lies flat on four 11 mm M2 stand-offs; hole spacing 24 x 26 mm (instructor, 2026-09-17), 2.4 mm holes; confirm on the delivered modules." (exclude_from_sim no) (at 14 37 0) (effects (font (size 1.4 1.4)) (justify left bottom)))
   (text "AO1/AO2: +-10 V, 49.9 ohm back-terminated. AI1..AI8: +-10 V, 1 kohm series on the main board. TRIG: 5 V into open circuit, about 2.4 V into 50 ohm. FAST1/FAST2 = the main-board nets FASTTTL1 / FASTTTL2." (exclude_from_sim no) (at 14 41 0) (effects (font (size 1.4 1.4)) (justify left bottom)))
   (text "J1 - analog (inner face): mates J6, the analog header" (exclude_from_sim no) (at 45 100 0) (effects (font (size 1.6 1.6) (bold yes)) (justify left bottom)))

Commit message: front panel: male link headers J1/J2/J3 (Decision #62), J1 escapes outward; routed, DRC 0/0 with zones filled; student copy regenerated
Co-Authored-By: Claude Fable 5.1 <noreply@anthropic.com>
Parts:
- J1, J2, J3: value Panel link 2x20 female -> Panel link 2x20 male; footprint Connector_PinSocket_2.54mm:PinSocket_2x20_P2.54mm_Vertical -> Connector_PinHeader_2.54mm:PinHeader_2x20_P2.54mm_Vertical; symbol class_board:HDR_2x20_FEMALE -> class_board:HDR_2x20_MALE; LCSC C5124634 -> C5224014; MPN 2.54-2*20P (8.5 mm) -> PZ2.54-2*20; Manufacturer BOOMELE -> ZHOURI; Purchase C5124634 -> C5224014
Other:
- note added: "The panel lies FLAT ON THE BACK of the main board (Decision #45). J1 / J2 / J3 are 2x20 MALE headers on the panel's INNER face (B.Cu); they mate J6 / J7 / J8, the FEMALE sockets on the main board's bottom side (its pins are live - user 2026-09-17)."
- note added: "With that mirror, panel pad k mates main-board pin k on all three headers (the KiCad PinSocket footprint on the main board carries the mating mirror). gen_panel.py proves it from the pad coordinates before the board is written."
- note removed: "The panel lies FLAT ON THE BACK of the main board (Decision #45). J1 / J2 / J3 are 2x20 FEMALE headers on the panel's INNER face (B.Cu); they mate J6 / J7 / J8, the male headers on the main board's bottom side."
- note removed: "With that mirror, panel pad k mates main-board pin k on all three headers (the KiCad PinSocket footprint already carries the mating mirror). gen_panel.py proves it from the pad coordinates before the board is written."

Commit message: Boards as hand-reworked by the instructor 2026-09-18 (Decision #66): three 2x20 links re-placed, jumpers -> headers, TCXO removed, 16 SMA; layout and routing in progress; review in the course repo notes
Co-Authored-By: Claude Fable 5.1 <noreply@anthropic.com>
Parts:
- removed D2: YELLOW, class_board:LED0603-RD-YELLOW, symbol class_board:LED_YELLOW_0603
- removed J1, J2, J3: Panel link 2x20 male, Connector_PinHeader_2.54mm:PinHeader_2x20_P2.54mm_Vertical, symbol class_board:HDR_2x20_MALE
- removed J26: SMA, class_board:SMA-TH_BWSMA-KE-Z001, symbol class_board:BWSMA-KE-Z001
- removed TP1: TP, class_board:TestPoint_Pad_D1.5mm, symbol class_board:TestPoint
- added D2: GREEN, class_board:LED0805-R-RD, symbol class_board:LED_GREEN_0805
- added J1, J2, J3: Conn_02x20_Odd_Even, Connector_PinHeader_2.54mm:PinHeader_2x20_P2.54mm_Vertical, symbol Connector_Generic:Conn_02x20_Odd_Even
Connections:
- net +3V3: now also J2.27 (Pin_27), J2.29 (Pin_29), J3.5 (Pin_5)
- net +5V_RAW: now also J3.1 (Pin_1), J3.3 (Pin_3)
- net AGND: now also J1.1 (Pin_1), J1.11 (Pin_11), J1.13 (Pin_13), J1.15 (Pin_15), J1.17 (Pin_17), J1.19 (Pin_19), J1.21 (Pin_21), J1.23 (Pin_23), J1.25 (Pin_25), J1.27 (Pin_27), J1.29 (Pin_29), J1.3 (Pin_3), J1.31 (Pin_31), J1.33 (Pin_33), J1.35 (Pin_35), J1.37 (Pin_37), J1.39 (Pin_39), J1.5 (Pin_5), J1.7 (Pin_7), J1.9 (Pin_9)
- net AI1: now also J1.40 (Pin_40)
- net AI2: now also J1.38 (Pin_38)
- net AI3: now also J1.36 (Pin_36)
- net AI4: now also J1.34 (Pin_34)
- net AI5: now also J1.30 (Pin_30)
- net AI6: now also J1.28 (Pin_28)
- net AI7: now also J1.26 (Pin_26)
- net AI8: now also J1.24 (Pin_24)
- net AO1: now also J1.18 (Pin_18)
- net AO2: now also J1.16 (Pin_16)
- net AUX: now also J1.12 (Pin_12)
- net FASTTTL1: now also J2.39 (Pin_39)
- net FASTTTL2: now also J2.37 (Pin_37)
- net GND: now also D2.1 (K), J2.10 (Pin_10), J2.12 (Pin_12), J2.14 (Pin_14), J2.16 (Pin_16), J2.18 (Pin_18), J2.2 (Pin_2), J2.20 (Pin_20), J2.22 (Pin_22), J2.24 (Pin_24), J2.26 (Pin_26), J2.28 (Pin_28), J2.30 (Pin_30), J2.32 (Pin_32), J2.34 (Pin_34), J2.36 (Pin_36), J2.38 (Pin_38), J2.4 (Pin_4), J2.40 (Pin_40), J2.6 (Pin_6), J2.8 (Pin_8), J3.10 (Pin_10), J3.12 (Pin_12), J3.14 (Pin_14), J3.16 (Pin_16), J3.18 (Pin_18), J3.2 (Pin_2), J3.20 (Pin_20), J3.22 (Pin_22), J3.24 (Pin_24), J3.26 (Pin_26), J3.28 (Pin_28), J3.30 (Pin_30), J3.32 (Pin_32), J3.34 (Pin_34), J3.36 (Pin_36), J3.38 (Pin_38), J3.4 (Pin_4), J3.40 (Pin_40), J3.6 (Pin_6), J3.8 (Pin_8)
- net I2C_SCL: now also J2.31 (Pin_31)
- net I2C_SDA: now also J2.33 (Pin_33)
- net LED_ACT: now also J2.23 (Pin_23)
- net LED_WIFI: now also J2.25 (Pin_25)
- net LED_WIFI_A: now also D2.2 (A)
- net MOD1: now also J3.23 (Pin_23)
- net MOD2: now also J3.25 (Pin_25)
- net MOD3: now also J3.27 (Pin_27)
- net MOD4: now also J3.29 (Pin_29)
- net MOD5: now also J3.31 (Pin_31)
- net MOD6: now also J3.33 (Pin_33)
- net MOD7: now also J3.35 (Pin_35)
- net OPTO_IN1: now also J3.15 (Pin_15)
- net OPTO_IN2: now also J3.17 (Pin_17)
- net RX: now also J1.32 (Pin_32)
- net TRIG_5V: now also J2.35 (Pin_35)
- net TTL1: now also J2.15 (Pin_15)
- net TTL2: now also J2.13 (Pin_13)
- net TTL3: now also J2.11 (Pin_11)
- net TTL4: now also J2.9 (Pin_9)
- net TTL5: now also J2.7 (Pin_7)
- net TTL6: now also J2.5 (Pin_5)
- net TTL7: now also J2.3 (Pin_3)
- net TTL8: now also J2.1 (Pin_1)
- net TX: now also J1.20 (Pin_20), J1.22 (Pin_22)
- no-connect marks 14 -> 21
Other:
- note added: "GPIO15"
- note added: "GPIO4"
- note added: "GPIO43"
- note added: "GPIO44"
- note added: "GPIO6"
- note added: "GPIO7"
- note added: "J1xtra - digital (inner face): mates J7, the digital header"
- note added: "MOD8"
- note removed: "J2 - digital (inner face): mates J7, the digital header"
- note removed: "panel label: SPARE (115, 61) mm"
- note removed: "panel x = 90 mm (main board x = 90 mm)"
- moved on the sheet: C401, C402, C410, D422, FID1, FID2, H1, H2, H3, H4, R1, R2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

Commit message: WIP masters (instructor), 2026-09-24 14:26
Co-Authored-By: Claude Fable 5.1 <noreply@anthropic.com>
Connections:
- net AGND: no longer J12.1 (GND), J12.2 (GND), J12.3 (GND), J12.4 (GND), J15.1 (GND), J15.2 (GND), J15.3 (GND), J15.4 (GND), J21.1 (GND), J21.2 (GND), J21.3 (GND), J21.4 (GND)
- net GND: now also J12.1 (GND), J12.2 (GND), J12.3 (GND), J12.4 (GND), J15.1 (GND), J15.2 (GND), J15.3 (GND), J15.4 (GND), J21.1 (GND), J21.2 (GND), J21.3 (GND), J21.4 (GND)
Other:
- moved on the sheet: R2

Commit message: hardware: instructor's masters of 2026-09-25 04:25 (main board) and 2026-09-24 22:43 (panel + schematic)
Co-Authored-By: Claude Fable 5.1 <noreply@anthropic.com>
Connections:
- net RX: now also J14.5 (SIG); no longer J20.5 (SIG)
- net TX: now also J20.5 (SIG); no longer J14.5 (SIG)
Changed lines of the file:
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@@
 		)
 	)
-	(label "TX"
+	(label "RX"
 		(at 411.48 209.55 180)
 		(effects
@@
 		)
 	)
-	(label "RX"
+	(label "TX"
 		(at 411.48 265.43 180)
 		(effects

Commit message: hardware: front panel as saved 2026-09-30 22:15
Co-Authored-By: Claude Fable 5.1 <noreply@anthropic.com>
Connections:
- net AGND: no longer J1.1 (Pin_1), J1.11 (Pin_11), J1.13 (Pin_13), J1.3 (Pin_3), J1.5 (Pin_5), J1.7 (Pin_7), J1.9 (Pin_9), J20.1 (GND), J20.2 (GND), J20.3 (GND), J20.4 (GND), J32.2
- net AUX: now also J1.20 (Pin_20); no longer J1.12 (Pin_12)
- net GND: now also J1.1 (Pin_1), J1.11 (Pin_11), J1.3 (Pin_3), J1.5 (Pin_5), J1.7 (Pin_7), J1.9 (Pin_9), J20.1 (GND), J20.2 (GND), J20.3 (GND), J20.4 (GND), J32.2
- net RX: now also J1.22 (Pin_22); no longer J1.32 (Pin_32)
- net TX: now also J1.10 (Pin_10), J1.12 (Pin_12); no longer J1.20 (Pin_20), J1.22 (Pin_22)
- no-connect marks 21 -> 22

Commit message: Schematic review fixes, part 2 (Konnect): panel RX/AUX labels + SMA labels swapped to match the main board (copper unchanged); TX_VMID -> R820 47k -> TX_IN (C810 couples into TX_IN); Q901 D/S corrected + D932 to +VEXT; R950 10k Q904 gate-source; R712 permanent (J3 pin 1 tied to pin 2); U302/C308 on +5VA; panel 6N137 VCC/VE + C401/C402 on +5V_RAW; R521-R528 DIO pull-downs; front_panel_link sheet removed from the root; change notes on six sheets; panel silk: pairing labels corrected, stale J3 texts deleted, TX/RX/AUX labels fixed, OUT1..7. ERC unchanged (2 cosmetic), panel DRC 0/0; netlist diff = intended changes only
Co-Authored-By: Claude Fable 5.1 <noreply@anthropic.com>
Connections:
- net +3V3: no longer C401.1, C402.1, U401.7 (VE), U401.8 (VCC), U402.7 (VE), U402.8 (VCC)
- net +5V_RAW: now also C401.1, C402.1, U401.7 (VE), U401.8 (VCC), U402.7 (VE), U402.8 (VCC)
- net AUX: now also J1.22 (Pin_22), J14.5 (SIG); no longer J1.20 (Pin_20), J13.5 (SIG)
- net RX: now also J1.20 (Pin_20), J13.5 (SIG); no longer J1.22 (Pin_22), J14.5 (SIG)
Other:
- note added: "2026-10-01: U401/U402 6N137 VCC and VE now on +5V_RAW (spec 4.5-5.5 V); the output pull-ups R471/R472 stay on +3V3 (GPIO16/17 are not 5 V tolerant). J1 pin 20 = RX (SMA J13, receiver tank), pin 22 = AUX (SMA J14, R715 option), matching the main board."

Commit message: hardware: instructor 2026-10-01 saves synced (one GND net on both boards, PCB updated, R951-R958, headers DNP per Decision #73) + nmr_tx R808 -> TX_VMID, C813 removed, R805/R806 10 k (review B2)
Co-Authored-By: Claude Fable 5.1 <noreply@anthropic.com>
Parts:
- J1, J2, J3, J40: now not fitted; now left out of the parts list
Connections:
- net AGND is gone; now on net GND: J1.15 (Pin_15), J1.17 (Pin_17), J1.19 (Pin_19), J1.21 (Pin_21), J1.23 (Pin_23), J1.25 (Pin_25), J1.27 (Pin_27), J1.29 (Pin_29), J1.31 (Pin_31), J1.33 (Pin_33), J1.35 (Pin_35), J1.37 (Pin_37), J1.39 (Pin_39), J10.1 (GND), J10.2 (GND), J10.3 (GND), J10.4 (GND), J11.1 (GND), J11.2 (GND), J11.3 (GND), J11.4 (GND), J13.1 (GND), J13.2 (GND), J13.3 (GND), J13.4 (GND), J14.1 (GND), J14.2 (GND), J14.3 (GND), J14.4 (GND), J16.1 (GND), J16.2 (GND), J16.3 (GND), J16.4 (GND), J17.1 (GND), J17.2 (GND), J17.3 (GND), J17.4 (GND), J18.1 (GND), J18.2 (GND), J18.3 (GND), J18.4 (GND), J19.1 (GND), J19.2 (GND), J19.3 (GND), J19.4 (GND), J22.1 (GND), J22.2 (GND), J22.3 (GND), J22.4 (GND), J23.1 (GND), J23.2 (GND), J23.3 (GND), J23.4 (GND), J24.1 (GND), J24.2 (GND), J24.3 (GND), J24.4 (GND), J25.1 (GND), J25.2 (GND), J25.3 (GND), J25.4 (GND)
- net GND: now also J1.13 (Pin_13)
- no-connect marks 22 -> 21
