File: hardware/front-panel/front-panel.kicad_sch (KiCad schematic)
At the start: 76 parts, among them J1 Conn_02x20_Odd_Even, J10 SMA, J11 SMA, J12 SMA, J13 SMA, J14 SMA, J15 SMA, J16 SMA, J17 SMA, J18 SMA, J19 SMA, J2 Conn_02x20_Odd_Even, J20 SMA, J21 SMA, J22 SMA, J23 SMA, J24 SMA, J25 SMA, J3 Conn_02x20_Odd_Even, J30 OLED 0.96in module on 1x4 soc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, J31 KF128-2.54-10P, J32 KF128-5.0-2P, J33 Qwiic (vertical), J40 Module header 2x6 (shrouded), J411 KF301-5.0-2P, J412 KF301-5.0-2P, Q411 MMBT5551, Q412 MMBT5551, Q421 MMBT5551, Q422 MMBT5551, U401 6N137S-TA1-L, U402 6N137S-TA1-L, U410 SN74AHCT541PWR

Commit message: Final boards (2026-10-01 23:44/23:48 saves) and re-exported release STEP models
- class-board and front-panel: DNP + out-of-BOM flags on the hand-soldered connectors, panel 3D-model paths on TIGP_BOARD_LIB, schematic sheets in step
- hardware/release: class-board.step and front-panel.step re-exported from these boards (filters as before, now without --no-dnp so the hand-soldered connectors keep their bodies; panel exported directly, no path-redirect copy); the STL meshes are unchanged (same triangles and bounding boxes)
- README: export note

Co-Authored-By: Claude Fable 5.1 <noreply@anthropic.com>
Parts:
- J1, J2, J3, J40: now fitted; now in the parts list
Changed lines of the file:
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@@
 		(body_style 1)
 		(exclude_from_sim no)
-		(in_bom no)
+		(in_bom yes)
 		(on_board yes)
 		(in_pos_files yes)
-		(dnp yes)
+		(dnp no)
 		(fields_autoplaced yes)
 		(property "Reference" "J40"
@@
 		(body_style 1)
 		(exclude_from_sim no)
-		(in_bom no)
+		(in_bom yes)
 		(on_board yes)
 		(in_pos_files yes)
-		(dnp yes)
+		(dnp no)
 		(property "Reference" "J3"
 			(at 66.294 65.278 0)
@@
 		(body_style 1)
 		(exclude_from_sim no)
-		(in_bom no)
+		(in_bom yes)
 		(on_board yes)
 		(in_pos_files yes)
-		(dnp yes)
+		(dnp no)
 		(property "Reference" "J2"
 			(at 245.872 124.46 0)
@@
 		(body_style 1)
 		(exclude_from_sim no)
-		(in_bom no)
+		(in_bom yes)
 		(on_board yes)
 		(in_pos_files yes)
-		(dnp yes)
+		(dnp no)
 		(property "Reference" "J1"
 			(at 398.018 66.04 0)

Commit message: LED polarity fixed in the design (synced from the class repo main aaaec0f)
Co-Authored-By: Claude Fable 5.1 <noreply@anthropic.com>
Connections:
- net GND: now also D1.2 (K), D2.2 (K), D3.2 (K); no longer D1.1 (K), D2.1 (K), D3.1 (K)
- net LED_ACT_A: now also D3.1 (A); no longer D3.2 (A)
- net LED_PWR_A: now also D1.1 (A); no longer D1.2 (A)
- net LED_WIFI_A: now also D2.1 (A); no longer D2.2 (A)
