File: hardware/front-panel/front-panel.kicad_pcb (KiCad board)
At the start: 4 copper layers, 180 x 100 mm, 76 parts, among them J1 Conn_02x20_Odd_Even, J10 SMA, J11 SMA, J12 SMA, J13 SMA, J14 SMA, J15 SMA, J16 SMA, J17 SMA, J18 SMA, J19 SMA, J2 Conn_02x20_Odd_Even, J20 SMA, J21 SMA, J22 SMA, J23 SMA, J24 SMA, J25 SMA, J3 Conn_02x20_Odd_Even, J30 OLED 0.96in module on 1x4 soc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, J31 KF128-2.54-10P, J32 KF128-5.0-2P, J33 Qwiic (vertical), J40 Module header 2x6 (shrouded), J411 KF301-5.0-2P, J412 KF301-5.0-2P, Q411 MMBT5551, Q412 MMBT5551, Q421 MMBT5551, Q422 MMBT5551, U401 6N137S-TA1-L, U402 6N137S-TA1-L, U410 SN74AHCT541PWR

Commit message: LED polarity fixed in the design (synced from the class repo main aaaec0f)
Co-Authored-By: Claude Fable 5.1 <noreply@anthropic.com>
Parts:
- turned D1 to 0 degrees
- turned D2 to 0 degrees
- turned D3 to 0 degrees
Connections:
- D1 pad 1: GND -> /LED_PWR_A
- D1 pad 2: /LED_PWR_A -> GND
- D2 pad 1: GND -> /LED_WIFI_A
- D2 pad 2: /LED_WIFI_A -> GND
- D3 pad 1: GND -> /LED_ACT_A
- D3 pad 2: /LED_ACT_A -> GND
Changed lines of the file:
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@@
 	(footprint "class_board:LED0805-R-RD"
 		(layer "F.Cu")
-		(at 116.450004 92.85 180)
+		(at 116.450004 92.85)
 		(descr "0805")
 		(property "Reference" "D3"
@@
 		(duplicate_pad_numbers_are_jumpers no)
 		(fp_line
-			(start 1.99 1.019999)
-			(end 1.99 -1.01)
+			(start -2.22 -0.63)
+			(end -1.84 -1.01)
 			(stroke
 				(width 0.25)
@@
 		)
 		(fp_line
-			(start 1.99 -1.01)
-			(end 0.44 -1.01)
+			(start -2.22 0.64)
+			(end -2.22 -0.63)
 			(stroke
 				(width 0.25)
@@
 		)
 		(fp_line
-			(start 0.44 1.02)
-			(end 1.99 1.019999)
+			(start -1.84 -1.01)
+			(end -0.32 -1.01)
 			(stroke
 				(width 0.25)
@@
 		)
 		(fp_line
-			(start 0.2 -0.5)
-			(end 0.2 0.5)
+			(start -1.82 1.04)
+			(end -2.22 0.64)
 			(stroke
 				(width 0.25)
@@
 		)
 		(fp_line
-			(start 0.2 -0.5)
-			(end -0.2 -0.1)
+			(start -0.34 1.04)
+			(end -1.82 1.04)
 			(stroke
 				(width 0.25)
@@
 		)
 		(fp_line
-			(start -0.2 0.1)
-			(end 0.2 0.5)
+			(start -0.3 0)
+			(end -0.2 0.1)
 			(stroke
 				(width 0.25)
@@
 		)
 		(fp_line
-			(start -0.3 0)
-			(end -0.2 0.1)
+			(start -0.2 0.1)
+			(end 0.2 0.5)
 			(stroke
 				(width 0.25)
@@
 		)
 		(fp_line
-			(start -0.34 1.04)
-			(end -1.82 1.04)
+			(start 0.2 -0.5)
+			(end -0.2 -0.1)
 			(stroke
 				(width 0.25)
@@
 		)
 		(fp_line
-			(start -1.82 1.04)
-			(end -2.22 0.64)
+			(start 0.2 -0.5)
+			(end 0.2 0.5)
 			(stroke
 				(width 0.25)
@@
 		)
 		(fp_line
-			(start -1.84 -1.01)
-			(end -0.32 -1.01)
+			(start 0.44 1.02)
+			(end 1.99 1.019999)
 			(stroke
 				(width 0.25)
@@
 		)
 		(fp_line
-			(start -2.22 0.64)
-			(end -2.22 -0.63)
+			(start 1.99 -1.01)
+			(end 0.44 -1.01)
 			(stroke
 				(width 0.25)
@@
 		)
 		(fp_line
-			(start -2.22 -0.63)
-			(end -1.84 -1.01)
+			(start 1.99 1.019999)
+			(end 1.99 -1.01)
 			(stroke
 				(width 0.25)
@@
 		)
 		(pad "1" smd rect
-			(at 1.05 0)
+			(at 1.05 0 180)
 			(size 1 1.4)
 			(layers "F.Cu" "F.Mask" "F.Paste")
-			(net "GND")
+			(net "/LED_ACT_A")
 			(pinfunction "K_1")
 			(pintype "passive")
 		)
 		(pad "2" smd rect
-			(at -1.05 0)
+			(at -1.05 0 180)
 			(size 1 1.4)
 			(layers "F.Cu" "F.Mask" "F.Paste")
-			(net "/LED_ACT_A")
+			(net "GND")
 			(pinfunction "A_2")
 			(pintype "passive")
@@
 	(footprint "class_board:LED0805-R-RD"
 		(layer "F.Cu")
-		(at 116.5 89.9 180)
+		(at 116.5 89.9)
 		(descr "0805")
 		(property "Reference" "D2"
@@
 		)
 		(property "LCSC" "C2297"
-			(at 0 0 180)
+			(at 0 0 0)
 			(unlocked yes)
 			(layer "F.Fab")
@@
 		)
 		(property "JLC_CLASS" "Basic"
-			(at 0 0 180)
+			(at 0 0 0)
 			(unlocked yes)
 			(layer "F.Fab")
@@
 		)
 		(property "MPN" "KT-0805G"
-			(at 0 0 180)
+			(at 0 0 0)
 			(unlocked yes)
 			(layer "F.Fab")
@@
 		)
 		(property "Manufacturer" "Hubei KENTO"
-			(at 0 0 180)
+			(at 0 0 0)
 			(unlocked yes)
 			(layer "F.Fab")
@@
 		)
 		(property "Block" "PANEL"
-			(at 0 0 180)
+			(at 0 0 0)
 			(unlocked yes)
 			(layer "F.Fab")
@@
 		(duplicate_pad_numbers_are_jumpers no)
 		(fp_line
-			(start 1.99 1.019999)
-			(end 1.99 -1.01)
+			(start -2.22 -0.63)
+			(end -1.84 -1.01)
 			(stroke
 				(width 0.25)
@@
 		)
 		(fp_line
-			(start 1.99 -1.01)
-			(end 0.44 -1.01)
+			(start -2.22 0.64)
+			(end -2.22 -0.63)
 			(stroke
 				(width 0.25)
@@
 		)
 		(fp_line
-			(start 0.44 1.02)
-			(end 1.99 1.019999)
+			(start -1.84 -1.01)
+			(end -0.32 -1.01)
 			(stroke
 				(width 0.25)
@@
 		)
 		(fp_line
-			(start 0.2 -0.5)
-			(end 0.2 0.5)
+			(start -1.82 1.04)
+			(end -2.22 0.64)
 			(stroke
 				(width 0.25)
@@
 		)
 		(fp_line
-			(start 0.2 -0.5)
-			(end -0.2 -0.1)
+			(start -0.34 1.04)
+			(end -1.82 1.04)
 			(stroke
 				(width 0.25)
@@
 		)
 		(fp_line
-			(start -0.2 0.1)
-			(end 0.2 0.5)
+			(start -0.3 0)
+			(end -0.2 0.1)
 			(stroke
 				(width 0.25)
@@
 		)
 		(fp_line
-			(start -0.3 0)
-			(end -0.2 0.1)
+			(start -0.2 0.1)
+			(end 0.2 0.5)
 			(stroke
 				(width 0.25)
@@
 		)
 		(fp_line
-			(start -0.34 1.04)
-			(end -1.82 1.04)
+			(start 0.2 -0.5)
+			(end -0.2 -0.1)
 			(stroke
 				(width 0.25)
@@
 		)
 		(fp_line
-			(start -1.82 1.04)
-			(end -2.22 0.64)
+			(start 0.2 -0.5)
+			(end 0.2 0.5)
 			(stroke
 				(width 0.25)
@@
 		)
 		(fp_line
-			(start -1.84 -1.01)
-			(end -0.32 -1.01)
+			(start 0.44 1.02)
+			(end 1.99 1.019999)
 			(stroke
 				(width 0.25)
@@
 		)
 		(fp_line
-			(start -2.22 0.64)
-			(end -2.22 -0.63)
+			(start 1.99 -1.01)
+			(end 0.44 -1.01)
 			(stroke
 				(width 0.25)
@@
 		)
 		(fp_line
-			(start -2.22 -0.63)
-			(end -1.84 -1.01)
+			(start 1.99 1.019999)
+			(end 1.99 -1.01)
 			(stroke
 				(width 0.25)
@@
 		)
 		(pad "1" smd rect
-			(at 1.05 0)
+			(at 1.05 0 180)
 			(size 1 1.4)
 			(layers "F.Cu" "F.Mask" "F.Paste")
-			(net "GND")
+			(net "/LED_WIFI_A")
 			(pinfunction "K_1")
 			(pintype "passive")
 		)
 		(pad "2" smd rect
-			(at -1.05 0)
+			(at -1.05 0 180)
 			(size 1 1.4)
 			(layers "F.Cu" "F.Mask" "F.Paste")
-			(net "/LED_WIFI_A")
+			(net "GND")
 			(pinfunction "A_2")
 			(pintype "passive")
@@
 	(footprint "class_board:LED0805-R-RD"
 		(layer "F.Cu")
-		(at 116.5 86.95 180)
+		(at 116.5 86.95)
 		(descr "0805")
 		(property "Reference" "D1"
@@
 		(duplicate_pad_numbers_are_jumpers no)
 		(fp_line
-			(start 1.99 1.019999)
-			(end 1.99 -1.01)
+			(start -2.22 -0.63)
+			(end -1.84 -1.01)
 			(stroke
 				(width 0.25)
@@
 		)
 		(fp_line
-			(start 1.99 -1.01)
-			(end 0.44 -1.01)
+			(start -2.22 0.64)
+			(end -2.22 -0.63)
 			(stroke
 				(width 0.25)
@@
 		)
 		(fp_line
-			(start 0.44 1.02)
-			(end 1.99 1.019999)
+			(start -1.84 -1.01)
+			(end -0.32 -1.01)
 			(stroke
 				(width 0.25)
@@
 		)
 		(fp_line
-			(start 0.2 -0.5)
-			(end 0.2 0.5)
+			(start -1.82 1.04)
+			(end -2.22 0.64)
 			(stroke
 				(width 0.25)
@@
 		)
 		(fp_line
-			(start 0.2 -0.5)
-			(end -0.2 -0.1)
+			(start -0.34 1.04)
+			(end -1.82 1.04)
 			(stroke
 				(width 0.25)
@@
 		)
 		(fp_line
-			(start -0.2 0.1)
-			(end 0.2 0.5)
+			(start -0.3 0)
+			(end -0.2 0.1)
 			(stroke
 				(width 0.25)
@@
 		)
 		(fp_line
-			(start -0.3 0)
-			(end -0.2 0.1)
+			(start -0.2 0.1)
+			(end 0.2 0.5)
 			(stroke
 				(width 0.25)
@@
 		)
 		(fp_line
-			(start -0.34 1.04)
-			(end -1.82 1.04)
+			(start 0.2 -0.5)
+			(end -0.2 -0.1)
 			(stroke
 				(width 0.25)
@@
 		)
 		(fp_line
-			(start -1.82 1.04)
-			(end -2.22 0.64)
+			(start 0.2 -0.5)
+			(end 0.2 0.5)
 			(stroke
 				(width 0.25)
@@
 		)
 		(fp_line
-			(start -1.84 -1.01)
-			(end -0.32 -1.01)
+			(start 0.44 1.02)
+			(end 1.99 1.019999)
 			(stroke
 				(width 0.25)
@@
 		)
 		(fp_line
-			(start -2.22 0.64)
-			(end -2.22 -0.63)
+			(start 1.99 -1.01)
+			(end 0.44 -1.01)
 			(stroke
 				(width 0.25)
@@
 		)
 		(fp_line
-			(start -2.22 -0.63)
-			(end -1.84 -1.01)
+			(start 1.99 1.019999)
+			(end 1.99 -1.01)
 			(stroke
 				(width 0.25)
@@
 		)
 		(pad "1" smd rect
-			(at 1.05 0)
+			(at 1.05 0 180)
 			(size 1 1.4)
 			(layers "F.Cu" "F.Mask" "F.Paste")
-			(net "GND")
+			(net "/LED_PWR_A")
 			(pinfunction "K_1")
 			(pintype "passive")
 		)
 		(pad "2" smd rect
-			(at -1.05 0)
+			(at -1.05 0 180)
 			(size 1 1.4)
 			(layers "F.Cu" "F.Mask" "F.Paste")
-			(net "/LED_PWR_A")
+			(net "GND")
 			(pinfunction "A_2")
 			(pintype "passive")
