File: hardware/class-board.kicad_pcb (KiCad board)
At the start: 4 copper layers, 180 x 100 mm, 341 parts, among them J1 DevKit J1 (left row), J2 DevKit J3 (right row), J201 USB-C 16P, J202 DC005-T20, J4 Qwiic, J5 Expansion 2x10, J6 Panel link 2x20 female, J7 Panel link 2x20 female, J8 Panel link 2x20 female, J901 KF301-5.0-2P, J903 KF301-5.0-2P, J905 KF301-5.0-3P, Q901 AOD4185, Q904 AOD4184A, U101 ADS8688IDBTR, U201 LM66100DCKR, U202 LM66100DCKR, U203 78L05G-AB3-R, U204 AMS1117-3.3, U301 DAC8563SDGSR, U302 74HCT125PW, U303 OPA2192IDR, U501 SN74AHCT541PWR, U502 74HCT125PW, U503 SN74LVC1T45DBVR, U504 SN74LVC1G17DBVR, U505 TCA9535PWR, U701 SI5351A-B-GT, U702 74HC74D,653, U703 OPA1656IDR, U704 DG419DY-T1-E3, U705 OPA1612AIDR, U706 OPA1612AIDR, U801 AD9834BRUZ, U802 OPA564AIDWPR, U901 TS5A23157DGSR, U902 TS5A23157DGSR, U903 DRV8871DDAR, U904 UCC27517DBVR, X501 10 MHz TCXO, Y701 25 MHz

Commit message: Boards as hand-reworked by the instructor 2026-09-18 (Decision #66): three 2x20 links re-placed, jumpers -> headers, TCXO removed, 16 SMA; layout and routing in progress; review in the course repo notes
Co-Authored-By: Claude Fable 5.1 <noreply@anthropic.com>
Parts:
- removed C505: 1nF, Capacitor_SMD:C_0603_1608Metric
- removed C506: 100nF, Capacitor_SMD:C_0603_1608Metric
- removed JP501: SolderJumper_2_Open, class_board:SolderJumper-2_P1.3mm_Open_RoundedPad1.0x1.5mm
- removed JP701: AUX -> LNA (open), class_board:SolderJumper-3_P1.3mm_Open_RoundedPad1.0x1.5mm
- removed JP702: G=101 / G=11, class_board:SolderJumper-3_P1.3mm_Bridged12_RoundedPad1.0x1.5mm
- removed JP703: open = G 1, class_board:SolderJumper-2_P1.3mm_Bridged_RoundedPad1.0x1.5mm
- removed JP801, JP802, JP904: SolderJumper_3_Bridged12, class_board:SolderJumper-3_P1.3mm_Bridged12_RoundedPad1.0x1.5mm
- removed R512, R513, R514, R515: 100k, Resistor_SMD:R_0603_1608Metric
- removed U504: SN74LVC1G17DBVR, class_board:SOT-23-5_L3.0-W1.7-P0.95-LS2.8-BR
- removed X501: 10 MHz TCXO, class_board:OSC-SMD_4P-L3.2-W2.5-BL
- added J10: C2937625_-_Conn_01x03, DDS_Library:C2937625-HDR-TH_3P-P2.54-V-M, F.Cu at (363.1, 71.8)
- added J11: C2937625_-_Conn_01x03, DDS_Library:C2937625-HDR-TH_3P-P2.54-V-M, F.Cu at (336.5, 159.4)
- added J12: C2937625_-_Conn_01x03, DDS_Library:C2937625-HDR-TH_3P-P2.54-V-M, F.Cu at (69.2, 44.5)
- added J13: C492401-PZ254V-11-02P, mike_JLCPCB:C492401-HDR-TH_2P-P2.54-V-M, F.Cu at (81.1, 40.0)
- added J3: C2937625_-_Conn_01x03, DDS_Library:C2937625-HDR-TH_3P-P2.54-V-M, F.Cu at (236.8, 179.4)
- added J9: C2937625_-_Conn_01x03, DDS_Library:C2937625-HDR-TH_3P-P2.54-V-M, F.Cu at (231.0, 198.9)
- added R715: 0, Resistor_SMD:R_0805_2012Metric_Pad1.20x1.40mm_HandSolder, F.Cu at (227.6, 182.8)
- added R716: 0, Resistor_SMD:R_0805_2012Metric_Pad1.20x1.40mm_HandSolder, F.Cu at (227.6, 189.0)
- moved U704 252.0 mm to (244.8, 189.1)
- moved R724 238.7 mm to (245.4, 183.2)
- moved R723 234.3 mm to (231.1, 195.4), turned to -90 degrees
- moved R721 232.0 mm to (240.8, 191.2)
- moved C720 231.6 mm to (239.8, 188.3), turned to 0 degrees
- moved R722 225.8 mm to (233.8, 194.6), turned to 0 degrees
- moved C721 224.8 mm to (233.8, 196.2), turned to 0 degrees
- moved C917 208.6 mm to (162.7, 229.3)
- moved C725 207.2 mm to (169.9, 229.3)
- moved C919 206.7 mm to (164.4, 229.3)
- moved C727 206.2 mm to (168.1, 229.2), turned to 90 degrees
- moved C905 205.2 mm to (171.4, 205.3), turned to 90 degrees
- moved FB901 204.7 mm to (166.2, 206.2), turned to 180 degrees
- moved C906 204.1 mm to (173.5, 205.4)
- moved C907 203.8 mm to (175.3, 205.4)
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Connections:
- net +3V3D renamed /nmr_tx/+3V3D
- net /nmr_rx/CLK2_TP renamed Net-(R705-Pad2)
- net /nmr_rx/SI_CLK0 renamed Net-(U701-CLK0)
- net /nmr_rx/SI_CLK1 renamed Net-(U701-CLK1)
- net /nmr_rx/SI_CLK2 renamed Net-(U701-CLK2)
- net CLK0_MCLK renamed /nmr_rx/CLK0_MCLK
- net COND_OUT1 renamed /b1_inputs/COND_OUT1
- net COND_OUT2 renamed /b1_inputs/COND_OUT2
- net CS_ADC renamed /b1_inputs/CS_ADC
- net CS_DAC renamed /b3_outputs/CS_DAC
- net DDS_FSYNC renamed /base_mcu/DDS_FSYNC
- net DDS_PSEL renamed /base_mcu/DDS_PSEL
- net DDS_RESET renamed /nmr_tx/DDS_RESET
- net DDS_SLEEP renamed /nmr_tx/DDS_SLEEP
- net DIO1 renamed /b5_dio_trig/DIO1
- net DIO2 renamed /b5_dio_trig/DIO2
- net DIO3 renamed /b5_dio_trig/DIO3
- net DIO4 renamed /b5_dio_trig/DIO4
- net DIO5 renamed /b5_dio_trig/DIO5
- net DIO6 renamed /b5_dio_trig/DIO6
- net DIO7 renamed /b5_dio_trig/DIO7
- net DIO8 renamed /b5_dio_trig/DIO8
- net EXP_P14 renamed /b5_dio_trig/EXP_P14
- net FET_GATE renamed /base_mcu/FET_GATE
- net HB_IN1 renamed /base_mcu/HB_IN1
- net HB_IN2 renamed /base_mcu/HB_IN2
- net ISENSE_COIL renamed /c_switch/ISENSE_COIL
- net RX_BLANK renamed /base_mcu/RX_BLANK
- net TRIG_DIR renamed /b5_dio_trig/TRIG_DIR
- net TRIG_IO renamed /base_mcu/TRIG_IO
- net TX_EN renamed /base_mcu/TX_EN
- net TX_IFLAG renamed /nmr_tx/TX_IFLAG
- net TX_TFLAG renamed /nmr_tx/TX_TFLAG
- net USB_DN renamed /b2_power/USB_D_N
- net USB_DP renamed /b2_power/USB_D_P
- net VREF_DAC renamed /b3_outputs/VREF_DAC
- C203 pad 1: GND -> Net-(D201-K)
- C204 pad 1: GND -> Net-(D202-K)
- C710 pad 1: RX -> AGND
- C710 pad 2: AGND -> /b1_inputs/AUX
- C711 pad 1: RX -> AGND
- C711 pad 2: AGND -> /b1_inputs/AUX
- C712 pad 1: RX -> AGND
- C712 pad 2: AGND -> /b1_inputs/AUX
- C910 pad 1: /nmr_rx/IF_IPF -> V_MID
- C910 pad 2: V_MID -> /nmr_rx/IF_IPF
- C911 pad 1: /nmr_rx/IF_QPF -> V_MID
- C911 pad 2: V_MID -> /nmr_rx/IF_QPF
- D201 pad 1: GND -> Net-(D201-K)
- D202 pad 1: GND -> Net-(D202-K)
- D301 pad 3: AO1 -> /b1_inputs/AO1
- D302 pad 3: AO2 -> /b1_inputs/AO2
- D501 pad 3: TRIG_5V -> /b5_dio_trig/TRIG_5V
- D703 pad 2: RX -> /b1_inputs/AUX
- D704 pad 1: RX -> /b1_inputs/AUX
- F201 pad 2: GND -> Net-(D201-K)
- F202 pad 2: GND -> Net-(D202-K)
- J1 pad 10: OPTO_IN2 -> /b5_dio_trig/OPTO_IN2
- J1 pad 11: FAST_OUT1 -> /b5_dio_trig/FAST_OUT2
- J1 pad 4: GPIO4 -> /base_mcu/GPIO4
- J1 pad 6: GPIO6 -> /base_mcu/GPIO6
- J1 pad 7: GPIO7 -> /base_mcu/GPIO7
- J1 pad 8: GPIO15 -> /base_mcu/GPIO15
- J1 pad 9: OPTO_IN1 -> /b5_dio_trig/OPTO_IN1
- J2 pad 18: FAST_OUT2 -> /b5_dio_trig/FAST_OUT1
- J2 pad 2: GPIO43 -> /base_mcu/GPIO43
- J2 pad 3: GPIO44 -> /base_mcu/GPIO44
- J5 pad 14: GPIO43 -> /base_mcu/GPIO43
- J5 pad 15: GPIO44 -> /base_mcu/GPIO44
- J5 pad 16: GPIO4 -> /base_mcu/GPIO4
- J5 pad 17: GPIO6 -> /base_mcu/GPIO6
- J5 pad 19: GPIO7 -> /base_mcu/GPIO7
- J5 pad 20: GPIO15 -> /base_mcu/GPIO15
- J6 pad 1: AI1 -> AGND
- J6 pad 10: AGND -> unconnected-(J6-Pad10)
- J6 pad 11: AI6 -> AGND
- J6 pad 12: AGND -> /b1_inputs/AUX
- J6 pad 13: AI7 -> AGND
- J6 pad 14: AGND -> unconnected-(J6-Pad14)
- J6 pad 15: AI8 -> AGND
- J6 pad 16: AGND -> /b1_inputs/AO2
- J6 pad 17: RX -> AGND
- J6 pad 18: AGND -> /b1_inputs/AO1
- J6 pad 19: TX -> AGND
- J6 pad 2: AGND -> unconnected-(J6-Pad2)
- J6 pad 20: AGND -> /b1_inputs/TX
- J6 pad 21: TX -> AGND
- J6 pad 22: AGND -> /b1_inputs/TX
- J6 pad 23: AUX -> AGND
- J6 pad 24: AGND -> /b1_inputs/AI8
- J6 pad 25: AO1 -> AGND
- J6 pad 26: AGND -> /b1_inputs/AI7
- J6 pad 27: AO2 -> AGND
- J6 pad 28: AGND -> /b1_inputs/AI6
- J6 pad 29: unconnected-(J6-Pad29) -> AGND
- J6 pad 3: AI2 -> AGND
- J6 pad 30: AGND -> /b1_inputs/AI5
- J6 pad 31: unconnected-(J6-Pad31) -> AGND
- J6 pad 32: AGND -> /b1_inputs/RX
- J6 pad 33: unconnected-(J6-Pad33) -> AGND
- J6 pad 34: AGND -> /b1_inputs/AI4
- J6 pad 35: unconnected-(J6-Pad35) -> AGND
- J6 pad 36: AGND -> /b1_inputs/AI3
- J6 pad 37: unconnected-(J6-Pad37) -> AGND
- J6 pad 38: AGND -> /b1_inputs/AI2
- J6 pad 39: unconnected-(J6-Pad39) -> AGND
- J6 pad 4: AGND -> unconnected-(J6-Pad4)
- J6 pad 40: AGND -> /b1_inputs/AI1
- J6 pad 5: AI3 -> AGND
- J6 pad 6: AGND -> unconnected-(J6-Pad6)
- J6 pad 7: AI4 -> AGND
- J6 pad 8: AGND -> unconnected-(J6-Pad8)
- J6 pad 9: AI5 -> AGND
- J7 pad 1: TTL1 -> +5V_RAW
- J7 pad 11: TTL6 -> unconnected-(J7-Pad11)
- J7 pad 13: TTL7 -> unconnected-(J7-Pad13)
- J7 pad 15: TTL8 -> /b5_dio_trig/OPTO_IN1
- J7 pad 17: FASTTTL1 -> /b5_dio_trig/OPTO_IN2
- J7 pad 19: FASTTTL2 -> unconnected-(J7-Pad19)
- J7 pad 21: TRIG_5V -> unconnected-(J7-Pad21)
- J7 pad 23: I2C_SDA -> /b5_dio_trig/MOD1
- J7 pad 25: I2C_SCL -> /b5_dio_trig/MOD2
- J7 pad 27: +3V3 -> /b5_dio_trig/MOD3
- J7 pad 29: +3V3 -> /b5_dio_trig/MOD4
- J7 pad 3: TTL2 -> +5V_RAW
- J7 pad 31: LED_WIFI -> /b5_dio_trig/MOD5
- J7 pad 33: LED_ACT -> /b5_dio_trig/MOD6
- J7 pad 35: unconnected-(J7-Pad35) -> /b5_dio_trig/MOD7
- J7 pad 5: TTL3 -> +3V3
- J7 pad 7: TTL4 -> unconnected-(J7-Pad7)
- J7 pad 9: TTL5 -> unconnected-(J7-Pad9)
- J8 pad 1: +5V_RAW -> /b5_dio_trig/TTL8
- J8 pad 11: GPIO7 -> /b5_dio_trig/TTL3
- J8 pad 13: GPIO15 -> /b5_dio_trig/TTL2
- J8 pad 15: GPIO43 -> /b5_dio_trig/TTL1
- J8 pad 17: GPIO44 -> unconnected-(J8-Pad17)
- J8 pad 19: MOD1 -> unconnected-(J8-Pad19)
- J8 pad 21: MOD2 -> unconnected-(J8-Pad21)
- J8 pad 23: MOD3 -> /b5_dio_trig/LED_ACT
- J8 pad 25: MOD4 -> /b5_dio_trig/LED_WIFI
- J8 pad 27: MOD5 -> +3V3
- J8 pad 29: MOD6 -> +3V3
- J8 pad 3: +5V_RAW -> /b5_dio_trig/TTL7
- J8 pad 31: MOD7 -> I2C_SCL
- J8 pad 33: unconnected-(J8-Pad33) -> I2C_SDA
- J8 pad 35: OPTO_IN1 -> /b5_dio_trig/TRIG_5V
- J8 pad 37: OPTO_IN2 -> /b5_dio_trig/FASTTTL2
- J8 pad 39: unconnected-(J8-Pad39) -> /b5_dio_trig/FASTTTL1
- J8 pad 5: +3V3 -> /b5_dio_trig/TTL6
- J8 pad 7: GPIO4 -> /b5_dio_trig/TTL5
- J8 pad 9: GPIO6 -> /b5_dio_trig/TTL4
- JP1 pad 1: GPIO43 -> /base_mcu/GPIO43
- JP1 pad 2: LED_WIFI -> /b5_dio_trig/LED_WIFI
- JP101 pad 1: AI7 -> /b1_inputs/AI7
- JP102 pad 1: AI8 -> /b1_inputs/AI8
- JP2 pad 1: GPIO44 -> /base_mcu/GPIO44
- JP2 pad 2: LED_ACT -> /b5_dio_trig/LED_ACT
- R111 pad 1: AI1 -> /b1_inputs/AI1
- R112 pad 1: AI2 -> /b1_inputs/AI2
- R113 pad 1: AI3 -> /b1_inputs/AI3
- R114 pad 1: AI4 -> /b1_inputs/AI4
- R115 pad 1: AI5 -> /b1_inputs/AI5
- R116 pad 1: AI6 -> /b1_inputs/AI6
- R309 pad 2: AO1 -> /b1_inputs/AO1
- R310 pad 2: AO2 -> /b1_inputs/AO2
- R501 pad 2: TTL1 -> /b5_dio_trig/TTL1
- R502 pad 2: TTL2 -> /b5_dio_trig/TTL2
- R503 pad 2: TTL3 -> /b5_dio_trig/TTL3
- R504 pad 2: TTL4 -> /b5_dio_trig/TTL4
- R505 pad 2: TTL5 -> /b5_dio_trig/TTL5
- R506 pad 2: TTL6 -> /b5_dio_trig/TTL6
- R507 pad 2: TTL7 -> /b5_dio_trig/TTL7
- R508 pad 2: TTL8 -> /b5_dio_trig/TTL8
- R509 pad 2: FASTTTL1 -> /b5_dio_trig/FASTTTL1
- R510 pad 2: FASTTTL2 -> /b5_dio_trig/FASTTTL2
- R511 pad 2: TRIG_5V -> /b5_dio_trig/TRIG_5V
- R710 pad 1: RX -> /nmr_rx/RX_IN
- R710 pad 2: /nmr_rx/RX_IN -> /b1_inputs/AUX
- R711 pad 1: RX -> AGND
- R711 pad 2: AGND -> /b1_inputs/AUX
- R712 pad 2: /nmr_rx/JP702A -> Net-(J3-Pin_1)
- R714 pad 2: /nmr_rx/JP702B -> Net-(J3-Pin_3)
- R923 pad 1: /nmr_rx/IF_QPF -> /nmr_rx/DIF_Q_P
- R923 pad 2: /nmr_rx/DIF_Q_P -> /nmr_rx/IF_QPF
- U101 pad 12: /b1_inputs/AIN1 -> /b1_inputs/AIN4
- U101 pad 14: /b1_inputs/AIN2 -> /b1_inputs/AIN3
- U101 pad 16: /b1_inputs/AIN3 -> /b1_inputs/AIN2
- U101 pad 18: /b1_inputs/AIN4 -> /b1_inputs/AIN1
- U101 pad 21: /b1_inputs/AIN5 -> /b1_inputs/AIN8
- U101 pad 23: /b1_inputs/AIN6 -> /b1_inputs/AIN7
- U101 pad 25: /b1_inputs/AIN7 -> /b1_inputs/AIN6
- U101 pad 27: /b1_inputs/AIN8 -> /b1_inputs/AIN5
- U201 pad 1: GND -> Net-(D201-K)
- U202 pad 1: GND -> Net-(D202-K)
- U502 pad 2: FAST_OUT1 -> /b5_dio_trig/FAST_OUT1
- U502 pad 5: FAST_OUT2 -> /b5_dio_trig/FAST_OUT2
- U505 pad 13: MOD1 -> /b5_dio_trig/MOD1
- U505 pad 14: MOD2 -> /b5_dio_trig/MOD2
- U505 pad 15: MOD3 -> /b5_dio_trig/MOD3
- U505 pad 16: MOD4 -> /b5_dio_trig/MOD4
- U505 pad 18: MOD5 -> /b5_dio_trig/MOD5
- U505 pad 19: MOD6 -> /b5_dio_trig/MOD6
- U505 pad 20: MOD7 -> /b5_dio_trig/MOD7
Routing:
- net /b5_dio_trig/TTL1: track 0.00 -> 269.9 mm, vias 0 -> 1
- net /b5_dio_trig/TTL3: track 0.00 -> 267.6 mm, vias 0 -> 1
- net /b5_dio_trig/TTL2: track 0.00 -> 265.1 mm, vias 0 -> 1
- net /b5_dio_trig/TTL5: track 0.00 -> 264.4 mm, vias 0 -> 1
- net /b5_dio_trig/TTL4: track 0.00 -> 262.4 mm, vias 0 -> 1
- net /b5_dio_trig/TTL7: track 0.00 -> 260.4 mm, vias 0 -> 1
- net /b5_dio_trig/TTL6: track 0.00 -> 259.0 mm, vias 0 -> 1
- net /b5_dio_trig/TTL8: track 0.00 -> 254.6 mm, vias 0 -> 1
- net /b2_power/USB_D_P: track 0.00 -> 100.3 mm, vias 0 -> 1
- net /b2_power/USB_D_N: track 0.00 -> 100.3 mm, vias 0 -> 1
- net /b5_dio_trig/FAST_OUT2: track 0.00 -> 39.0 mm
- net /b5_dio_trig/MOD7: track 0.00 -> 27.8 mm
- net /b1_inputs/AIN1: track 0.00 -> 27.7 mm
- net /b5_dio_trig/MOD6: track 0.00 -> 26.1 mm
- net /b1_inputs/AIN8: track 0.00 -> 25.3 mm
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