File: hardware/class-board.kicad_pcb (KiCad board)
At the start: 4 copper layers, 180 x 100 mm, 334 parts, among them J1 DevKit J1 (left row), J10 C2937625_-_Conn_01x03, J11 C2937625_-_Conn_01x03, J12 C2937625_-_Conn_01x03, J13 C492401-PZ254V-11-02P, J2 DevKit J3 (right row), J201 USB-C 16P, J202 DC005-T20, J3 C2937625_-_Conn_01x03, J4 Qwiic, J5 Expansion 2x10, J6 Panel link 2x20 female, J7 Panel link 2x20 female, J8 Panel link 2x20 female, J9 C2937625_-_Conn_01x03, J901 KF301-5.0-2P, J903 KF301-5.0-2P, J905 KF301-5.0-3P, Q901 AOD4185, Q904 AOD4184A, U101 ADS8688IDBTR, U201 LM66100DCKR, U202 LM66100DCKR, U203 78L05G-AB3-R, U204 AMS1117-3.3, U301 DAC8563SDGSR, U302 74HCT125PW, U303 OPA2192IDR, U501 SN74AHCT541PWR, U502 74HCT125PW, U503 SN74LVC1T45DBVR, U505 TCA9535PWR, U701 SI5351A-B-GT, U702 74HC74D,653, U703 OPA1656IDR, U704 DG419DY-T1-E3, U705 OPA1612AIDR, U706 OPA1612AIDR, U801 AD9834BRUZ, U802 OPA564AIDWPR, U901 TS5A23157DGSR, U902 TS5A23157DGSR, U903 DRV8871DDAR, U904 UCC27517DBVR, Y701 25 MHz

Commit message: WIP main board layout/routing (instructor), 2026-09-19 03:04; PROGRESS notes
Parts:
- moved J11 208.6 mm to (151.0, 64.0), turned to 90 degrees
- moved J10 205.4 mm to (157.9, 82.0)
- moved C711 205.0 mm to (19.1, 188.8)
- moved C721 205.0 mm to (28.8, 201.4)
- moved D703 205.0 mm to (14.9, 187.8)
- moved D704 205.0 mm to (14.9, 193.1)
- moved J3 205.0 mm to (31.8, 184.6)
- moved R712 205.0 mm to (34.1, 190.8)
- moved R714 205.0 mm to (32.3, 190.8)
- moved R715 205.0 mm to (22.6, 187.9)
- moved R722 205.0 mm to (28.8, 199.7)
- moved R724 205.0 mm to (40.4, 188.3)
- moved C710 205.0 mm to (17.4, 188.8)
- moved C712 205.0 mm to (17.4, 192.1)
- moved C720 205.0 mm to (34.9, 193.4)
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Routing:
- net +VEXT: track 0.00 -> 28.0 mm
- net /c_switch/VIN_F: track 0.00 -> 15.2 mm
- net /c_switch/VIN: track 0.00 -> 8.08 mm
- net Net-(D933-A): track 0.00 -> 3.58 mm
- net Net-(D932-A): track 0.00 -> 2.31 mm
