File: hardware/front-panel/sections/A/front-panel.kicad_pcb (KiCad board)
At the start: 4 copper layers, 180 x 100 mm, 76 parts, among them J1 Conn_02x20_Odd_Even, J10 SMA, J11 SMA, J12 SMA, J13 SMA, J14 SMA, J15 SMA, J16 SMA, J17 SMA, J18 SMA, J19 SMA, J2 Conn_02x20_Odd_Even, J20 SMA, J21 SMA, J22 SMA, J23 SMA, J24 SMA, J25 SMA, J3 Conn_02x20_Odd_Even, J30 OLED 0.96in module on 1x4 soc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, J31 KF128-2.54-10P, J32 KF128-5.0-2P, J33 Qwiic (vertical), J40 Module header 2x6 (shrouded), J411 KF301-5.0-2P, J412 KF301-5.0-2P, Q411 MMBT5551, Q412 MMBT5551, Q421 MMBT5551, Q422 MMBT5551, U401 6N137S-TA1-L, U402 6N137S-TA1-L, U410 SN74AHCT541PWR

Commit message: hardware: masters with student A's routing merged (area A + panel section A), from repo main
Co-Authored-By: Claude Fable 5.1 <noreply@anthropic.com>
Routing:
- net /TX: track 0.00 -> 226.3 mm
- net /AI8: track 0.00 -> 133.5 mm
- net /AUX: track 0.00 -> 116.2 mm
- net /AO2: track 0.00 -> 115.7 mm
- net /AI7: track 0.00 -> 108.9 mm
- net /RX: track 0.00 -> 98.5 mm
- net /AI4: track 0.00 -> 94.2 mm
- net /AI6: track 0.00 -> 83.4 mm
- net /AO1: track 0.00 -> 77.3 mm
- net /AI3: track 0.00 -> 65.1 mm
- net /AI5: track 0.00 -> 44.4 mm
- net /AI2: track 0.00 -> 42.9 mm
- net /AI1: track 0.00 -> 13.7 mm

Commit message: section A: put AUX on its correct ground plane, add GND stitching vias
Addresses Shayne's two review points. No parts moved; DRC on both boards shows
no new violation of any kind against the post-merge baseline.

1. AUX was on the wrong reference plane.

The panel stackup is F.Cu / In1.Cu=AGND / In2.Cu=GND / B.Cu, so which outer layer
a trace sits on decides which ground it references. AUX is analog but was routed
entirely on B.Cu - 13 segments over the *digital* plane, forcing its return
current into GND and across the plane split. The other twelve analog nets were
already on F.Cu; AUX was the only one wrong.

Rerouted onto F.Cu: 13 B.Cu segments removed, 8 F.Cu segments in their place.
Checked first that an F.Cu path existed without moving anything - it did. The
original router had picked B.Cu only because it was emptier, not because F.Cu was
blocked. Cost of the fix: 172 mm instead of 107 mm, because F.Cu is congested. For
an analog net a correct return path is worth more than 65 mm of length, but that
is a judgement call and worth a second opinion.

2. Signal vias had no local return path.

36 of the 38 signal vias inside ZONE_A had no ground via within 2 mm, several over
10 mm away. A via that changes layer forces its return current to change reference
plane, and with no ground via nearby the return has to loop until it finds one -
that loop is what radiates.

Added 17 GND stitching vias (0.6/0.3 mm) beside my own signal vias (-12V, +3V3,
+12V, +5VA), clustered so one via covers several. Under-stitched vias in ZONE_A:
36/38 -> 13/38. The 13 left are TTL vias belonging to section B and the TX net, so
not mine to fix - flagging rather than touching them.

Note on net choice: the stitching vias are GND, not AGND. Both inner layers are
GND, so only a GND via actually reaches them; an AGND via would be cleared out of
those planes and would only join the outer AGND pours.

Two of my signal vias (+5VA at 128.90,41.85 and -12V at 139.60,42.05) had no legal
spot within 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
Routing:
- net /AUX: track 116.2 -> 172.0 mm
