File: hardware/front-panel/sections/A/front-panel.kicad_pcb (KiCad board)
At the start: 4 copper layers, 180 x 100 mm, 76 parts, among them J1 Conn_02x20_Odd_Even, J10 SMA, J11 SMA, J12 SMA, J13 SMA, J14 SMA, J15 SMA, J16 SMA, J17 SMA, J18 SMA, J19 SMA, J2 Conn_02x20_Odd_Even, J20 SMA, J21 SMA, J22 SMA, J23 SMA, J24 SMA, J25 SMA, J3 Conn_02x20_Odd_Even, J30 OLED 0.96in module on 1x4 soc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, J31 KF128-2.54-10P, J32 KF128-5.0-2P, J33 Qwiic (vertical), J40 Module header 2x6 (shrouded), J411 KF301-5.0-2P, J412 KF301-5.0-2P, Q411 MMBT5551, Q412 MMBT5551, Q421 MMBT5551, Q422 MMBT5551, U401 6N137S-TA1-L, U402 6N137S-TA1-L, U410 SN74AHCT541PWR

Commit message: Sections re-split from the instructor's 2026-09-25 masters (panel complete: 0 unconnected; main board 73 unconnected)
Co-Authored-By: Claude Fable 5.1 <noreply@anthropic.com>
Parts:
- moved R472 8.80 mm to (47.4, 91.5)
- moved C402 6.30 mm to (47.5, 95.9), turned to -90 degrees
- moved R451 5.63 mm to (91.5, 91.1), turned to -90 degrees
- moved R461 5.17 mm to (89.3, 91.0), turned to -90 degrees
- moved R442 4.98 mm to (66.8, 99.3)
- moved R441 4.95 mm to (94.3, 99.2)
- moved R471 4.72 mm to (74.5, 89.0)
- moved Q421 1.70 mm to (94.5, 90.8)
- moved D421 1.36 mm to (92.5, 102.5), turned to 180 degrees
- moved C410 1.33 mm to (39.5, 90.9), turned to 0 degrees
- moved R432 0.98 mm to (64.4, 99.2)
- moved R431 0.75 mm to (92.1, 99.3)
- moved C401 0.72 mm to (73.9, 92.0), turned to 180 degrees
- moved Q411 0.47 mm to (93.3, 95.4), turned to 0 degrees
- turned Q412 to 0 degrees
Connections:
- J14 pad 5: /TX -> /RX
- J20 pad 5: /RX -> /TX
Routing:
- net +3V3: track 0.00 -> 299.0 mm, vias 0 -> 3
- net GND: track 242.2 -> 32.1 mm, vias 1 -> 21
- net /AUX: track 244.8 -> 110.0 mm
- net +5V_RAW: track 0.00 -> 120.2 mm
- net /TX: track 100.3 -> 206.6 mm
- net /OPTO_IN1: track 0.00 -> 89.1 mm
- net /I2C_SDA: track 0.00 -> 65.7 mm
- net /OPTO_IN2: track 0.00 -> 65.5 mm
- net /I2C_SCL: track 0.00 -> 63.8 mm
- net /LED_ACT: track 0.00 -> 56.7 mm
- net /LED_WIFI: track 0.00 -> 56.7 mm
- net /MOD1: track 0.00 -> 51.2 mm
- net /MOD2: track 0.00 -> 46.4 mm
- net /TRIG_5V: track 0.00 -> 45.4 mm
- net /ISO2_IN-: track 0.00 -> 45.3 mm
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- added copper zone on F.Cu, net /TX
Other:
- board text removed: "J1 = J8"
- board text removed: "J1 J2 J3 mate J6 J7 J8 of the main board; pin 1 marked"
- board text removed: "J1 pin 1"
- board text removed: "J1 pin 40"
- board text removed: "J2 pin 1"
- board text removed: "J2 pin 40"
