File: hardware/sections/A/class-board.kicad_pcb (KiCad board)
At the start: 4 copper layers, 180 x 100 mm, 334 parts, among them J1 DevKit J1 (left row), J10 C2937625_-_Conn_01x03, J11 C2937625_-_Conn_01x03, J12 C2937625_-_Conn_01x03, J13 C492401-PZ254V-11-02P, J14 C2937625_-_Conn_01x03, J15 C2937625_-_Conn_01x03, J2 DevKit J3 (right row), J201 USB-C 16P, J202 DC005-T20, J3 C2937625_-_Conn_01x03, J4 Qwiic, J5 Expansion 2x10, J6 Panel link 2x20 female, J7 Panel link 2x20 female, J8 Panel link 2x20 female, J9 C2937625_-_Conn_01x03, J901 KF301-5.0-2P, J903 KF301-5.0-2P, J905 KF301-5.0-3P, Q901 AOD4185, Q904 AOD4184A, U101 ADS8688IDBTR, U201 LM66100DCKR, U202 LM66100DCKR, U203 78L05G-AB3-R, U204 AMS1117-3.3, U301 DAC8563SDGSR, U302 74HCT125PW, U303 OPA2192IDR, U501 SN74AHCT541PWR, U502 74HCT125PW, U503 SN74LVC1T45DBVR, U505 TCA9535PWR, U701 SI5351A-B-GT, U702 74HC74D,653, U703 OPA1656IDR, U704 DG419DY-T1-E3, U705 OPA1612AIDR, U706 OPA1612AIDR, U801 AD9834BRUZ, U802 OPA564AIDWPR, U901 TS5A23157DGSR, U902 TS5A23157DGSR, U903 DRV8871DDAR, U904 UCC27517DBVR, Y701 25 MHz

Commit message: section A: put AUX on its correct ground plane, add GND stitching vias
Addresses Shayne's two review points. No parts moved; DRC on both boards shows
no new violation of any kind against the post-merge baseline.

1. AUX was on the wrong reference plane.

The panel stackup is F.Cu / In1.Cu=AGND / In2.Cu=GND / B.Cu, so which outer layer
a trace sits on decides which ground it references. AUX is analog but was routed
entirely on B.Cu - 13 segments over the *digital* plane, forcing its return
current into GND and across the plane split. The other twelve analog nets were
already on F.Cu; AUX was the only one wrong.

Rerouted onto F.Cu: 13 B.Cu segments removed, 8 F.Cu segments in their place.
Checked first that an F.Cu path existed without moving anything - it did. The
original router had picked B.Cu only because it was emptier, not because F.Cu was
blocked. Cost of the fix: 172 mm instead of 107 mm, because F.Cu is congested. For
an analog net a correct return path is worth more than 65 mm of length, but that
is a judgement call and worth a second opinion.

2. Signal vias had no local return path.

36 of the 38 signal vias inside ZONE_A had no ground via within 2 mm, several over
10 mm away. A via that changes layer forces its return current to change reference
plane, and with no ground via nearby the return has to loop until it finds one -
that loop is what radiates.

Added 17 GND stitching vias (0.6/0.3 mm) beside my own signal vias (-12V, +3V3,
+12V, +5VA), clustered so one via covers several. Under-stitched vias in ZONE_A:
36/38 -> 13/38. The 13 left are TTL vias belonging to section B and the TX net, so
not mine to fix - flagging rather than touching them.

Note on net choice: the stitching vias are GND, not AGND. Both inner layers are
GND, so only a GND via actually reaches them; an AGND via would be cleared out of
those planes and would only join the outer AGND pours.

Two of my signal vias (+5VA at 128.90,41.85 and -12V at 139.60,42.05) had no legal
spot within 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
Routing:
- net GND: vias 70 -> 87

Commit message: main board area A: route +5V_RAW; four left, and why
+5V_RAW (U501 pad 20 -> J7) now routes: 6 tracks + 3 vias. DRC unchanged against
baseline - clearance 0, every other count identical. No parts moved, nothing
outside ZONE_A, nothing on an inner layer. ZONE_A remaining: 5 -> 4.

Two of my own router settings, not the board, were blocking this:

- the via penalty was set to 12 mm, left over from an earlier experiment. That is
  so punitive the search reports "no path" rather than drop to B.Cu for two hops.
  Now 3 mm.
- the seed margin was 0.15 mm, added earlier to fix a U501 clearance miss. It was
  strict enough that no starting cell qualified at all, so every route failed
  before it began. Now 0.03 mm, and the U501 clearance is still clean.

The remaining four are around U101 and are a real geometric limit, not a settings
problem. Sampling free space within 0.3 mm of each endpoint:

    AGND    F.Cu  85/180 free      B.Cu 180/180
    +5VA    F.Cu   0/180 free      B.Cu 180/180
    AIN7    F.Cu   0/180 free      B.Cu 175/180
    AIN8    F.Cu  34/180 free      B.Cu   5/180

+5VA and AIN7 are sealed on F.Cu - no free copper in any direction - so the only
escape is a via. The smallest via on this board is 0.6/0.3 mm, which needs about
0.6 mm of room from neighbouring pad edges once clearance is added (0.3 mm for the
AIN nets under analog_in_clearance). U101 is on 0.5 mm pitch. It does not fit.

So these need what Shayne suggested: a neighbouring track ripped up and re-routed
by another path to open an escape corridor, rather than a cleverer search. Which
track to sacrifice is a judgement call about his layout, so it is going to him as
a question rather than a guess.

Recorded so it is not re-derived later: an earlier diagnostic claimed all five were
routable. It was wrong - it seeded both layers at the endpoints, so it "escaped"
onto B.Cu without paying for a via, producing paths that connect nothing. Layer
pinning at the endpoints is what makes the search honest.

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
Routing:
- net +5V_RAW: track 89.1 -> 108.1 mm, vias 0 -> 3
Changed lines of the file:
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@@
+	)
+	(segment
+		(start 163.840002 40.51)
+		(end 166.390002 40.51)
+		(width 0.8)
+		(layer "F.Cu")
+		(net "+5V_RAW")
 	)
 	(segment
@@
 	)
 	(segment
+		(start 166.390002 40.51)
+		(end 168.540002 38.36)
+		(width 0.8)
+		(layer "F.Cu")
+		(net "+5V_RAW")
+	)
+	(segment
 		(start 6.55 34.624999)
 		(end 6.525001 34.6)
@@
 		(net "+5V_RAW")
 	)
+	(via
+		(at 157.540002 39.01)
+		(size 0.8)
+		(drill 0.4)
+		(layers "F.Cu" "B.Cu")
+		(net "+5V_RAW")
+	)
+	(via
+		(at 163.840002 40.51)
+		(size 0.8)
+		(drill 0.4)
+		(layers "F.Cu" "B.Cu")
+		(net "+5V_RAW")
+	)
+	(via
+		(at 168.540002 38.36)
+		(size 0.8)
+		(drill 0.4)
+		(layers "F.Cu" "B.Cu")
+		(net "+5V_RAW")
+	)
+	(segment
+		(start 159.040002 40.51)
+		(end 163.840002 40.51)
+		(width 0.8)
+		(layer "B.Cu")
+		(net "+5V_RAW")
+	)
+	(segment
+		(start 168.540002 38.36)
+		(end 168.540002 36.16)
+		(width 0.8)
+		(layer "B.Cu")
+		(net "+5V_RAW")
+	)
+	(segment
+		(start 157.540002 39.01)
+		(end 159.040002 40.51)
+		(width 0.8)
+		(layer "B.Cu")
+		(net "+5V_RAW")
+	)
+	(segment
+		(start 168.540002 36.16)
+		(end 171.73 33.41)
+		(width 0.8)
+		(layer "B.Cu")
+		(net "+5V_RAW")
+	)
