File: hardware/front-panel/sections/B/front-panel.kicad_pcb (KiCad board)
At the start: 4 copper layers, 180 x 100 mm, 76 parts, among them J1 Conn_02x20_Odd_Even, J10 SMA, J11 SMA, J12 SMA, J13 SMA, J14 SMA, J15 SMA, J16 SMA, J17 SMA, J18 SMA, J19 SMA, J2 Conn_02x20_Odd_Even, J20 SMA, J21 SMA, J22 SMA, J23 SMA, J24 SMA, J25 SMA, J3 Conn_02x20_Odd_Even, J30 OLED 0.96in module on 1x4 soc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, J31 KF128-2.54-10P, J32 KF128-5.0-2P, J33 Qwiic (vertical), J40 Module header 2x6 (shrouded), J411 KF301-5.0-2P, J412 KF301-5.0-2P, Q411 MMBT5551, Q412 MMBT5551, Q421 MMBT5551, Q422 MMBT5551, U401 6N137S-TA1-L, U402 6N137S-TA1-L, U410 SN74AHCT541PWR

Commit message: panel section B: 200 track segments (work in progress snapshot)
Safety snapshot taken before merging 14 upstream commits, which also
modify this section's board file. Also contains three PWR_AGND symbols
changed to PWR_GND in the sheet, which needs review: the section rules
say the schematic is not the student's to edit.

Co-Authored-By: Claude Opus 5 (1M context) <noreply@anthropic.com>
Parts:
- moved J13 18.2 mm to (111.5, 61.7)
- moved J12 17.8 mm to (129.4, 61.5)
Routing:
- net GND: track 0.00 -> 242.2 mm, vias 0 -> 1
- net /TTL1: track 0.00 -> 67.6 mm
- net /MOD5: track 0.00 -> 66.7 mm
- net /TTL2: track 0.00 -> 62.3 mm
- net /TTL3: track 0.00 -> 57.8 mm
- net /TTL4: track 0.00 -> 52.2 mm
- net /TTL5: track 0.00 -> 47.2 mm
- net /TTL6: track 0.00 -> 42.0 mm
- net /TTL7: track 0.00 -> 36.8 mm
- net /FASTTTL1: track 0.00 -> 35.6 mm
- net /TTL8: track 0.00 -> 31.8 mm
- net /FASTTTL2: track 0.00 -> 20.2 mm
- net /ISO1_IN+: track 0.00 -> 13.3 mm
- net /ISO2_B: track 0.00 -> 13.1 mm
- net /MODOUT3: track 0.00 -> 11.2 mm
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- added copper zone on B.Cu, net AGND
- added copper zone on In2.Cu, net AGND
- added copper zone on F.Cu, net GND
- added copper zone on In1.Cu, net GND
Other:
- board outline removed
