File: hardware/front-panel/sections/B/front-panel.kicad_sch (KiCad schematic)
At the start: 76 parts, among them J1 Conn_02x20_Odd_Even, J10 SMA, J11 SMA, J12 SMA, J13 SMA, J14 SMA, J15 SMA, J16 SMA, J17 SMA, J18 SMA, J19 SMA, J2 Conn_02x20_Odd_Even, J20 SMA, J21 SMA, J22 SMA, J23 SMA, J24 SMA, J25 SMA, J3 Conn_02x20_Odd_Even, J30 OLED 0.96in module on 1x4 soc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, J31 KF128-2.54-10P, J32 KF128-5.0-2P, J33 Qwiic (vertical), J40 Module header 2x6 (shrouded), J411 KF301-5.0-2P, J412 KF301-5.0-2P, Q411 MMBT5551, Q412 MMBT5551, Q421 MMBT5551, Q422 MMBT5551, U401 6N137S-TA1-L, U402 6N137S-TA1-L, U410 SN74AHCT541PWR

Commit message: panel section B: 200 track segments (work in progress snapshot)
Safety snapshot taken before merging 14 upstream commits, which also
modify this section's board file. Also contains three PWR_AGND symbols
changed to PWR_GND in the sheet, which needs review: the section rules
say the schematic is not the student's to edit.

Co-Authored-By: Claude Opus 5 (1M context) <noreply@anthropic.com>
Connections:
- net AGND: no longer J12.1 (GND), J12.2 (GND), J12.3 (GND), J12.4 (GND), J15.1 (GND), J15.2 (GND), J15.3 (GND), J15.4 (GND), J21.1 (GND), J21.2 (GND), J21.3 (GND), J21.4 (GND)
- net GND: now also J12.1 (GND), J12.2 (GND), J12.3 (GND), J12.4 (GND), J15.1 (GND), J15.2 (GND), J15.3 (GND), J15.4 (GND), J21.1 (GND), J21.2 (GND), J21.3 (GND), J21.4 (GND)
